File: Modules/PowerSupply/LION1CELL01B/SCH_PCB/untitled.brd (EAGLE design)
At the start: 80.8 x 50.3 mm, 87 parts, among them P1 BSMD, P2 1.1A, T1 IRLML6244, U1 BQ24103, X1 BQ34Z100PW, X10 TPS63036, X3 SN74HC164D, X4 BQ294602, X5 SROUB3M, X6 SROUB3M, X7 SROUB3M, X8 SROUB3M, X9 APX809-26SAG-7

Commit message: 
Parts:
- R12: value 10k -> 0R
