File: Modules/Sensors/RPS01A/PCB/RPS01A.sch (KiCad schematic (older format))
At the start: 17 parts, among them J1 JUMP_5X2, J2 JUMP_2x1, J3 JUMP_5X2, P1 _, P2 _, P3 _, P4 _, U1 AS5048B

Commit message: upravy PCB a vygenerovani technologickych dat.
Parts:
- added C3: 10uF, symbol CP
- added D1: M4, symbol D
- R6, R7: value 0R -> 10k
Connections:
- wire segments 45 -> 51
Changed lines of the file:
@@
 LIBS:contrib
 LIBS:valves
-LIBS:MLAB_IO
-LIBS:Jumpers
 LIBS:RPS01A-cache
-EELAYER 24 0
+EELAYER 25 0
 EELAYER END
 $Descr A4 11693 8268
@@
 $EndComp
 Wire Wire Line
-	5950 3300 6500 3300
-Wire Wire Line
-	6050 3350 6050 3300
+	5950 3300 6600 3300
+Wire Wire Line
+	6050 3300 6050 3400
 Connection ~ 6050 3300
 Wire Wire Line
-	6300 3100 6300 3350
+	6300 3100 6300 3400
 Connection ~ 6300 3200
 $Comp
@@
 $EndComp
 Wire Wire Line
-	6050 3800 6050 3750
-Wire Wire Line
-	6300 3800 6300 3750
+	6050 3700 6050 3800
+Wire Wire Line
+	6300 3700 6300 3800
 $Comp
 L R R1
@@
 $EndComp
 Wire Wire Line
-	7050 3300 7000 3300
-Wire Wire Line
-	7050 3100 7050 3300
+	6900 3300 7050 3300
+Wire Wire Line
+	7050 3300 7050 3100
 $Comp
 L JUMP_5X2 J1
@@
 $EndComp
 Wire Wire Line
-	9400 4800 9400 5000
-Wire Wire Line
-	9550 4800 9550 5000
-Wire Wire Line
-	9400 5500 9400 5550
-Wire Wire Line
-	9550 5500 9550 5550
+	9400 4700 9400 5100
+Wire Wire Line
+	9550 4700 9550 5100
+Wire Wire Line
+	9400 5400 9400 5550
+Wire Wire Line
+	9550 5400 9550 5550
 Wire Wire Line
 	9400 4850 9700 4850
@@
 A2
 Wire Wire Line
-	9400 4300 9400 4250
-Wire Wire Line
-	9550 4300 9550 4250
+	9400 4250 9400 4400
+Wire Wire Line
+	9550 4250 9550 4400
 $Comp
 L _ P1
@@
 P 4700 2600
 F 0 "R6" V 4780 2600 40  0000 C CNN
-F 1 "0R" V 4707 2601 40  0000 C CNN
+F 1 "10k" V 4707 2601 40  0000 C CNN
 F 2 "" V 4630 2600 30  0000 C CNN
 F 3 "" H 4700 2600 30  0000 C CNN
@@
 P 4900 2600
 F 0 "R7" V 4980 2600 40  0000 C CNN
-F 1 "0R" V 4907 2601 40  0000 C CNN
+F 1 "10k" V 4907 2601 40  0000 C CNN
 F 2 "" V 4830 2600 30  0000 C CNN
 F 3 "" H 4900 2600 30  0000 C CNN
@@
 $EndComp
 Wire Wire Line
-	4700 2850 4700 3100
+	4700 2750 4700 3100
 Connection ~ 4700 3100
 Wire Wire Line
-	4900 2850 4900 3300
+	4900 2750 4900 3300
 Connection ~ 4900 3300
 $Comp
@@
 $EndComp
 Wire Wire Line
-	4700 2350 4700 2300
-Wire Wire Line
-	4900 2350 4900 2300
+	4700 2300 4700 2450
+Wire Wire Line
+	4900 2300 4900 2450
 $Comp
 L JUMP_5X2 J3
@@
 Wire Wire Line
 	4700 1650 4700 1600
+$Comp
+L VDD #PWR018
+U 1 1 55134882
+P 6200 1400
+F 0 "#PWR018" H 6200 1500 30  0001 C CNN
+F 1 "VDD" H 6200 1510 30  0000 C CNN
+F 2 "" H 6200 1400 60  0000 C CNN
+F 3 "" H 6200 1400 60  0000 C CNN
+	1    6200 1400
+	1    0    0    -1
+$EndComp
+Wire Wire Line
+	6200 1400 6200 1550
+$Comp
+L CP C3
+U 1 1 55133722
+P 6000 1750
+F 0 "C3" H 6025 1850 50  0000 L CNN
+F 1 "10uF" H 6025 1650 50  0000 L CNN
+F 2 "" H 6038 1600 30  0000 C CNN
+F 3 "" H 6000 1750 60  0000 C CNN
+	1    6000 1750
+	1    0    0    -1
+$EndComp
+$Comp
+L D D1
+U 1 1 551338EE
+P 6400 1750
+F 0 "D1" H 6400 1850 50  0000 C CNN
+F 1 "M4" H 6400 1650 50  0000 C CNN
+F 2 "" H 6400 1750 60  0000 C CNN
+F 3 "" H 6400 1750 60  0000 C CNN
+	1    6400 1750
+	0    -1   -1   0
+$EndComp
+$Comp
+L GND #PWR019
+U 1 1 55133AAC
+P 6400 1950
+F 0 "#PWR019" H 6400 1950 30  0001 C CNN
+F 1 "GND" H 6400 1880 30  0001 C CNN
+F 2 "" H 6400 1950 60  0000 C CNN
+F 3 "" H 6400 1950 60  0000 C CNN
+	1    6400 1950
+	1    0    0    -1
+$EndComp
+$Comp
+L GND #PWR020
+U 1 1 55133AC5
+P 6000 1950
+F 0 "#PWR020" H 6000 1950 30  0001 C CNN
+F 1 "GND" H 6000 1880 30  0001 C CNN
+F 2 "" H 6000 1950 60  0000 C CNN
+F 3 "" H 6000 1950 60  0000 C CNN
+	1    6000 1950
+	1    0    0    -1
+$EndComp
+Wire Wire Line
+	6000 1550 6400 1550
+Wire Wire Line
+	6000 1550 6000 1600
+Wire Wire Line
+	6400 1550 6400 1600
+Connection ~ 6200 1550
+Wire Wire Line
+	6000 1900 6000 1950
+Wire Wire Line
+	6400 1900 6400 1950
 $EndSCHEMATC
