File: H_Bridge/DRV8835HB01B/SCH_PCB/DRV8835HB01B.kicad_pcb (KiCad board)
At the start: 2 copper layers, 30 x 40.1 mm, 25 parts, among them J1 JUMP_3X2, J10 WAGO256, J11 WAGO256, J12 WAGO256, J13 WAGO256, J2 CONN1_1, J3 JUMP_2x1, J4 JUMP_2x1, J5 JUMP_2x1, J6 JUMP_2x1, J7 JUMP2_2x1, J8 WAGO256, J9 WAGO256, M1 HOLE, M2 HOLE, M3 HOLE, M4 HOLE, U1 DRV8835

Commit message: zmena
Routing:
- net GND: track 0.00 -> 36.9 mm, vias 0 -> 15
- net /AIN2: track 0.00 -> 22.5 mm
- net /BIN2: track 0.00 -> 19.7 mm
- net /BIN1: track 0.00 -> 16.8 mm
- net Net-(J7-Pad1): track 2.66 -> 16.6 mm
- net /AOUT1: track 0.00 -> 10.9 mm
- net /AOUT2: track 0.00 -> 6.82 mm
- net /VM: track 11.7 -> 16.8 mm
- net /AIN1: track 14.4 -> 17.8 mm
