File: Modules/Sensors/SHT31V01A/SCH_PCB/SHT31V01A.sch (KiCad schematic (older format))
At the start: 24 parts, among them J1 CONN1_1, J10 JUMP_2x1, J11 JUMP_2x1, J12 JUMP_2x1, J13 JUMP_2x1, J2 CONN1_1, J3 CONN1_1, J4 CONN1_1, J5 CONN1_1, J6 CONN1_1, J7 CONN1_1, J8 CONN1_1, J9 JUMP_2x1, M1 HOLE, M2 HOLE, U1 SHT31

Commit message: Nahrani dokumentace
Parts:
- removed J3, J4, J5, J6, J7, J8: CONN1_1, Mlab_Pin_Headers:SMD_1_2x1, symbol CONN1_1
- D1: value BZV55C-3,6V -> BZV55C-5,6V
Other:
- moved on the sheet: C1, D1, J1, J10, J11, J12, J13, J2, J9, M1, M2, R1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
