File: Modules/OpAmps/OZDUAL03A/SCH_PCB/OZDUAL03A.sch (KiCad schematic (older format))
At the start: 47 parts, among them J1 Umin ... Umax, M1 HOLE, M2 HOLE, M3 HOLE, M4 HOLE

Commit message: uprava schematu
Parts:
- removed C1: C/U, symbol CP_Small
- removed C2: 100nF, symbol C_Small
- removed C? (x2): C, symbol C
- removed D1: M4, symbol D_Small
- removed D?: TL431D, SO8, symbol TL431D
- removed D?: TL431DBZ, SOT-23, symbol TL431DBZ
- removed GS? (x4): GS3, GS3, symbol GS3
- removed J1: Umin ... Umax, symbol HEADER_2x03_PARALLEL
- removed R? (x3): R, symbol R
- added C? (x4): C/U, symbol CP_Small
- added C? (x2): 100nF, symbol C_Small
- added C? (x5): C, symbol C
- added D? (x2): M4, symbol D_Small
- added J?: JUMP2_2x1, symbol JUMP2_2x1
- added J?: POWER, symbol HEADER_2x05_PARALLEL
- added J?: OPAMPA, symbol HEADER_2x05_PARALLEL
- added J?: OPAMPB, symbol HEADER_2x05_PARALLEL
- added J?: TRANSISTOR, symbol HEADER_2x05_PARALLEL
- added Q?: MOSFET-N, SOT-23, symbol MOSFET-N
- added R? (x6): R, symbol R
- added U?: MAX6066, SOT-23, symbol ISL21070CIH320Z-TK
Connections:
- net labels added: D, G, GNDA, INA+, INA-, INB+, INB-, OUTA, OUTB, S, VIN+, VIN-, VSS
- net labels removed: (OUT+), (OUT-), IN1+, IN1-, IN2+, IN2-, OUT1, OUT2
- wire segments 164 -> 186
Other:
- note added: "REFERENCE\n"
- note added: "TRANSISTOR"
- note removed: "možná zapojení 1OZ:\nzesilovač\n invertující\n neinvertující\n rozdílový\n derivační\n integrační (nábojový) \npropust 1. řádu\n horní\n dolní\n pásmová\nSchmittův KO\nmultivibrátor\n\nmožná zapojení 2OZ:\nzesilovač\n jednoduchý vstup->diferenciální výstup\n diferenciální vstup->diferenciální výstup\nfiltry diferenciálního signálu"
- moved on the sheet: C?, M1, M2, M3, M4, R?, U?B

Commit message: pcb
Parts:
- removed Q?: MOSFET-N, SOT-23, symbol MOSFET-N
- added Q1: 2N7002, Mlab_IO:SOT-23, symbol 2N7002
- C1, C10, C11, C12, C13, C14, C15, C16, C17, C18, C19, C2, C20, C21, C3, C4, C5, C6, C7, C8, C9: renamed from C?; footprint (none) -> Mlab_R:SMD-0805
- D1, D2: renamed from D?; footprint (none) -> Mlab_D:LED_0805
- J1: renamed from J?; footprint (none) -> Mlab_Pin_Headers:Straight_2x01
- J2, J3, J4, J5: renamed from J?; footprint (none) -> Mlab_Pin_Headers:Straight_2x05
- M1, M2, M3, M4: footprint (none) -> Mlab_Mechanical:MountingHole_3mm
- R1, R10, R11, R12, R13, R14, R15, R16, R17, R18, R19, R2, R20, R21, R22, R3, R4, R5, R6, R7, R8, R9: renamed from R?; footprint (none) -> Mlab_R:SMD-0805
- U1: renamed from U?; value LM358 -> OZ; footprint (none) -> Mlab_IO:SO-8
- U2: renamed from U?; footprint SOT-23 -> Mlab_IO:SOT-23
Connections:
- wire segments 186 -> 134

Commit message: rastr
Parts:
- removed C16, C17, C19: C, Mlab_R:SMD-0805, symbol C
- removed Q1: 2N7002, Mlab_IO:SOT-23, symbol 2N7002
- removed R11, R12, R18, R19: R, Mlab_R:SMD-0805, symbol R
- added e5, i5: R, Mlab_R:SMD-0805, symbol R
- J5: value TRANSISTOR -> VREF/TRANSISTOR
- renumbered C1 to a5, C2 to b1, R3 to b5, R5 to c1, C3 to c2, C4 to c3, R1 to c4, R4 to c5, C5 to d1, R8 to d2, R7 to d3, R2 to d4, R6 to d5, D2 to e1, C10 to e2, C9 to f1, C11 to f2, C12 to f5, R10 to g1, R9 to g2, C6 to h1, C7 to h2, C13 to h5, D1 to i1, C8 to i2, C21 to j1, R22 to j2, R21 to j3, R16 to j4, R15 to j5, C14 to k1, C18 to k2, C20 to k3, R17 to k4, R20 to k5, R14 to l1, R13 to l5, C15 to m5
Connections:
- net labels added: T1, T3, VREF/T2, VREFA, VREFB
- net labels removed: D, G, S, VREF
- wire segments 134 -> 115
Other:
- note added: "REFERENCE/TRANSISTOR"
- note removed: "REFERENCE\n"
- note removed: "TRANSISTOR"
- moved on the sheet: J2, J3, J4, J5, U2, f5, h5

Commit message: pridani kot a srovnani potisku.
Parts:
- a5, b1, c2, c3, d1, f5, h5, j1, k1, k2, k3, m5: symbol C -> C-RESCUE-OZDUAL03A
Changed lines of the file:
@@
 EESchema Schematic File Version 2
-LIBS:MLAB_BATERY
-LIBS:MLAB_CONNECTORS
-LIBS:MLAB_D
-LIBS:MLAB_DISPLAY
-LIBS:MLAB_HEADER
-LIBS:MLAB_IO
-LIBS:MLAB_Jumpers
-LIBS:MLAB_MECHANICAL
-LIBS:MLAB_SW
-LIBS:MLAB_T
-LIBS:MLAB_U
-LIBS:mlab-default-cache
+LIBS:OZDUAL03A-rescue
 LIBS:74xgxx
 LIBS:74xx
@@
 $EndComp
 $Comp
-L C c2
+L C-RESCUE-OZDUAL03A c2
 U 1 1 574854BB
 P 4800 2350
@@
 $EndComp
 $Comp
-L C d1
+L C-RESCUE-OZDUAL03A d1
 U 1 1 574882F0
 P 3850 3500
@@
 $EndComp
 $Comp
-L C c3
+L C-RESCUE-OZDUAL03A c3
 U 1 1 5749B98D
 P 2550 3250
@@
 $EndComp
 $Comp
-L C a5
+L C-RESCUE-OZDUAL03A a5
 U 1 1 574D513E
 P 2550 1450
@@
 $EndComp
 $Comp
-L C b1
+L C-RESCUE-OZDUAL03A b1
 U 1 1 574D5CE9
 P 3850 1150
@@
 $EndComp
 $Comp
-L C k2
+L C-RESCUE-OZDUAL03A k2
 U 1 1 574D6C2E
 P 4750 5800
@@
 $EndComp
 $Comp
-L C k1
+L C-RESCUE-OZDUAL03A k1
 U 1 1 574D6C58
 P 3850 4650
@@
 $EndComp
 $Comp
-L C m5
+L C-RESCUE-OZDUAL03A m5
 U 1 1 574D6C6A
 P 2550 4900
@@
 OUTB
 $Comp
-L C k3
+L C-RESCUE-OZDUAL03A k3
 U 1 1 574D6CA2
 P 2550 6700
@@
 $EndComp
 $Comp
-L C j1
+L C-RESCUE-OZDUAL03A j1
 U 1 1 574D6CAA
 P 3850 7000
@@
 VREF/T2
 $Comp
-L C f5
+L C-RESCUE-OZDUAL03A f5
 U 1 1 57618EB4
 P 6350 4350
@@
 $EndComp
 $Comp
-L C h5
+L C-RESCUE-OZDUAL03A h5
 U 1 1 5761FADF
 P 7350 4600

Commit message: oboustrany pcb
Parts:
- added c0, c9: C, Mlab_R:SMD-0805, symbol C-RESCUE-OZDUAL03A
- C1: renamed from h1; value C/U -> 47u; footprint Mlab_R:SMD-0805 -> Mlab_C:TantalC_SizeC_Reflow
- C2: renamed from f1; value C/U -> 47u; footprint Mlab_R:SMD-0805 -> Mlab_C:TantalC_SizeC_Reflow
- C3: renamed from h2; value C/U -> 47u; footprint Mlab_R:SMD-0805 -> Mlab_C:TantalC_SizeC_Reflow
- C4: renamed from e2; value C/U -> 47u; footprint Mlab_R:SMD-0805 -> Mlab_C:TantalC_SizeC_Reflow
- D1: renamed from i1; footprint Mlab_D:LED_0805 -> Mlab_D:Diode-SMA_Standard
- D2: renamed from e1; footprint Mlab_D:LED_0805 -> Mlab_D:Diode-SMA_Standard
- U2: footprint Mlab_IO:SOT-23 -> sot23-6:SOT-23-6
- renumbered g2 to R1, g1 to R2, c2 to a0, d2 to a1, b1 to a2, c1 to a3, d1 to a4, i2 to a5, k1 to a6, l1 to a7, j2 to a8, k2 to a9, c3 to b0, d3 to b1, d4 to b2, j1 to b7, j3 to b8, k3 to b9, a5 to c1, c4 to c2, f2 to c3, f5 to c4, h5 to c5, j4 to c6, m5 to c7, k4 to c8, b5 to d0, c5 to d1, d5 to d2, e5 to d3, i5 to d6, j5 to d7, l5 to d8, k5 to d9
Connections:
- net GNDA: now also c0.2, c9.2
- net VREFA: now also c0.1
- net VREFB: now also c9.1

Commit message: uprava popisku
Parts:
- C1, C2, C3, C4: footprint Mlab_C:TantalC_SizeC_Reflow -> sot23-6:TantalC_SizeC_Reflow
Changed lines of the file:
@@
 F 0 "C1" H 6700 1350 50  0000 L CNN
 F 1 "47u" H 6700 1150 50  0000 L CNN
-F 2 "Mlab_C:TantalC_SizeC_Reflow" H 6700 1250 60  0001 C CNN
+F 2 "sot23-6:TantalC_SizeC_Reflow" H 6700 1250 60  0001 C CNN
 F 3 "" H 6700 1250 60  0000 C CNN
 	1    6700 1250
@@
 F 0 "C3" H 7400 1350 50  0000 L CNN
 F 1 "47u" H 7400 1150 50  0000 L CNN
-F 2 "Mlab_C:TantalC_SizeC_Reflow" H 7400 1250 60  0001 C CNN
+F 2 "sot23-6:TantalC_SizeC_Reflow" H 7400 1250 60  0001 C CNN
 F 3 "" H 7400 1250 60  0000 C CNN
 	1    7400 1250
@@
 F 0 "C2" H 6700 2050 50  0000 L CNN
 F 1 "47u" H 6700 1850 50  0000 L CNN
-F 2 "Mlab_C:TantalC_SizeC_Reflow" H 6700 1950 60  0001 C CNN
+F 2 "sot23-6:TantalC_SizeC_Reflow" H 6700 1950 60  0001 C CNN
 F 3 "" H 6700 1950 60  0000 C CNN
 	1    6700 1950
@@
 F 0 "C4" H 7400 2050 50  0000 L CNN
 F 1 "47u" H 7400 1850 50  0000 L CNN
-F 2 "Mlab_C:TantalC_SizeC_Reflow" H 7400 1950 60  0001 C CNN
+F 2 "sot23-6:TantalC_SizeC_Reflow" H 7400 1950 60  0001 C CNN
 F 3 "" H 7400 1950 60  0000 C CNN
 	1    7400 1950

Commit message: dalsi
Parts:
- removed J5: VREF/TRANSISTOR, Mlab_Pin_Headers:Straight_2x05, symbol HEADER_2x05_PARALLEL
- added J5: SOT23-6, Mlab_Pin_Headers:Straight_2x08, symbol HEADER_2x08_PARALLEL
- added Q1: BC846, SOT-23-3, symbol BC849
- added U3: ANALOG SWITCH, Mlab_IO:SOT-23-6, symbol TS5A3159
- U2: footprint sot23-6:SOT-23-6 -> SOT-23-3
Connections:
- net GNDA: now also J5.1, J5.2
- net VCC: now also J5.15, J5.16
- net T1 renamed 1
- net 1: now also J5.13, J5.14, U3.1 (NO); no longer d3.2
- net T3 renamed 5
- net 5: now also J5.5, J5.6, U3.5 (V+); no longer d6.1
- net VREF/T2 renamed 3
- net 3: now also J5.10, J5.9, U3.3 (NC)
- new net 2: J5.11, J5.12, Q1.3 (C), U3.2 (GND), d3.2
- new net 4: J5.7, J5.8, Q1.1 (B), U3.4 (COM)
- new net 6: J5.3, J5.4, Q1.2 (E), U3.6 (IN), d6.1
Other:
- note added: "REFERENCE, TRANSISTOR, SWITCH, ... in SOT23-3,5,6"
- note removed: "REFERENCE/TRANSISTOR"
- moved on the sheet: U1A, U1B, U2, a0, a1, a2, a3, a4, a6, a7, a8, a9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
