File: Universal/RJ12V01A/SCH_PCB/RJ12V01A.sch (KiCad schematic (older format))
At the start: 22 parts, among them J1 JUMP_2x1, J10 JUMP2_2x1, J11 JUMP2_2x1, J12 JUMP2_2x1, J13 JUMP2_2x1, J2 JUMP_2x1, J3 JUMP_2x1, J4 JUMP_2x1, J5 JUMP_2x1, J6 JUMP_2X2, J7 JUMP2_2x1, J8 RJ12GLP-AMP, J9 RJ12GLP-AMP, M1 HOLE, M2 HOLE, M3 HOLE, M4 HOLE

Commit message: Vyrobni data
Parts:
- added J14: JUMP_4X2, Mlab_Pin_Headers:Straight_2x04, symbol JUMP_4X2
Connections:
- wire segments 54 -> 59
Changed lines of the file:
@@
 Text Label 2650 6900 0    60   ~ 0
 5
+$Comp
+L JUMP_4X2 J14
+U 1 1 586A30B1
+P 9150 3750
+F 0 "J14" H 9079 3768 50  0000 L CNN
+F 1 "JUMP_4X2" H 9079 3684 40  0000 L CNN
+F 2 "Mlab_Pin_Headers:Straight_2x04" H 9150 3750 60  0001 C CNN
+F 3 "" H 9150 3750 60  0000 C CNN
+	1    9150 3750
+	1    0    0    -1
+$EndComp
+$Comp
+L GND #PWR09
+U 1 1 586A37F0
+P 8600 3950
+F 0 "#PWR09" H 8600 3700 60  0001 C CNN
+F 1 "GND" H 8600 3800 60  0000 C CNN
+F 2 "" H 8600 3950 60  0000 C CNN
+F 3 "" H 8600 3950 60  0000 C CNN
+	1    8600 3950
+	1    0    0    -1
+$EndComp
+Wire Wire Line
+	8750 3600 8600 3600
+Wire Wire Line
+	8600 3600 8600 3950
+Wire Wire Line
+	8750 3900 8600 3900
+Connection ~ 8600 3900
+Wire Wire Line
+	8750 3800 8600 3800
+Connection ~ 8600 3800
+Wire Wire Line
+	8750 3700 8600 3700
+Connection ~ 8600 3700
 $EndSCHEMATC
