File: PowerSupply/UNIPOWER04A/SCH_PCB/UNIPOWER04A.sch (KiCad schematic (older format))
At the start: 82 parts, among them CON1 JACK_DC2.1, J1 CONN1_1, J11 JUMP_4X2, J12 CONN1_1, J13 CONN1_1, J2 JUMP_4X2, J3 JUMP_4X2, J4 JUMP_4X2, J5 JUMP_4X2, J6 JUMP_4X2, J7 JUMP_4X2, J8 JUMP_4X2, J9 JUMP_4X2, P1 _, P2 _, P3 _, P4 _

Commit message: Edit schema
Connections:
- net GND: no longer P1.1 (P1), P2.1 (P1), P3.1 (P1), P4.1 (P1)
Changed lines of the file:
@@
 EESchema Schematic File Version 2
+LIBS:MLAB_SW
 LIBS:power
 LIBS:device
@@
 LIBS:contrib
 LIBS:valves
-LIBS:header
 LIBS:mechanical
+LIBS:MLAB_BATERY
+LIBS:MLAB_CONNECTORS
+LIBS:MLAB_D
+LIBS:MLAB_IO
+LIBS:MLAB_Jumpers
+LIBS:MLAB_T
+LIBS:MLAB_U
 LIBS:UNIPOWER04A-cache
 EELAYER 26 0
@@
 $EndComp
 $Comp
-L GND #PWR04
-U 1 1 58812A5A
-P 3800 1050
-F 0 "#PWR04" H 3800 800 50  0001 C CNN
-F 1 "GND" H 3800 900 50  0000 C CNN
-F 2 "" H 3800 1050 50  0000 C CNN
-F 3 "" H 3800 1050 50  0000 C CNN
-	1    3800 1050
-	1    0    0    -1
-$EndComp
-Wire Wire Line
-	3850 750  3800 750
-Wire Wire Line
-	3800 750  3800 1050
-Wire Wire Line
-	3850 950  3800 950
-Connection ~ 3800 950
-$Comp
-L GND #PWR05
-U 1 1 588131E7
-P 4400 1050
-F 0 "#PWR05" H 4400 800 50  0001 C CNN
-F 1 "GND" H 4400 900 50  0000 C CNN
-F 2 "" H 4400 1050 50  0000 C CNN
-F 3 "" H 4400 1050 50  0000 C CNN
-	1    4400 1050
-	1    0    0    -1
-$EndComp
-Wire Wire Line
-	4400 750  4400 1050
-Wire Wire Line
-	4400 750  4450 750
-Wire Wire Line
-	4450 950  4400 950
-Connection ~ 4400 950
-$Comp
 L JUMP_4X2 J3
