File: Sensors/SHT31V01A/SCH_PCB/SHT31V01A.kicad_pcb (KiCad board)
At the start: 2 copper layers, 40.1 x 9.7 mm, 18 parts, among them J1 CONN1_1, J10 JUMP_2x1, J11 JUMP_2x1, J12 JUMP_2x1, J13 JUMP_2x1, J2 CONN1_1, J9 JUMP_2x1, M1 HOLE, M2 HOLE, U1 SHT31

Commit message: data generation
Other:
- rule pad_to_mask_clearance: 0.12 -> 0.2
Changed lines of the file:
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@@
-(kicad_pcb (version 4) (host pcbnew 4.0.1-stable)
+(kicad_pcb (version 20170123) (host pcbnew "(2017-02-05 revision 431abcf)-makepkg")
   (general
     (links 32)
     (no_connects 0)
-    (area 117.475 79.297 164.005143 93.980001)
+    (area 117.475 79.4545 164.005143 93.980001)
     (thickness 1.6)
     (drawings 16)
@@
     (pad_size 1.524 1.524)
     (pad_drill 0.762)
-    (pad_to_mask_clearance 0.12)
+    (pad_to_mask_clearance 0.2)
+    (solder_mask_min_width 0.2)
     (aux_axis_origin 0 0)
     (visible_elements 7FFFFF7F)
     (pcbplotparams
-      (layerselection 0x010e0_80000001)
+      (layerselection 0x010e0_ffffffff)
       (usegerberextensions false)
       (excludeedgelayer true)
@@
       (hpglpenspeed 20)
       (hpglpendiameter 15)
-      (hpglpenoverlay 2)
       (psnegative false)
       (psa4output false)
@@
       (pts
         (xy 117.729 80.137) (xy 163.068 80.137) (xy 163.068 93.98) (xy 117.475 93.98) (xy 117.475 80.137)
-        (xy 117.729 80.137)
       )
     )
