File: PowerSW/DIG4SW01A/SCH_PCB/DIG4SW01A.sch (KiCad schematic (older format))
At the start: 24 parts, among them J1 CONN1_1, J2 CONN1_1, M1 HOLE, M2 HOLE, M3 HOLE, M4 HOLE

Commit message: Edit
Parts:
- added D2, D3, D4, D5: SMBJ15A-E3/52, Mlab_D:SMB_Standard, symbol D_ZENER
- added J10, J11, J12, J13, J4, J5, J6, J7, J8, J9: JUMP_2x1, Mlab_Pin_Headers:Straight_2x01, symbol JUMP_2x1
- added J14, J15, J16, J17, J3: JUMP_4X2, Mlab_Pin_Headers:Straight_2x04, symbol JUMP_4X2
- added R13: -, Mlab_R:SMD-0805, symbol R
- added R14, R15, R16, R17: 20k, Mlab_R:SMD-0805, symbol R
- R1, R10, R11, R2, R3, R4, R5, R6, R7, R8, R9: renamed from R?; footprint (none) -> Mlab_R:SMD-0805
- R12: renamed from R?; value 800R -> 820R; footprint (none) -> Mlab_R:SMD-0805
- gave numbers to parts that had none: 2
Connections:
- net GND: now also C4.2, R12.1, R3.1, D2.2 (A), D3.2 (A), D4.2 (A), D5.2 (A), J14.1 (2), J14.2, J14.7 (8), J14.8, J15.1 (2), J15.2, J15.7 (8), J15.8, J16.1 (2), J16.2, J16.7 (8), J16.8, J17.1 (2), J17.2, J17.7 (8), J17.8, J3.1 (2), J3.2, J3.7 (8), J3.8, R13.1
- net VCC: now also R11.2, U1.20 (VS), U1.21 (VS), U1.22 (VS), U1.23 (VS), J3.3 (4), J3.4, J3.5, J3.6 (5), R14.2, R15.2, R16.2, R17.2
- net at U1.10 (CS): now also R1.1, R3.2
- net at U1.11 (CL): now also R12.2
- net at U1.13 (THER): now also J13.1, J13.2 (1), R13.2
- net at U1.14 (DIAG_EN): now also R10.1
- net at U1.15 (OUT4), U1.16 (OUT4): now also D5.1 (K), J17.3 (4), J17.4, J17.5, J17.6 (5), R17.1
- net at U1.17 (OUT3), U1.18 (OUT3): now also D4.1 (K), J16.3 (4), J16.4, J16.5, J16.6 (5), R16.1
- net at U1.25 (OUT2), U1.26 (OUT2): now also D2.1 (K), D3.1 (K), J15.3 (4), J15.4, J15.5, J15.6 (5), R15.1
- net at U1.27 (OUT1), U1.28 (OUT1): now also J14.3 (4), J14.4, J14.5, J14.6 (5), R14.1
- net at U1.3 (IN1): now also R4.1
- net at U1.4 (IN2): now also R5.1
- net at U1.5 (IN3): now also R6.1
- net at U1.6 (IN4): now also R7.1
- net at U1.7 (SEH): now also R8.1
- net at U1.8 (SEL): now also R9.1
- net at U1.9 (FAULT): now also R11.1, R2.1
- net at R4.2: now also J6.1, J6.2 (1)
- net at R5.2: now also J7.1, J7.2 (1)
- net at R6.2: now also J8.1, J8.2 (1)
- net at R7.2: now also J9.1, J9.2 (1)
- net at R8.2: now also J10.1, J10.2 (1)
- net at R9.2: now also J11.1, J11.2 (1)
- net at R10.2: now also J12.1, J12.2 (1)
- net at R2.2: now also J4.1, J4.2 (1)
- net at R1.2: now also C4.1, J5.1, J5.2 (1)
Other:
- moved on the sheet: R12

Commit message: Edit
Parts:
- removed C2: 100nF/50V, Mlab_R:SMD-0805, symbol C
- removed J3: JUMP_4X2, Mlab_Pin_Headers:Straight_2x04, symbol JUMP_4X2
- added J3: CONN1_2, Mlab_Pin_Headers:Straight_1x02, symbol CONN1_2
- U1: footprint (none) -> Mlab_IO:HTSSOP28
Connections:
- net GND: now also J3.2 (PM)
- net VCC: now also J3.1 (P1)
- net THER: now reaches J13.1, J13.2 (1), R13.2, U1.13 (THER)
- net OUT4: now reaches D5.1 (K), J17.3 (4), J17.4, J17.5, J17.6 (5), R17.1, U1.15 (OUT4), U1.16 (OUT4)
- net OUT3: now reaches D4.1 (K), J16.3 (4), J16.4, J16.5, J16.6 (5), R16.1, U1.17 (OUT3), U1.18 (OUT3)
- net OUT2: now reaches D3.1 (K), J15.3 (4), J15.4, J15.5, J15.6 (5), R15.1, U1.25 (OUT2), U1.26 (OUT2)
- net OUT2: no longer D2.1 (K)
- net OUT1: now reaches J14.3 (4), J14.4, J14.5, J14.6 (5), R14.1, U1.27 (OUT1), U1.28 (OUT1)
- net OUT1: now also D2.1 (K)
- net IN1: now reaches J6.1, J6.2 (1), R4.2
- net IN2: now reaches J7.1, J7.2 (1), R5.2
- net IN3: now reaches J8.1, J8.2 (1), R6.2
- net IN4: now reaches J9.1, J9.2 (1), R7.2
- net SEH: now reaches J10.1, J10.2 (1), R8.2
- net SEL: now reaches J11.1, J11.2 (1), R9.2
- net DIAG_EN: now reaches J12.1, J12.2 (1), R10.2
- net #FAULT: now reaches J4.1, J4.2 (1), R2.2
- net CS: now reaches C4.1, J5.1, J5.2 (1), R1.2
Other:
- moved on the sheet: J10, J11, J12, J6, J7, J8, J9

Commit message: Edit
Parts:
- removed C1: 47uF/63V, Capacitors_ThroughHole:C_Radial_D6.3_L11.2_P2.5, symbol CP
- added J18: JUMP_2x1, Mlab_Pin_Headers:Straight_2x01, symbol JUMP_2x1
Connections:
- net GND: now also J18.1, J18.2 (1)
Other:
- moved on the sheet: C3, D1
Changed lines of the file:
@@
 L D_Schottky D1
 U 1 1 58246F3B
-P 2250 1000
-F 0 "D1" V 2204 1079 50  0000 L CNN
-F 1 "STPS340U" V 2295 1079 50  0000 L CNN
-F 2 "Mlab_D:Diode-SMB_Standard" H 2250 1000 50  0001 C CNN
-F 3 "" H 2250 1000 50  0000 C CNN
-	1    2250 1000
+P 700 1000
+F 0 "D1" V 654 1079 50  0000 L CNN
+F 1 "STPS340U" V 745 1079 50  0000 L CNN
+F 2 "Mlab_D:Diode-SMB_Standard" H 700 1000 50  0001 C CNN
+F 3 "" H 700 1000 50  0000 C CNN
+	1    700  1000
 	0    1    1    0
 $EndComp
@@
 L VCC #PWR02
 U 1 1 5824706E
-P 2250 750
-F 0 "#PWR02" H 2250 600 50  0001 C CNN
-F 1 "VCC" H 2267 923 50  0000 C CNN
-F 2 "" H 2250 750 50  0000 C CNN
-F 3 "" H 2250 750 50  0000 C CNN
-	1    2250 750
+P 700 750
+F 0 "#PWR02" H 700 600 50  0001 C CNN
+F 1 "VCC" H 717 923 50  0000 C CNN
+F 2 "" H 700 750 50  0000 C CNN
+F 3 "" H 700 750 50  0000 C CNN
+	1    700  750
 	1    0    0    -1
 $EndComp
@@
 L GND #PWR03
 U 1 1 582470A0
-P 2250 1250
-F 0 "#PWR03" H 2250 1000 50  0001 C CNN
-F 1 "GND" H 2255 1077 50  0000 C CNN
-F 2 "" H 2250 1250 50  0000 C CNN
-F 3 "" H 2250 1250 50  0000 C CNN
-	1    2250 1250
-	1    0    0    -1
-$EndComp
-Wire Wire Line
-	2250 1250 2250 1150
-Wire Wire Line
-	2250 850  2250 750
+P 700 1250
+F 0 "#PWR03" H 700 1000 50  0001 C CNN
+F 1 "GND" H 705 1077 50  0000 C CNN
+F 2 "" H 700 1250 50  0000 C CNN
+F 3 "" H 700 1250 50  0000 C CNN
+	1    700  1250
+	1    0    0    -1
+$EndComp
+Wire Wire Line
+	700  1250 700  1150
+Wire Wire Line
+	700  850  700  750
 $Comp
 L CONN1_1 J1
@@
 L CP C3
 U 1 1 5824A2B3
-P 2900 1000
-F 0 "C3" H 3018 1046 50  0000 L CNN
-F 1 "47uF/16V" H 3018 955 50  0000 L CNN
-F 2 "Mlab_C:TantalC_SizeC_Reflow" H 2938 850 50  0001 C CNN
-F 3 "" H 2900 1000 50  0000 C CNN
-	1    2900 1000
+P 1350 1000
+F 0 "C3" H 1468 1046 50  0000 L CNN
+F 1 "47uF/16V" H 1468 955 50  0000 L CNN
+F 2 "Mlab_C:TantalC_SizeC_Reflow" H 1388 850 50  0001 C CNN
+F 3 "" H 1350 1000 50  0000 C CNN
+	1    1350 1000
 	1    0    0    -1
 $EndComp
@@
 L GND #PWR07
 U 1 1 5824A2B9
-P 2900 1250
-F 0 "#PWR07" H 2900 1000 50  0001 C CNN
-F 1 "GND" H 2905 1077 50  0000 C CNN
-F 2 "" H 2900 1250 50  0000 C CNN
-F 3 "" H 2900 1250 50  0000 C CNN
-	1    2900 1250
-	1    0    0    -1
-$EndComp
-Wire Wire Line
-	2900 1250 2900 1150
-Wire Wire Line
-	2900 850  2900 750
+P 1350 1250
+F 0 "#PWR07" H 1350 1000 50  0001 C CNN
+F 1 "GND" H 1355 1077 50  0000 C CNN
+F 2 "" H 1350 1250 50  0000 C CNN
+F 3 "" H 1350 1250 50  0000 C CNN
+	1    1350 1250
+	1    0    0    -1
+$EndComp
+Wire Wire Line
+	1350 1250 1350 1150
+Wire Wire Line
+	1350 850  1350 750
 $Comp
 L TPS4H160-Q1-B U1
@@
 	0    1    1    0
 $EndComp
-Wire Wire Line
-	750  850  750  750
-Wire Wire Line
-	750  1250 750  1150
-$Comp
-L GND #PWR014
-U 1 1 58245AC9
-P 750 1250
-F 0 "#PWR014" H 750 1000 50  0001 C CNN
-F 1 "GND" H 755 1077 50  0000 C CNN
-F 2 "" H 750 1250 50  0000 C CNN
-F 3 "" H 750 1250 50  0000 C CNN
-	1    750  1250
-	1    0    0    -1
-$EndComp
-$Comp
-L CP C1
-U 1 1 582452D7
-P 750 1000
-F 0 "C1" H 868 1046 50  0000 L CNN
-F 1 "47uF/63V" H 868 955 50  0000 L CNN
-F 2 "Capacitors_ThroughHole:C_Radial_D6.3_L11.2_P2.5" H 788 850 50  0001 C CNN
-F 3 "" H 750 1000 50  0000 C CNN
-	1    750  1000
-	1    0    0    -1
-$EndComp
-$Comp
-L VCC #PWR015
-U 1 1 58245252
-P 750 750
-F 0 "#PWR015" H 750 600 50  0001 C CNN
-F 1 "VCC" H 767 923 50  0000 C CNN
-F 2 "" H 750 750 50  0000 C CNN
-F 3 "" H 750 750 50  0000 C CNN
-	1    750  750
-	1    0    0    -1
-$EndComp
 $Comp
 L R R14
@@
 	5600 6150 5600 6100
 $Comp
-L GND #PWR016
+L GND #PWR014
 U 1 1 591715B5
 P 6800 3700
-F 0 "#PWR016" H 6800 3450 50  0001 C CNN
+F 0 "#PWR014" H 6800 3450 50  0001 C CNN
 F 1 "GND" H 6805 3527 50  0000 C CNN
 F 2 "" H 6800 3700 50  0000 C CNN
@@
 $EndComp
 $Comp
-L GND #PWR017
+L GND #PWR015
 U 1 1 591720D6
 P 7100 3700
-F 0 "#PWR017" H 7100 3450 50  0001 C CNN
+F 0 "#PWR015" H 7100 3450 50  0001 C CNN
 F 1 "GND" H 7105 3527 50  0000 C CNN
 F 2 "" H 7100 3700 50  0000 C CNN
@@
 $EndComp
 $Comp
-L GND #PWR018
+L GND #PWR016
 U 1 1 59172162
 P 7400 3700
-F 0 "#PWR018" H 7400 3450 50  0001 C CNN
+F 0 "#PWR016" H 7400 3450 50  0001 C CNN
 F 1 "GND" H 7405 3527 50  0000 C CNN
 F 2 "" H 7400 3700 50  0000 C CNN
@@
 $EndComp
 $Comp
-L GND #PWR019
+L GND #PWR017
 U 1 1 591721EE
 P 7700 3700
-F 0 "#PWR019" H 7700 3450 50  0001 C CNN
+F 0 "#PWR017" H 7700 3450 50  0001 C CNN
 F 1 "GND" H 7705 3527 50  0000 C CNN
 F 2 "" H 7700 3700 50  0000 C CNN
@@
 $EndComp
 $Comp
-L GND #PWR020
+L GND #PWR018
 U 1 1 59177536
 P 8400 1900
-F 0 "#PWR020" H 8400 1650 50  0001 C CNN
+F 0 "#PWR018" H 8400 1650 50  0001 C CNN
 F 1 "GND" H 8405 1727 50  0000 C CNN
 F 2 "" H 8400 1900 50  0000 C CNN
@@
 $EndComp
 $Comp
-L GND #PWR021
+L GND #PWR019
 U 1 1 59178F40
 P 8400 2550
-F 0 "#PWR021" H 8400 2300 50  0001 C CNN
+F 0 "#PWR019" H 8400 2300 50  0001 C CNN
 F 1 "GND" H 8405 2377 50  0000 C CNN
 F 2 "" H 8400 2550 50  0000 C CNN
@@
 $EndComp
 $Comp
-L GND #PWR022
+L GND #PWR020
 U 1 1 59179307
 P 8400 3200
-F 0 "#PWR022" H 8400 2950 50  0001 C CNN
+F 0 "#PWR020" H 8400 2950 50  0001 C CNN
 F 1 "GND" H 8405 3027 50  0000 C CNN
 F 2 "" H 8400 3200 50  0000 C CNN
@@
 $EndComp
 $Comp
-L GND #PWR023
+L GND #PWR021
 U 1 1 5917931A
 P 8400 3850
-F 0 "#PWR023" H 8400 3600 50  0001 C CNN
+F 0 "#PWR021" H 8400 3600 50  0001 C CNN
 F 1 "GND" H 8405 3677 50  0000 C CNN
 F 2 "" H 8400 3850 50  0000 C CNN
@@
 Connection ~ 8450 3650
 $Comp
-L GND #PWR024
+L GND #PWR022
 U 1 1 5917F494
 P 1400 2200
-F 0 "#PWR024" H 1400 1950 50  0001 C CNN
+F 0 "#PWR022" H 1400 1950 50  0001 C CNN
 F 1 "GND" H 1405 2027 50  0000 C CNN
 F 2 "" H 1400 2200 50  0000 C CNN
@@
 $EndComp
 $Comp
-L VCC #PWR025
+L VCC #PWR023
 U 1 1 5917F743
 P 1400 1900
-F 0 "#PWR025" H 1400 1750 50  0001 C CNN
+F 0 "#PWR023" H 1400 1750 50  0001 C CNN
 F 1 "VCC" H 1417 2073 50  0000 C CNN
 F 2 "" H 1400 1900 50  0000 C CNN
@@
 	1400 2050 1400 1900
 $Comp
-L VCC #PWR026
+L VCC #PWR024
 U 1 1 5918067E
-P 2900 750
-F 0 "#PWR026" H 2900 600 50  0001 C CNN
-F 1 "VCC" H 2917 923 50  0000 C CNN
-F 2 "" H 2900 750 50  0000 C CNN
-F 3 "" H 2900 750 50  0000 C CNN
-	1    2900 750
+P 1350 750
+F 0 "#PWR024" H 1350 600 50  0001 C CNN
+F 1 "VCC" H 1367 923 50  0000 C CNN
+F 2 "" H 1350 750 50  0000 C CNN
+F 3 "" H 1350 750 50  0000 C CNN
+	1    1350 750
 	1    0    0    -1
 $EndComp
@@
 Wire Wire Line
 	1400 2050 1600 2050
+$Comp
+L JUMP_2x1 J18
+U 1 1 591AD2D9
+P 4100 3850
+F 0 "J18" H 4106 3954 50  0000 C CNN
+F 1 "JUMP_2x1" V 1050 1100 40  0001 C CNN
+F 2 "Mlab_Pin_Headers:Straight_2x01" H 1100 1100 60  0001 C CNN
+F 3 "" H 1100 1100 60  0000 C CNN
+	1    4100 3850
+	1    0    0    -1
+$EndComp
+$Comp
+L GND #PWR025
+U 1 1 591AD674
+P 4300 3950
+F 0 "#PWR025" H 4300 3700 50  0001 C CNN
+F 1 "GND" H 4305 3777 50  0000 C CNN
+F 2 "" H 4300 3950 50  0000 C CNN
+F 3 "" H 4300 3950 50  0000 C CNN
+	1    4300 3950
+	1    0    0    -1
+$EndComp
+Wire Wire Line
+	4250 3850 4300 3850
+Wire Wire Line
+	4300 3850 4300 3950
 $EndSCHEMATC
