File: PowerSW/DIG4SWHI01A/SCH_PCB/DIG4SWHI01A.sch (KiCad schematic (older format))
At the start: 21 parts, among them J1 CONN1_1, J10 JUMP_2x1, J2 CONN1_1, J3 JUMP_2x1, J4 JUMP_2x1, J5 JUMP_2x1, J6 CONN1_1, J7 CONN1_1, J9 JUMP_2x1, M1 HOLE, M2 HOLE, M3 HOLE, M4 HOLE, U1 DRV8871

Commit message: Edit module
Parts:
- removed C1: 47uF/63V, Capacitors_ThroughHole:C_Radial_D6.3_L11.2_P2.5, symbol CP
- removed J6, J7: CONN1_1, Mlab_CON:WAGO256, symbol CONN1_1
- removed U1: DRV8871, Mlab_IO:HSOP-8, symbol DRV8871
- added C3: 100pF, Mlab_R:SMD-0805, symbol C
- added C4, C5, C6, C7: 10nF, Mlab_R:SMD-0805, symbol C
- added D2, D3, D4, D5: SMBJ15A-E3/52, Mlab_D:SMB_Standard, symbol D_ZENER
- added J11, J6, J7, J8: JUMP_2x1, Mlab_Pin_Headers:Straight_2x01, symbol JUMP_2x1
- added J12, J13, J14, J15, J16, J17, J18, J19: CONN1_1, Mlab_CON:WAGO256, symbol CONN1_1
- added R10, R4, R5, R6, R7, R8, R9: 10k, Mlab_R:SMD-0805, symbol R
- added R11, R12, R13, R14: 20k, Mlab_R:SMD-0805, symbol R
- added U1: VNQ7050AJ, Mlab_IO:PowerSSO-16, symbol VNQ7050AJ
- C2: value 100nF/50V -> 100nF
- R1: value 33k -> 10k
- R2: value 10k -> 510
- renumbered C3 to C1
Connections:
- net labels added: #FRST, CS, IN0, IN3, OUT0, OUT3, SEL0, SEL1, SEn
- wire segments 38 -> 73
Other:
- moved on the sheet: C1, D1

Commit message: Edit
Parts:
- D1: value STPS340U -> SMBJ15A-E3/52
Changed lines of the file:
@@
 $EndComp
 $Comp
-L GND #PWR22
+L GND #PWR01
 U 1 1 549D770F
 P 10950 850
-F 0 "#PWR22" H 10950 600 60  0001 C CNN
+F 0 "#PWR01" H 10950 600 60  0001 C CNN
 F 1 "GND" H 10950 700 60  0000 C CNN
 F 2 "" H 10950 850 60  0000 C CNN
@@
 P 700 1000
 F 0 "D1" V 654 1079 50  0000 L CNN
-F 1 "STPS340U" V 745 1079 50  0000 L CNN
+F 1 "SMBJ15A-E3/52" H 750 1200 50  0000 L CNN
 F 2 "Mlab_D:Diode-SMB_Standard" H 700 1000 50  0001 C CNN
 F 3 "" H 700 1000 50  0000 C CNN
@@
 $EndComp
 $Comp
-L VCC #PWR1
+L VCC #PWR02
 U 1 1 5824706E
 P 700 750
-F 0 "#PWR1" H 700 600 50  0001 C CNN
+F 0 "#PWR02" H 700 600 50  0001 C CNN
 F 1 "VCC" H 717 923 50  0000 C CNN
 F 2 "" H 700 750 50  0000 C CNN
@@
 $EndComp
 $Comp
-L GND #PWR2
+L GND #PWR03
 U 1 1 582470A0
 P 700 1250
-F 0 "#PWR2" H 700 1000 50  0001 C CNN
+F 0 "#PWR03" H 700 1000 50  0001 C CNN
 F 1 "GND" H 705 1077 50  0000 C CNN
 F 2 "" H 700 1250 50  0000 C CNN
@@
 $EndComp
 $Comp
-L GND #PWR4
+L GND #PWR04
 U 1 1 58248A9A
 P 750 2200
-F 0 "#PWR4" H 750 1950 50  0001 C CNN
+F 0 "#PWR04" H 750 1950 50  0001 C CNN
 F 1 "GND" H 755 2027 50  0000 C CNN
 F 2 "" H 750 2200 50  0000 C CNN
@@
 $EndComp
 $Comp
-L VCC #PWR3
+L VCC #PWR05
 U 1 1 58248F95
 P 750 1950
-F 0 "#PWR3" H 750 1800 50  0001 C CNN
+F 0 "#PWR05" H 750 1800 50  0001 C CNN
 F 1 "VCC" H 767 2123 50  0000 C CNN
 F 2 "" H 750 1950 50  0000 C CNN
@@
 	750  2150 800  2150
 $Comp
-L VCC #PWR12
+L VCC #PWR06
 U 1 1 5824A2AD
 P 4400 1950
-F 0 "#PWR12" H 4400 1800 50  0001 C CNN
+F 0 "#PWR06" H 4400 1800 50  0001 C CNN
 F 1 "VCC" H 4417 2123 50  0000 C CNN
 F 2 "" H 4400 1950 50  0000 C CNN
@@
 $EndComp
 $Comp
-L GND #PWR6
+L GND #PWR07
 U 1 1 5824A2B9
 P 1350 1250
-F 0 "#PWR6" H 1350 1000 50  0001 C CNN
+F 0 "#PWR07" H 1350 1000 50  0001 C CNN
 F 1 "GND" H 1355 1077 50  0000 C CNN
 F 2 "" H 1350 1250 50  0000 C CNN
@@
 	1350 850  1350 750
 $Comp
-L GND #PWR11
+L GND #PWR08
 U 1 1 591462E1
 P 4350 4800
-F 0 "#PWR11" H 4350 4550 50  0001 C CNN
+F 0 "#PWR08" H 4350 4550 50  0001 C CNN
 F 1 "GND" H 4355 4627 50  0000 C CNN
 F 2 "" H 4350 4800 50  0000 C CNN
@@
 $EndComp
 $Comp
-L GND #PWR10
+L GND #PWR09
 U 1 1 591578E5
 P 3600 4800
-F 0 "#PWR10" H 3600 4550 50  0001 C CNN
+F 0 "#PWR09" H 3600 4550 50  0001 C CNN
 F 1 "GND" H 3605 4627 50  0000 C CNN
 F 2 "" H 3600 4800 50  0000 C CNN
@@
 $EndComp
 $Comp
-L GND #PWR9
+L GND #PWR010
 U 1 1 59157ACB
 P 3100 4800
-F 0 "#PWR9" H 3100 4550 50  0001 C CNN
+F 0 "#PWR010" H 3100 4550 50  0001 C CNN
 F 1 "GND" H 3105 4627 50  0000 C CNN
 F 2 "" H 3100 4800 50  0000 C CNN
@@
 Connection ~ 6050 2050
 $Comp
-L GND #PWR13
+L GND #PWR011
 U 1 1 591715B5
 P 5500 3950
-F 0 "#PWR13" H 5500 3700 50  0001 C CNN
+F 0 "#PWR011" H 5500 3700 50  0001 C CNN
 F 1 "GND" H 5505 3777 50  0000 C CNN
 F 2 "" H 5500 3950 50  0000 C CNN
@@
 $EndComp
 $Comp
-L GND #PWR14
+L GND #PWR012
 U 1 1 591720D6
 P 5800 3950
-F 0 "#PWR14" H 5800 3700 50  0001 C CNN
+F 0 "#PWR012" H 5800 3700 50  0001 C CNN
 F 1 "GND" H 5805 3777 50  0000 C CNN
 F 2 "" H 5800 3950 50  0000 C CNN
@@
 $EndComp
 $Comp
-L GND #PWR15
+L GND #PWR013
 U 1 1 59172162
 P 6100 3950
-F 0 "#PWR15" H 6100 3700 50  0001 C CNN
+F 0 "#PWR013" H 6100 3700 50  0001 C CNN
 F 1 "GND" H 6105 3777 50  0000 C CNN
 F 2 "" H 6100 3950 50  0000 C CNN
@@
 $EndComp
 $Comp
-L GND #PWR16
+L GND #PWR014
 U 1 1 591721EE
 P 6400 3950
-F 0 "#PWR16" H 6400 3700 50  0001 C CNN
+F 0 "#PWR014" H 6400 3700 50  0001 C CNN
 F 1 "GND" H 6405 3777 50  0000 C CNN
 F 2 "" H 6400 3950 50  0000 C CNN
@@
 Connection ~ 6400 3150
 $Comp
-L VCC #PWR5
+L VCC #PWR015
 U 1 1 5918067E
 P 1350 750
-F 0 "#PWR5" H 1350 600 50  0001 C CNN
+F 0 "#PWR015" H 1350 600 50  0001 C CNN
 F 1 "VCC" H 1367 923 50  0000 C CNN
 F 2 "" H 1350 750 50  0000 C CNN
@@
 $EndComp
 $Comp
-L VCC #PWR7
+L VCC #PWR016
 U 1 1 592A2546
 P 2050 750
-F 0 "#PWR7" H 2050 600 50  0001 C CNN
+F 0 "#PWR016" H 2050 600 50  0001 C CNN
 F 1 "VCC" H 2067 923 50  0000 C CNN
 F 2 "" H 2050 750 50  0000 C CNN
@@
 $EndComp
 $Comp
-L GND #PWR8
+L GND #PWR017
 U 1 1 592A25DB
 P 2050 1250
-F 0 "#PWR8" H 2050 1000 50  0001 C CNN
+F 0 "#PWR017" H 2050 1000 50  0001 C CNN
 F 1 "GND" H 2055 1077 50  0000 C CNN
 F 2 "" H 2050 1250 50  0000 C CNN
@@
 $EndComp
 $Comp
-L GND #PWR17
+L GND #PWR018
 U 1 1 592A8675
 P 6850 3950
-F 0 "#PWR17" H 6850 3700 50  0001 C CNN
+F 0 "#PWR018" H 6850 3700 50  0001 C CNN
 F 1 "GND" H 6855 3777 50  0000 C CNN
 F 2 "" H 6850 3950 50  0000 C CNN
@@
 $EndComp
 $Comp
-L GND #PWR18
+L GND #PWR019
 U 1 1 592A8D34
 P 7300 3950
-F 0 "#PWR18" H 7300 3700 50  0001 C CNN
+F 0 "#PWR019" H 7300 3700 50  0001 C CNN
 F 1 "GND" H 7305 3777 50  0000 C CNN
 F 2 "" H 7300 3950 50  0000 C CNN
@@
 $EndComp
 $Comp
-L GND #PWR19
+L GND #PWR020
 U 1 1 592A9057
 P 7750 3950
-F 0 "#PWR19" H 7750 3700 50  0001 C CNN
+F 0 "#PWR020" H 7750 3700 50  0001 C CNN
 F 1 "GND" H 7755 3777 50  0000 C CNN
 F 2 "" H 7750 3950 50  0000 C CNN
@@
 $EndComp
 $Comp
-L GND #PWR20
+L GND #PWR021
 U 1 1 592A90E6
 P 8200 3950
-F 0 "#PWR20" H 8200 3700 50  0001 C CNN
+F 0 "#PWR021" H 8200 3700 50  0001 C CNN
 F 1 "GND" H 8205 3777 50  0000 C CNN
 F 2 "" H 8200 3950 50  0000 C CNN
@@
 $EndComp
 $Comp
-L GND #PWR21
+L GND #PWR022
 U 1 1 592B4758
 P 8900 3700
-F 0 "#PWR21" H 8900 3450 50  0001 C CNN
+F 0 "#PWR022" H 8900 3450 50  0001 C CNN
 F 1 "GND" H 8905 3527 50  0000 C CNN
 F 2 "" H 8900 3700 50  0000 C CNN

Commit message: Edit PCB
Parts:
- added J20: JUMP_2x1, Mlab_Pin_Headers:Straight_2x01, symbol JUMP_2x1
Connections:
- net GND: now also J20.1, J20.2 (1)
Changed lines of the file:
@@
 $EndComp
 $Comp
-L GND #PWR01
+L GND #PWR23
 U 1 1 549D770F
 P 10950 850
-F 0 "#PWR01" H 10950 600 60  0001 C CNN
+F 0 "#PWR23" H 10950 600 60  0001 C CNN
 F 1 "GND" H 10950 700 60  0000 C CNN
 F 2 "" H 10950 850 60  0000 C CNN
@@
 $EndComp
 $Comp
-L VCC #PWR02
+L VCC #PWR1
 U 1 1 5824706E
 P 700 750
-F 0 "#PWR02" H 700 600 50  0001 C CNN
+F 0 "#PWR1" H 700 600 50  0001 C CNN
 F 1 "VCC" H 717 923 50  0000 C CNN
 F 2 "" H 700 750 50  0000 C CNN
@@
 $EndComp
 $Comp
-L GND #PWR03
+L GND #PWR2
 U 1 1 582470A0
 P 700 1250
-F 0 "#PWR03" H 700 1000 50  0001 C CNN
+F 0 "#PWR2" H 700 1000 50  0001 C CNN
 F 1 "GND" H 705 1077 50  0000 C CNN
 F 2 "" H 700 1250 50  0000 C CNN
@@
 $EndComp
 $Comp
-L GND #PWR04
+L GND #PWR4
 U 1 1 58248A9A
 P 750 2200
-F 0 "#PWR04" H 750 1950 50  0001 C CNN
+F 0 "#PWR4" H 750 1950 50  0001 C CNN
 F 1 "GND" H 755 2027 50  0000 C CNN
 F 2 "" H 750 2200 50  0000 C CNN
@@
 $EndComp
 $Comp
-L VCC #PWR05
+L VCC #PWR3
 U 1 1 58248F95
 P 750 1950
-F 0 "#PWR05" H 750 1800 50  0001 C CNN
+F 0 "#PWR3" H 750 1800 50  0001 C CNN
 F 1 "VCC" H 767 2123 50  0000 C CNN
 F 2 "" H 750 1950 50  0000 C CNN
@@
 	750  2150 800  2150
 $Comp
-L VCC #PWR06
+L VCC #PWR13
 U 1 1 5824A2AD
 P 4400 1950
-F 0 "#PWR06" H 4400 1800 50  0001 C CNN
+F 0 "#PWR13" H 4400 1800 50  0001 C CNN
 F 1 "VCC" H 4417 2123 50  0000 C CNN
 F 2 "" H 4400 1950 50  0000 C CNN
@@
 $EndComp
 $Comp
-L GND #PWR07
+L GND #PWR6
 U 1 1 5824A2B9
 P 1350 1250
-F 0 "#PWR07" H 1350 1000 50  0001 C CNN
+F 0 "#PWR6" H 1350 1000 50  0001 C CNN
 F 1 "GND" H 1355 1077 50  0000 C CNN
 F 2 "" H 1350 1250 50  0000 C CNN
@@
 	1350 850  1350 750
 $Comp
-L GND #PWR08
+L GND #PWR12
 U 1 1 591462E1
 P 4350 4800
-F 0 "#PWR08" H 4350 4550 50  0001 C CNN
+F 0 "#PWR12" H 4350 4550 50  0001 C CNN
 F 1 "GND" H 4355 4627 50  0000 C CNN
 F 2 "" H 4350 4800 50  0000 C CNN
@@
 $EndComp
 $Comp
-L GND #PWR09
+L GND #PWR11
 U 1 1 591578E5
 P 3600 4800
-F 0 "#PWR09" H 3600 4550 50  0001 C CNN
+F 0 "#PWR11" H 3600 4550 50  0001 C CNN
 F 1 "GND" H 3605 4627 50  0000 C CNN
 F 2 "" H 3600 4800 50  0000 C CNN
@@
 $EndComp
 $Comp
-L GND #PWR010
+L GND #PWR10
 U 1 1 59157ACB
 P 3100 4800
-F 0 "#PWR010" H 3100 4550 50  0001 C CNN
+F 0 "#PWR10" H 3100 4550 50  0001 C CNN
 F 1 "GND" H 3105 4627 50  0000 C CNN
 F 2 "" H 3100 4800 50  0000 C CNN
@@
 Connection ~ 6050 2050
 $Comp
-L GND #PWR011
+L GND #PWR14
 U 1 1 591715B5
 P 5500 3950
-F 0 "#PWR011" H 5500 3700 50  0001 C CNN
+F 0 "#PWR14" H 5500 3700 50  0001 C CNN
 F 1 "GND" H 5505 3777 50  0000 C CNN
 F 2 "" H 5500 3950 50  0000 C CNN
@@
 $EndComp
 $Comp
-L GND #PWR012
+L GND #PWR15
 U 1 1 591720D6
 P 5800 3950
-F 0 "#PWR012" H 5800 3700 50  0001 C CNN
+F 0 "#PWR15" H 5800 3700 50  0001 C CNN
 F 1 "GND" H 5805 3777 50  0000 C CNN
 F 2 "" H 5800 3950 50  0000 C CNN
@@
 $EndComp
 $Comp
-L GND #PWR013
+L GND #PWR16
 U 1 1 59172162
 P 6100 3950
-F 0 "#PWR013" H 6100 3700 50  0001 C CNN
+F 0 "#PWR16" H 6100 3700 50  0001 C CNN
 F 1 "GND" H 6105 3777 50  0000 C CNN
 F 2 "" H 6100 3950 50  0000 C CNN
@@
 $EndComp
 $Comp
-L GND #PWR014
+L GND #PWR17
 U 1 1 591721EE
 P 6400 3950
-F 0 "#PWR014" H 6400 3700 50  0001 C CNN
+F 0 "#PWR17" H 6400 3700 50  0001 C CNN
 F 1 "GND" H 6405 3777 50  0000 C CNN
 F 2 "" H 6400 3950 50  0000 C CNN
@@
 Connection ~ 6400 3150
 $Comp
-L VCC #PWR015
+L VCC #PWR5
 U 1 1 5918067E
 P 1350 750
-F 0 "#PWR015" H 1350 600 50  0001 C CNN
+F 0 "#PWR5" H 1350 600 50  0001 C CNN
 F 1 "VCC" H 1367 923 50  0000 C CNN
 F 2 "" H 1350 750 50  0000 C CNN
@@
 $EndComp
 $Comp
-L VCC #PWR016
+L VCC #PWR8
 U 1 1 592A2546
 P 2050 750
-F 0 "#PWR016" H 2050 600 50  0001 C CNN
+F 0 "#PWR8" H 2050 600 50  0001 C CNN
 F 1 "VCC" H 2067 923 50  0000 C CNN
 F 2 "" H 2050 750 50  0000 C CNN
@@
 $EndComp
 $Comp
-L GND #PWR017
+L GND #PWR9
 U 1 1 592A25DB
 P 2050 1250
-F 0 "#PWR017" H 2050 1000 50  0001 C CNN
+F 0 "#PWR9" H 2050 1000 50  0001 C CNN
 F 1 "GND" H 2055 1077 50  0000 C CNN
 F 2 "" H 2050 1250 50  0000 C CNN
@@
 $EndComp
 $Comp
-L GND #PWR018
+L GND #PWR18
 U 1 1 592A8675
 P 6850 3950
-F 0 "#PWR018" H 6850 3700 50  0001 C CNN
+F 0 "#PWR18" H 6850 3700 50  0001 C CNN
 F 1 "GND" H 6855 3777 50  0000 C CNN
 F 2 "" H 6850 3950 50  0000 C CNN
@@
 $EndComp
 $Comp
-L GND #PWR019
+L GND #PWR19
 U 1 1 592A8D34
 P 7300 3950
-F 0 "#PWR019" H 7300 3700 50  0001 C CNN
+F 0 "#PWR19" H 7300 3700 50  0001 C CNN
 F 1 "GND" H 7305 3777 50  0000 C CNN
 F 2 "" H 7300 3950 50  0000 C CNN
@@
 $EndComp
 $Comp
-L GND #PWR020
+L GND #PWR20
 U 1 1 592A9057
 P 7750 3950
-F 0 "#PWR020" H 7750 3700 50  0001 C CNN
+F 0 "#PWR20" H 7750 3700 50  0001 C CNN
 F 1 "GND" H 7755 3777 50  0000 C CNN
 F 2 "" H 7750 3950 50  0000 C CNN
@@
 $EndComp
 $Comp
-L GND #PWR021
+L GND #PWR21
 U 1 1 592A90E6
 P 8200 3950
-F 0 "#PWR021" H 8200 3700 50  0001 C CNN
+F 0 "#PWR21" H 8200 3700 50  0001 C CNN
 F 1 "GND" H 8205 3777 50  0000 C CNN
 F 2 "" H 8200 3950 50  0000 C CNN
@@
 $EndComp
 $Comp
-L GND #PWR022
+L GND #PWR22
 U 1 1 592B4758
 P 8900 3700
-F 0 "#PWR022" H 8900 3450 50  0001 C CNN
+F 0 "#PWR22" H 8900 3450 50  0001 C CNN
 F 1 "GND" H 8905 3527 50  0000 C CNN
 F 2 "" H 8900 3700 50  0000 C CNN
@@
 	9000 3450 8900 3450
 Connection ~ 8900 3450
+$Comp
+L JUMP_2x1 J20
+U 1 1 593026ED
+P 1650 1850
+F 0 "J20" H 1656 1954 50  0000 C CNN
+F 1 "JUMP_2x1" V -1400 -900 40  0001 C CNN
+F 2 "Mlab_Pin_Headers:Straight_2x01" H -1350 -900 60  0001 C CNN
+F 3 "" H -1350 -900 60  0000 C CNN
+	1    1650 1850
+	1    0    0    -1
+$EndComp
+$Comp
+L GND #PWR7
+U 1 1 59305CBE
+P 1900 1950
+F 0 "#PWR7" H 1900 1700 50  0001 C CNN
+F 1 "GND" H 1905 1777 50  0000 C CNN
+F 2 "" H 1900 1950 50  0000 C CNN
+F 3 "" H 1900 1950 50  0000 C CNN
+	1    1900 1950
+	1    0    0    -1
+$EndComp
+Wire Wire Line
+	1800 1850 1900 1850
+Wire Wire Line
+	1900 1850 1900 1950
 $EndSCHEMATC

Commit message: Production data
Parts:
- J1, J12, J13, J14, J15, J16, J17, J18, J19, J2: footprint Mlab_CON:WAGO256 -> Mlab_CON:WAGO256_2
Changed lines of the file:
@@
 $EndComp
 $Comp
-L GND #PWR23
+L GND #PWR01
 U 1 1 549D770F
 P 10950 850
-F 0 "#PWR23" H 10950 600 60  0001 C CNN
+F 0 "#PWR01" H 10950 600 60  0001 C CNN
 F 1 "GND" H 10950 700 60  0000 C CNN
 F 2 "" H 10950 850 60  0000 C CNN
@@
 $EndComp
 $Comp
-L VCC #PWR1
+L VCC #PWR02
 U 1 1 5824706E
 P 700 750
-F 0 "#PWR1" H 700 600 50  0001 C CNN
+F 0 "#PWR02" H 700 600 50  0001 C CNN
 F 1 "VCC" H 717 923 50  0000 C CNN
 F 2 "" H 700 750 50  0000 C CNN
@@
 $EndComp
 $Comp
-L GND #PWR2
+L GND #PWR03
 U 1 1 582470A0
 P 700 1250
-F 0 "#PWR2" H 700 1000 50  0001 C CNN
+F 0 "#PWR03" H 700 1000 50  0001 C CNN
 F 1 "GND" H 705 1077 50  0000 C CNN
 F 2 "" H 700 1250 50  0000 C CNN
@@
 F 0 "J1" H 1079 2080 50  0000 L CNN
 F 1 "CONN1_1" H 1200 2000 40  0001 C CNN
-F 2 "Mlab_CON:WAGO256" H 1150 2000 60  0001 C CNN
+F 2 "Mlab_CON:WAGO256_2" H 1150 2000 60  0001 C CNN
 F 3 "" H 1150 2000 60  0000 C CNN
 	1    1100 2050
@@
 F 0 "J2" H 1079 2230 50  0000 L CNN
 F 1 "CONN1_1" H 1200 2150 40  0001 C CNN
-F 2 "Mlab_CON:WAGO256" H 1150 2150 60  0001 C CNN
+F 2 "Mlab_CON:WAGO256_2" H 1150 2150 60  0001 C CNN
 F 3 "" H 1150 2150 60  0000 C CNN
 	1    1100 2200
@@
 $EndComp
 $Comp
-L GND #PWR4
+L GND #PWR04
 U 1 1 58248A9A
 P 750 2200
-F 0 "#PWR4" H 750 1950 50  0001 C CNN
+F 0 "#PWR04" H 750 1950 50  0001 C CNN
 F 1 "GND" H 755 2027 50  0000 C CNN
 F 2 "" H 750 2200 50  0000 C CNN
@@
 $EndComp
 $Comp
-L VCC #PWR3
+L VCC #PWR05
 U 1 1 58248F95
 P 750 1950
-F 0 "#PWR3" H 750 1800 50  0001 C CNN
+F 0 "#PWR05" H 750 1800 50  0001 C CNN
 F 1 "VCC" H 767 2123 50  0000 C CNN
 F 2 "" H 750 1950 50  0000 C CNN
@@
 	750  2150 800  2150
 $Comp
-L VCC #PWR13
+L VCC #PWR06
 U 1 1 5824A2AD
 P 4400 1950
-F 0 "#PWR13" H 4400 1800 50  0001 C CNN
+F 0 "#PWR06" H 4400 1800 50  0001 C CNN
 F 1 "VCC" H 4417 2123 50  0000 C CNN
 F 2 "" H 4400 1950 50  0000 C CNN
@@
 $EndComp
 $Comp
-L GND #PWR6
+L GND #PWR07
 U 1 1 5824A2B9
 P 1350 1250
-F 0 "#PWR6" H 1350 1000 50  0001 C CNN
+F 0 "#PWR07" H 1350 1000 50  0001 C CNN
 F 1 "GND" H 1355 1077 50  0000 C CNN
 F 2 "" H 1350 1250 50  0000 C CNN
@@
 	1350 850  1350 750
 $Comp
-L GND #PWR12
+L GND #PWR08
 U 1 1 591462E1
 P 4350 4800
-F 0 "#PWR12" H 4350 4550 50  0001 C CNN
+F 0 "#PWR08" H 4350 4550 50  0001 C CNN
 F 1 "GND" H 4355 4627 50  0000 C CNN
 F 2 "" H 4350 4800 50  0000 C CNN
@@
 $EndComp
 $Comp
-L GND #PWR11
+L GND #PWR09
 U 1 1 591578E5
 P 3600 4800
-F 0 "#PWR11" H 3600 4550 50  0001 C CNN
+F 0 "#PWR09" H 3600 4550 50  0001 C CNN
 F 1 "GND" H 3605 4627 50  0000 C CNN
 F 2 "" H 3600 4800 50  0000 C CNN
@@
 $EndComp
 $Comp
-L GND #PWR10
+L GND #PWR010
 U 1 1 59157ACB
 P 3100 4800
-F 0 "#PWR10" H 3100 4550 50  0001 C CNN
+F 0 "#PWR010" H 3100 4550 50  0001 C CNN
 F 1 "GND" H 3105 4627 50  0000 C CNN
 F 2 "" H 3100 4800 50  0000 C CNN
@@
 Connection ~ 6050 2050
 $Comp
-L GND #PWR14
+L GND #PWR011
 U 1 1 591715B5
 P 5500 3950
-F 0 "#PWR14" H 5500 3700 50  0001 C CNN
+F 0 "#PWR011" H 5500 3700 50  0001 C CNN
 F 1 "GND" H 5505 3777 50  0000 C CNN
 F 2 "" H 5500 3950 50  0000 C CNN
@@
 $EndComp
 $Comp
-L GND #PWR15
+L GND #PWR012
 U 1 1 591720D6
 P 5800 3950
-F 0 "#PWR15" H 5800 3700 50  0001 C CNN
+F 0 "#PWR012" H 5800 3700 50  0001 C CNN
 F 1 "GND" H 5805 3777 50  0000 C CNN
 F 2 "" H 5800 3950 50  0000 C CNN
@@
 $EndComp
 $Comp
-L GND #PWR16
+L GND #PWR013
 U 1 1 59172162
 P 6100 3950
-F 0 "#PWR16" H 6100 3700 50  0001 C CNN
+F 0 "#PWR013" H 6100 3700 50  0001 C CNN
 F 1 "GND" H 6105 3777 50  0000 C CNN
 F 2 "" H 6100 3950 50  0000 C CNN
@@
 $EndComp
 $Comp
-L GND #PWR17
+L GND #PWR014
 U 1 1 591721EE
 P 6400 3950
-F 0 "#PWR17" H 6400 3700 50  0001 C CNN
+F 0 "#PWR014" H 6400 3700 50  0001 C CNN
 F 1 "GND" H 6405 3777 50  0000 C CNN
 F 2 "" H 6400 3950 50  0000 C CNN
@@
 Connection ~ 6400 3150
 $Comp
-L VCC #PWR5
+L VCC #PWR015
 U 1 1 5918067E
 P 1350 750
-F 0 "#PWR5" H 1350 600 50  0001 C CNN
+F 0 "#PWR015" H 1350 600 50  0001 C CNN
 F 1 "VCC" H 1367 923 50  0000 C CNN
 F 2 "" H 1350 750 50  0000 C CNN
@@
 $EndComp
 $Comp
-L VCC #PWR8
+L VCC #PWR016
 U 1 1 592A2546
 P 2050 750
-F 0 "#PWR8" H 2050 600 50  0001 C CNN
+F 0 "#PWR016" H 2050 600 50  0001 C CNN
 F 1 "VCC" H 2067 923 50  0000 C CNN
 F 2 "" H 2050 750 50  0000 C CNN
@@
 $EndComp
 $Comp
-L GND #PWR9
+L GND #PWR017
 U 1 1 592A25DB
 P 2050 1250
-F 0 "#PWR9" H 2050 1000 50  0001 C CNN
+F 0 "#PWR017" H 2050 1000 50  0001 C CNN
 F 1 "GND" H 2055 1077 50  0000 C CNN
 F 2 "" H 2050 1250 50  0000 C CNN
@@
 F 0 "J12" H 9279 2780 50  0000 L CNN
 F 1 "CONN1_1" H 9400 2700 40  0001 C CNN
-F 2 "Mlab_CON:WAGO256" H 9350 2700 60  0001 C CNN
+F 2 "Mlab_CON:WAGO256_2" H 9350 2700 60  0001 C CNN
 F 3 "" H 9350 2700 60  0000 C CNN
 	1    9300 2750
@@
 F 0 "J14" H 9279 3080 50  0000 L CNN
 F 1 "CONN1_1" H 9400 3000 40  0001 C CNN
-F 2 "Mlab_CON:WAGO256" H 9350 3000 60  0001 C CNN
+F 2 "Mlab_CON:WAGO256_2" H 9350 3000 60  0001 C CNN
 F 3 "" H 9350 3000 60  0000 C CNN
 	1    9300 3050
@@
 $EndComp
 $Comp
-L GND #PWR18
+L GND #PWR018
 U 1 1 592A8675
 P 6850 3950
-F 0 "#PWR18" H 6850 3700 50  0001 C CNN
+F 0 "#PWR018" H 6850 3700 50  0001 C CNN
 F 1 "GND" H 6855 3777 50  0000 C CNN
 F 2 "" H 6850 3950 50  0000 C CNN
@@
 $EndComp
 $Comp
-L GND #PWR19
+L GND #PWR019
 U 1 1 592A8D34
 P 7300 3950
-F 0 "#PWR19" H 7300 3700 50  0001 C CNN
+F 0 "#PWR019" H 7300 3700 50  0001 C CNN
 F 1 "GND" H 7305 3777 50  0000 C CNN
 F 2 "" H 7300 3950 50  0000 C CNN
@@
 $EndComp
 $Comp
-L GND #PWR20
+L GND #PWR020
 U 1 1 592A9057
 P 7750 3950
-F 0 "#PWR20" H 7750 3700 50  0001 C CNN
+F 0 "#PWR020" H 7750 3700 50  0001 C CNN
 F 1 "GND" H 7755 3777 50  0000 C CNN
 F 2 "" H 7750 3950 50  0000 C CNN
@@
 $EndComp
 $Comp
-L GND #PWR21
+L GND #PWR021
 U 1 1 592A90E6
 P 8200 3950
-F 0 "#PWR21" H 8200 3700 50  0001 C CNN
+F 0 "#PWR021" H 8200 3700 50  0001 C CNN
 F 1 "GND" H 8205 3777 50  0000 C CNN
 F 2 "" H 8200 3950 50  0000 C CNN
@@
 F 0 "J13" H 9279 2930 50  0000 L CNN
 F 1 "CONN1_1" H 9400 2850 40  0001 C CNN
-F 2 "Mlab_CON:WAGO256" H 9350 2850 60  0001 C CNN
+F 2 "Mlab_CON:WAGO256_2" H 9350 2850 60  0001 C CNN
 F 3 "" H 9350 2850 60  0000 C CNN
 	1    9300 2900
@@
 F 0 "J15" H 9279 3230 50  0000 L CNN
 F 1 "CONN1_1" H 9400 3150 40  0001 C CNN
-F 2 "Mlab_CON:WAGO256" H 9350 3150 60  0001 C CNN
+F 2 "Mlab_CON:WAGO256_2" H 9350 3150 60  0001 C CNN
 F 3 "" H 9350 3150 60  0000 C CNN
 	1    9300 3200
@@
 F 0 "J16" H 9279 3430 50  0000 L CNN
 F 1 "CONN1_1" H 9400 3350 40  0001 C CNN
-F 2 "Mlab_CON:WAGO256" H 9350 3350 60  0001 C CNN
+F 2 "Mlab_CON:WAGO256_2" H 9350 3350 60  0001 C CNN
 F 3 "" H 9350 3350 60  0000 C CNN
 	1    9300 3400
@@
 F 0 "J17" H 9279 3530 50  0000 L CNN
 F 1 "CONN1_1" H 9400 3450 40  0001 C CNN
-F 2 "Mlab_CON:WAGO256" H 9350 3450 60  0001 C CNN
+F 2 "Mlab_CON:WAGO256_2" H 9350 3450 60  0001 C CNN
 F 3 "" H 9350 3450 60  0000 C CNN
 	1    9300 3500
@@
 F 0 "J18" H 9279 3630 50  0000 L CNN
 F 1 "CONN1_1" H 9400 3550 40  0001 C CNN
-F 2 "Mlab_CON:WAGO256" H 9350 3550 60  0001 C CNN
+F 2 "Mlab_CON:WAGO256_2" H 9350 3550 60  0001 C CNN
 F 3 "" H 9350 3550 60  0000 C CNN
 	1    9300 3600
@@
 F 0 "J19" H 9279 3730 50  0000 L CNN
 F 1 "CONN1_1" H 9400 3650 40  0001 C CNN
-F 2 "Mlab_CON:WAGO256" H 9350 3650 60  0001 C CNN
+F 2 "Mlab_CON:WAGO256_2" H 9350 3650 60  0001 C CNN
 F 3 "" H 9350 3650 60  0000 C CNN
 	1    9300 3700
@@
 $EndComp
 $Comp
-L GND #PWR22
+L GND #PWR022
 U 1 1 592B4758
 P 8900 3700
-F 0 "#PWR22" H 8900 3450 50  0001 C CNN
+F 0 "#PWR022" H 8900 3450 50  0001 C CNN
 F 1 "GND" H 8905 3527 50  0000 C CNN
 F 2 "" H 8900 3700 50  0000 C CNN
@@
 $EndComp
 $Comp
-L GND #PWR7
+L GND #PWR023
 U 1 1 59305CBE
 P 1900 1950
-F 0 "#PWR7" H 1900 1700 50  0001 C CNN
+F 0 "#PWR023" H 1900 1700 50  0001 C CNN
 F 1 "GND" H 1905 1777 50  0000 C CNN
 F 2 "" H 1900 1950 50  0000 C CNN
