File: PowerSupply/UNIPOWER07A/SCH_PCB/UNIPOWER07A.kicad_pcb (KiCad board)
At the start: 2 copper layers, 40.1 x 40.1 mm, 18 parts, among them CON1 JACK_DC2.1, J12 JUMP_4X2, J3 CONN1_1, J4 CONN1_1, J7 CONN1_1, J8 CONN1_1, J9 CONN1_1, P1 _, P2 _, P3 _, P4 _, SW1 Prepinac

Commit message: Production data
Other:
- board text added: "POWER IN"
Changed lines of the file:
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@@
     (links 31)
     (no_connects 0)
-    (area 0.178999 -40.461001 40.461001 -0.178999)
+    (area -11.176 -45.466 85.598001 5.080001)
     (thickness 1.6)
-    (drawings 14)
+    (drawings 15)
     (tracks 161)
     (zones 0)
@@
       (net 3 "Net-(D2-Pad1)"))
   )
+  (gr_text "POWER IN" (at 8.128 -14.478 90) (layer F.SilkS)
+    (effects (font (size 1.5 1.5) (thickness 0.3)))
+  )
   (gr_text - (at 12.446 -24.638) (layer F.SilkS)
     (effects (font (size 1.5 1.5) (thickness 0.3)))
@@
     (effects (font (size 1.5 1.5) (thickness 0.3)))
   )
-  (gr_text MLAB.CZ (at 24.638 -17.272) (layer F.SilkS)
-    (effects (font (size 1.5 1.5) (thickness 0.3)))
+  (gr_text MLAB.CZ (at 25.4 -17.272) (layer F.SilkS)
+    (effects (font (size 1.8 1.8) (thickness 0.3)))
   )
   (gr_text JACHO (at 4.826 -29.464) (layer F.SilkS)
     (effects (font (size 1.5 1.5) (thickness 0.3)))
   )
-  (gr_text UNIPOWER07A (at 27.432 -19.558) (layer F.SilkS)
-    (effects (font (size 1.5 1.5) (thickness 0.3)))
+  (gr_text UNIPOWER07A (at 29.21 -19.558) (layer F.SilkS)
+    (effects (font (size 1.8 1.8) (thickness 0.3)))
   )
   (gr_text MLAB.CZ (at 3.556 -25.654 90) (layer B.Cu)
