File: power_supply/DOWNCONV01A/hw/sch_pcb/STEPDOWN1A.sch (KiCad schematic (older format))
At the start: 38 parts, among them J1 CONN1_1, J2 CONN1_1, J3 CONN1_1, J4 CONN1_1, P1 _NC, P2 _NC, P3 _NC, P4 _NC, P5 CONN_01X02, U1 L7987

Commit message: A PDF version of power module schematics plotted.
Parts:
- C1, C12, C14, C16: symbol CP -> STEPDOWN1A-rescue:CP-RESCUE-STEPDOWN1A
- C10, C11, C13, C15, C2, C3, C4, C5, C6, C7, C8, C9: symbol C -> STEPDOWN1A-rescue:C-RESCUE-STEPDOWN1A
- D1: symbol D_Schottky -> STEPDOWN1A-rescue:D_Schottky-RESCUE-STEPDOWN1A
- D2: symbol LED -> STEPDOWN1A-rescue:LED-RESCUE-STEPDOWN1A
- J1, J2, J3, J4: symbol CONN1_1 -> STEPDOWN1A-rescue:CONN1_1-RESCUE-STEPDOWN1A
- L1, L2: symbol INDUCTOR -> STEPDOWN1A-rescue:INDUCTOR-RESCUE-STEPDOWN1A
- P1, P2, P3, P4: symbol CONN_01X01 -> STEPDOWN1A-rescue:CONN_01X01-RESCUE-STEPDOWN1A
- P5: symbol CONN_01X02 -> STEPDOWN1A-rescue:CONN_01X02-RESCUE-STEPDOWN1A
- R1, R2, R3, R4, R5, R6, R7, R8: symbol R -> STEPDOWN1A-rescue:R-RESCUE-STEPDOWN1A
- U1: symbol L7987 -> STEPDOWN1A-rescue:L7987-RESCUE-STEPDOWN1A
Connections:
- wire segments 84 -> 115
