File: power_supply/DOWNCONV02A/hw/sch_pcb/STEPDOWN2A.sch (KiCad schematic (older format))
At the start: 30 parts, among them J1 CONN1_1, J2 CONN1_1, J3 CONN1_1, J4 CONN1_1, P1 _NC, P2 _NC, P3 _NC, P4 _NC, P5 CONN_01X01, U1 TPS54332

Commit message: A PDF version of power module schematics plotted.
Parts:
- C1, C10, C12, C8: symbol CP -> STEPDOWN2A-rescue:CP-RESCUE-STEPDOWN2A
- C11, C2, C3, C4, C5, C6, C7, C9: symbol C -> STEPDOWN2A-rescue:C-RESCUE-STEPDOWN2A
- D1: symbol D_Schottky -> STEPDOWN2A-rescue:D_Schottky-RESCUE-STEPDOWN2A
- D2: symbol Led_Small -> STEPDOWN2A-rescue:Led_Small-RESCUE-STEPDOWN2A
- J1, J2, J3, J4: symbol CONN1_1 -> STEPDOWN2A-rescue:CONN1_1-RESCUE-STEPDOWN2A
- L1, L2: symbol INDUCTOR -> STEPDOWN2A-rescue:INDUCTOR-RESCUE-STEPDOWN2A
- P1, P2, P3, P4, P5: symbol CONN_01X01 -> STEPDOWN2A-rescue:CONN_01X01-RESCUE-STEPDOWN2A
- R1, R2, R3, R4: symbol R -> STEPDOWN2A-rescue:R-RESCUE-STEPDOWN2A
- U1: symbol TPS54332 -> STEPDOWN2A-rescue:TPS54332-RESCUE-STEPDOWN2A
Connections:
- wire segments 53 -> 71
