File: sensors/DATALOGGER01A/hw/sch_pcb/DATALOGGER01A.kicad_pcb (KiCad board)
At the start: 2 copper layers, 0 parts

Commit message: edit
Parts:
- added BT1: BX0037, Connector_Card:SD_TE_2041021, F.Cu at (114.1, 117.3)
- added C1: 100nF, Mlab_R:SMD-0805, F.Cu at (169.8, 156.3)
- added C10: EMI_Filter_C, Mlab_L:FIR1, F.Cu at (192.8, 144.3)
- added C11: 10uF, Mlab_R:SMD-0805, F.Cu at (161.3, 157.1)
- added C12: 1nF, Mlab_R:SMD-0805, F.Cu at (165.6, 154.5)
- added C13: 100nF, Mlab_R:SMD-0805, F.Cu at (152.7, 129.7)
- added C14: 10uF, Mlab_R:SMD-0805, F.Cu at (144.2, 129.7)
- added C15: 100nF, Mlab_R:SMD-0805, F.Cu at (140.0, 129.7)
- added C16: 4u7, Mlab_R:SMD-0805, F.Cu at (135.7, 129.7)
- added C17: 100nF, Mlab_R:SMD-0805, F.Cu at (165.6, 157.1)
- added C18: 100nF, Mlab_R:SMD-0805, F.Cu at (185.2, 152.9)
- added C2: 100nF, Mlab_R:SMD-0805, F.Cu at (174.1, 156.3)
- added C3: 100nF, Mlab_R:SMD-0805, F.Cu at (242.9, 86.7)
- added C4: 100nF, Mlab_R:SMD-0805, F.Cu at (208.1, 128.1)
- added C5: 100nF, Mlab_R:SMD-0805, F.Cu at (247.2, 86.7)
- added C6: 100nF, Mlab_R:SMD-0805, F.Cu at (178.3, 156.3)
- added C7: 1uF, Mlab_R:SMD-0805, F.Cu at (217.7, 120.6)
- added C8: 100nF, Mlab_R:SMD-0805, F.Cu at (199.3, 138.4)
- added C9: 47uF, Mlab_C:TantalC_SizeC_Reflow, F.Cu at (235.1, 106.4)
- added D2: M4, Mlab_D:SMA_Standard, F.Cu at (186.6, 146.1)
- added F1: 750mA, Mlab_F:1812, F.Cu at (201.5, 131.6)
- added J1: HEADER_2x01_PARALLEL, Mlab_Pin_Headers:Straight_2x01, F.Cu at (143.1, 77.7)
- added J10: HEADER_2x03_PARALLEL, Mlab_Pin_Headers:Straight_2x03, F.Cu at (143.1, 105.1)
- added J11: HEADER_2x01, Mlab_Pin_Headers:Straight_2x01, F.Cu at (162.9, 149.0)
- added J12: HEADER_2x01_PARALLEL, Mlab_Pin_Headers:Straight_2x01, F.Cu at (171.0, 77.7)
- added J13: HEADER_2x01_PARALLEL, Mlab_Pin_Headers:Straight_2x01, F.Cu at (143.1, 94.3)
- added J14: HEADER_2x01_PARALLEL, Mlab_Pin_Headers:Straight_2x01, F.Cu at (143.1, 86.0)
- added J15: HEADER_2x01_PARALLEL, Mlab_Pin_Headers:Straight_2x01, F.Cu at (143.1, 115.9)
- added J16: HEADER_2x01_PARALLEL, Mlab_Pin_Headers:Straight_2x01, F.Cu at (171.0, 102.6)
- added J17: HEADER_2x01_PARALLEL, Mlab_Pin_Headers:Straight_2x01, F.Cu at (198.9, 77.7)
- added J18: HEADER_2x01_PARALLEL, Mlab_Pin_Headers:Straight_2x01, F.Cu at (226.8, 86.0)
- added J19: HEADER_2x01_PARALLEL, Mlab_Pin_Headers:Straight_2x01, F.Cu at (140.9, 143.7)
- added J2: HEADER_2x01_PARALLEL, Mlab_Pin_Headers:Straight_2x01, F.Cu at (143.1, 124.2)
- added J20: HEADER_2x01_PARALLEL, Mlab_Pin_Headers:Straight_2x01, F.Cu at (198.9, 110.8)
- added J21: HEADER_2x01, Mlab_Pin_Headers:Straight_2x01, F.Cu at (220.9, 94.3)
- added J22: HEADER_2x01_PARALLEL, Mlab_Pin_Headers:Straight_2x01, F.Cu at (168.7, 140.8)
- added J23: HEADER_2x01_PARALLEL, Mlab_Pin_Headers:Straight_2x01, F.Cu at (226.8, 77.7)
- added J24: HEADER_2x01_PARALLEL, Mlab_Pin_Headers:Straight_2x01, F.Cu at (198.9, 86.0)
- added J25: HEADER_2x01_PARALLEL, Mlab_Pin_Headers:Straight_2x01, F.Cu at (198.9, 102.6)
- added J26: HEADER_2x01_PARALLEL, Mlab_Pin_Headers:Straight_2x01, F.Cu at (140.9, 152.0)
- added J27: HEADER_2x01_PARALLEL, Mlab_Pin_Headers:Straight_2x01, F.Cu at (198.9, 94.3)
- added J28: HEADER_2x01_PARALLEL, Mlab_Pin_Headers:Straight_2x01, F.Cu at (171.0, 119.1)
- added J29: HEADER_2x01_PARALLEL, Mlab_Pin_Headers:Straight_2x01, F.Cu at (168.7, 132.5)
- added J3: HEADER_2x01_PARALLEL, Mlab_Pin_Headers:Straight_2x01, F.Cu at (171.0, 94.3)
- added J30: HEADER_2x01_PARALLEL, Mlab_Pin_Headers:Straight_2x01, F.Cu at (171.0, 110.8)
- added J31: HEADER_2x03, Mlab_Pin_Headers:Straight_2x03, F.Cu at (220.9, 105.1)
- added J4: HEADER_2x01_PARALLEL, Mlab_Pin_Headers:Straight_2x01, F.Cu at (140.9, 135.4)
- added J5: HEADER_2x01_PARALLEL, Mlab_Pin_Headers:Straight_2x01, F.Cu at (171.0, 86.0)
- added J6: HEADER_2x03_PARALLEL, Mlab_Pin_Headers:Straight_2x03, F.Cu at (113.0, 138.0)
- added J7: SD_Card, Connector_Card:SD_TE_2041021, F.Cu at (114.1, 88.4)
- added J8: HEADER_2x01_PARALLEL, Mlab_Pin_Headers:Straight_2x01, F.Cu at (113.0, 148.8)
- added J9: HEADER_2x01, Mlab_Pin_Headers:Straight_2x01, F.Cu at (193.0, 119.1)
- added M1: HOLE, Mlab_Mechanical:MountingHole_3mm, F.Cu at (244.3, 79.4)
- added M2: HOLE, Mlab_Mechanical:MountingHole_3mm, F.Cu at (204.7, 120.8)
- added M3: HOLE, Mlab_Mechanical:MountingHole_3mm, F.Cu at (211.9, 120.8)
- added M4: HOLE, Mlab_Mechanical:MountingHole_3mm, F.Cu at (232.6, 96.0)
- added R1: 100, Mlab_R:SMD-0805, F.Cu at (161.3, 154.5)
- added R10: 1k, Mlab_R:SMD-0805, F.Cu at (122.5, 154.3)
- added R2: 100, Mlab_R:SMD-0805, F.Cu at (131.5, 129.7)
- added R3: 100, Mlab_R:SMD-0805, F.Cu at (157.1, 157.1)
- added R4: 100, Mlab_R:SMD-0805, F.Cu at (106.7, 72.7)
- added R5: 4k7, Mlab_R:SMD-0805, F.Cu at (180.4, 124.6)
- added R6: 10k, Mlab_R:SMD-0805, F.Cu at (176.2, 124.6)
- added R7: 10k, Mlab_R:SMD-0805, F.Cu at (148.5, 129.7)
- added R8: -, Mlab_R:SMD-0805, F.Cu at (171.9, 124.6)
- added R9: 10k, Mlab_R:SMD-0805, F.Cu at (122.5, 156.9)
- added U1: ISL21080CIH320Z-TK, Package_TO_SOT_SMD:SOT-23, F.Cu at (217.2, 130.8)
- added U2: TPS22965-Q1, Package_SON:WSON-8-1EP_2x2mm_P0.5mm_EP0.9x1.6mm_ThermalVias, F.Cu at (242.0, 93.3)
- added U3: ATMEGA1284P-AU, Package_QFP:TQFP-44_10x10mm_P0.8mm, F.Cu at (189.9, 131.9)
- added U4: PCF85263A, Mlab_IO:TSSOP-10_3x3mm_Pitch0.5mm, F.Cu at (220.2, 115.6)
- added U5: LM4041CIM3-1.2(neosazovat), Package_TO_SOT_SMD:SOT-23, F.Cu at (219.7, 137.2)
- added Y1: 16MHz, Mlab_XTAL:Crystal_HC49-U_Vertical, F.Cu at (177.0, 149.9)
- added Y2: ABS07-120-32.768KHZ-T, Mlab_XTAL:ABS07, F.Cu at (109.8, 156.8)

Commit message: Edit
Parts:
- added BT2: BX0037, Mlab_Batery:BX0037, F.Cu at (36.8, -34.3)
- added SW1: 5MS1S102AM6QE, Mlab_SW:5MS1S102AM6QE, F.Cu at (50.8, -1.27)
- BT1: footprint Connector_Card:SD_TE_2041021 -> Mlab_Batery:BX0037
- C1, C10, C11, C12, C13, C14, C15, C16, C17, C18, C2, C3, C4, C5, C6, C7, C8, C9, D2, F1, J7, R1, R10, R2, R3, R4, R5, R6, R7, R8, R9, U1, U2, U3, U4, U5, Y2: moved to B.Cu
- moved U5 294.0 mm to (44.2, -98.7)
- moved M3 292.7 mm to (5.08, -86.4)
- moved R6 291.8 mm to (35.6, -131.1), turned to 90 degrees
- moved R7 288.1 mm to (30.8, -133.3)
- moved J31 288.0 mm to (15.2, -96.5), turned to 90 degrees
- moved U1 283.3 mm to (43.2, -92.7)
- moved J4 282.8 mm to (35.6, -127.0), turned to 90 degrees
- moved C4 278.5 mm to (38.4, -92.7)
- moved J2 275.3 mm to (30.5, -127.0), turned to 90 degrees
- moved C7 269.9 mm to (46.0, -87.6)
- moved C2 268.7 mm to (43.2, -78.4), turned to 270 degrees
- moved C1 267.9 mm to (40.6, -78.4), turned to 270 degrees
- moved C6 267.1 mm to (50.8, -78.4), turned to 270 degrees
- moved C17 266.0 mm to (50.8, -82.9), turned to 270 degrees
- moved J22 265.0 mm to (50.8, -96.5), turned to 90 degrees
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Connections:
- J27 pad 1: Net-(J27-Pad1) -> /PB6
- J27 pad 2: Net-(J27-Pad1) -> /PB6
- J28 pad 1: Net-(J28-Pad1) -> /PB7
- J28 pad 2: Net-(J28-Pad1) -> /PB7
- J29 pad 1: Net-(J29-Pad1) -> /PB5
- J29 pad 2: Net-(J29-Pad1) -> /PB5
- J5 pad 1: Net-(J5-Pad1) -> GND
- J5 pad 2: Net-(J5-Pad1) -> GND
Other:
- board outline added: 80.8 x 101.1 mm

Commit message: Edit
Parts:
- added D3: HLMP-K150+FIX-LED-313, Mlab_D:FIX-LED-313, F.Cu at (67.3, -5.08)
- added L1: 10uH - LQH32CN100K23L, Mlab_R:SMD-1210, B.Cu at (41.9, -76.8)
- R10: value 1k -> 2k2
- moved J1 95.5 mm to (74.9, -43.8), turned to 180 degrees
- moved J2 92.1 mm to (74.9, -46.4), turned to 180 degrees
- moved R7 90.0 mm to (63.5, -49.5), turned to 90 degrees
- moved R6 88.9 mm to (64.1, -47.0), turned to 180 degrees
- moved J3 88.6 mm to (74.9, -48.9), turned to 180 degrees
- moved J11 85.4 mm to (44.5, -8.89), turned to 270 degrees
- moved J4 85.2 mm to (74.9, -51.4), turned to 180 degrees
- moved J5 81.8 mm to (74.9, -54.0), turned to 180 degrees
- moved C7 66.2 mm to (71.8, -26.7)
- moved J31 60.3 mm to (74.9, -87.6), turned to 180 degrees
- moved J21 27.8 mm to (74.9, -37.5)
- moved J30 23.5 mm to (74.9, -40.0)
- moved U4 21.4 mm to (59.1, -45.1)
- moved C18 21.4 mm to (55.6, -47.6)
- moved Y2 21.4 mm to (60.3, -48.9)
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Routing:
- net /LED: track 0.00 -> 83.4 mm, vias 0 -> 2
- net VDD: track 0.00 -> 19.7 mm
- net Net-(C8-Pad1): track 0.00 -> 15.6 mm
- net /AVCC: track 0.00 -> 9.30 mm
- net Net-(C14-Pad1): track 0.00 -> 7.96 mm
- net Net-(C16-Pad1): track 0.00 -> 7.13 mm
- net /PC3: track 0.00 -> 6.06 mm
- net /AREF: track 0.00 -> 5.52 mm
- net /RST#: track 0.00 -> 3.07 mm
- net /INT: track 0.00 -> 2.88 mm, vias 0 -> 1
- net Net-(C5-Pad1): track 0.00 -> 2.62 mm
- net /PC1: vias 0 -> 1
Other:
- net class Default: via_dia 0.6 -> 0.8
- net class MLAB_default: via_dia 0.6 -> 0.8
- rule via_min_drill: 0.3 -> 0.4
- rule via_min_size: 0.4 -> 0.8
- board text added: "RST"

Commit message: edit
Parts:
- added C19: 100nF, Mlab_R:SMD-0805, B.Cu at (56.8, -90.2)
- added C20: 100nF, Mlab_R:SMD-0805, B.Cu at (60.3, -73.0)
- added C21: 100nF, Mlab_R:SMD-0805, B.Cu at (66.0, -82.2)
- moved M2 236.0 mm to (5.08, -5.08)
- moved M4 139.0 mm to (131.4, -94.6)
- moved D3 54.0 mm to (13.3, -5.08)
- moved R10 49.4 mm to (15.9, -10.8), turned to 90 degrees
- moved J11 24.8 mm to (19.7, -7.62)
- moved J12 17.8 mm to (12.7, -94.0)
- moved R2 15.0 mm to (31.8, -29.5), turned to 90 degrees
- moved J13 12.7 mm to (15.2, -94.0)
- moved C12 12.2 mm to (59.7, -29.8)
- moved C11 12.1 mm to (35.2, -31.8), turned to 180 degrees
- moved C7 11.6 mm to (60.3, -28.6)
- moved R3 11.1 mm to (39.4, -29.5), turned to 90 degrees
- moved J7 10.8 mm to (36.2, -14.0)
- moved R4 9.55 mm to (43.8, -29.5), turned to 90 degrees
- moved C18 9.34 mm to (64.8, -46.0), turned to 270 degrees
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Routing:
- net VDD: track 19.7 -> 165.9 mm, vias 0 -> 4
- net Net-(J11-Pad1): track 0.00 -> 104.9 mm, vias 0 -> 1
- net /PB7: track 0.00 -> 91.8 mm, vias 0 -> 2
- net /PB5: track 0.00 -> 90.8 mm, vias 0 -> 3
- net /PB6: track 0.00 -> 90.6 mm, vias 0 -> 3
- net Net-(BT1-Pad1): track 0.00 -> 87.3 mm
- net /PB4: track 0.00 -> 78.0 mm, vias 0 -> 2
- net /PC2: track 0.00 -> 56.8 mm
- net /PC5: track 0.00 -> 48.4 mm
- net /INT: track 2.88 -> 50.2 mm, vias 1 -> 0
- net /PC3: track 6.06 -> 53.2 mm
- net /PC6: track 0.00 -> 46.7 mm
- net /PC1: track 0.00 -> 44.7 mm, vias 1 -> 0
- net /PC0: track 0.00 -> 40.5 mm, vias 0 -> 2
- net /TX1: track 0.00 -> 29.9 mm
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
Commit message: Edit
Parts:
- added BT3: Battery_Cell-device, Mlab_Batery:CH28-2032, B.Cu at (37.5, -53.3)
- added F2: 750mA, Mlab_F:1812, B.Cu at (69.2, -28.6)
- added J32: HEADER_2x01, Mlab_Pin_Headers:Straight_2x01, F.Cu at (76.2, -17.8)
- added J33: HEADER_2x03_PARALLEL, Mlab_Pin_Headers:Straight_2x03, F.Cu at (76.2, -12.7)
- added J34: MCC-SD (kouka z modulu), Mlab_CON:MCC-SD, B.Cu at (36.8, -14.0)
- J7: value SD_Card -> MCC-SD
- moved M4 55.2 mm to (76.2, -96.2)
- moved R4 11.8 mm to (45.1, -41.3)
- moved R3 11.8 mm to (40.0, -41.3)
- moved R1 11.8 mm to (29.8, -41.3)
- moved R2 11.8 mm to (32.4, -41.3)
- moved C11 11.5 mm to (36.2, -43.2)
- moved C15 11.5 mm to (36.2, -40.6)
- moved J7 11.4 mm to (36.8, -25.4)
- moved C12 9.92 mm to (66.0, -37.5), turned to 180 degrees
- moved J6 8.98 mm to (76.2, -22.9), turned to 90 degrees
- moved C7 8.67 mm to (61.6, -37.1), turned to 90 degrees
- moved J10 8.25 mm to (74.9, -31.8)
- moved U2 7.41 mm to (65.4, -34.9)
Connections:
- F1 pad 2: Net-(BT1-Pad1) -> Net-(F1-Pad2)
- J6 pad 3: Net-(BT1-Pad1) -> Net-(F2-Pad1)
- J6 pad 4: Net-(BT1-Pad1) -> Net-(F2-Pad1)
Routing:
- net GND: track 0.00 -> 331.3 mm, vias 0 -> 154
- net (no net): track 0.00 -> 75.6 mm, vias 0 -> 30
- net /PA2: track 0.00 -> 63.9 mm, vias 0 -> 4
- net VDD: track 165.9 -> 221.3 mm, vias 4 -> 6
- net /SD_VDD: track 0.00 -> 49.9 mm
- net Net-(BT1-Pad1): track 87.3 -> 59.9 mm
- net /PB4: track 78.0 -> 59.2 mm
- net Net-(F2-Pad1): track 0.00 -> 16.8 mm
- net /PB7: track 91.8 -> 76.1 mm
- net Net-(F1-Pad2): track 0.00 -> 14.6 mm
- net Net-(J34-Pad7): track 0.00 -> 14.5 mm
- net Net-(J34-Pad1): track 0.00 -> 14.4 mm
- net Net-(J34-Pad2): track 0.00 -> 14.4 mm
- net Net-(J34-Pad5): track 0.00 -> 14.4 mm
- net Net-(J10-Pad3): track 0.00 -> 13.6 mm
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- added copper zone on B.Cu, net GND
- added copper zone on F.Cu, net GND
Other:
- board text added: "2018"
- board text added: "AREF"
- board text added: "AREF_IN"
- board text added: "ATMEL ISP"
- board text added: "BATERY"
- board text added: "DATALOGGER01A"
- board text added: "GND"
- board text added: "INT"
- board text added: "INTA"
- board text added: "JACHO"
- board text added: "MLAB.CZ"
- board text added: "PA0"
- board text added: "PA1"
- board text added: "PB0"
- board text added: "PB5"
- board text added: "PB6"
- board text added: "PB7"
- board text added: "PC2"
- board text added: "PC3"
- board text added: "PC5"
- board text added: "PC6"
- board text added: "POWER IN"
- board text added: "RST#"
- board text added: "RX0"
- board text added: "RX1"
- board text added: "SCL"
- board text added: "SDA"
- board text added: "SDVDD"
- board text added: "SW POWER"
- board text added: "TX0"
- board text added: "TX1"
- board text added: "VDD"
- board text removed: "RST"

Commit message: Edit
Routing:
- net GND: track 331.3 -> 435.8 mm, vias 154 -> 191
- net (no net): track 75.6 -> 0.00 mm, vias 30 -> 0

Commit message: Edit
Parts:
- moved SW1 1.02 mm to (62.9, -2.29)
Connections:
- SW1 pad 4: (no net) -> GND
Routing:
- net Net-(D2-Pad1): track 9.42 -> 8.40 mm
- net Net-(C10-Pad1): track 10.7 -> 9.80 mm
Changed lines of the file:
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@@
-(kicad_pcb (version 20171130) (host pcbnew "(5.0.0-rc2-18-g3893c43eb)")
+(kicad_pcb (version 20171130) (host pcbnew "(2018-02-10 revision a04965c36)-makepkg")
   (general
     (thickness 1.6)
-    (drawings 41)
-    (tracks 924)
+    (drawings 39)
+    (tracks 927)
     (zones 0)
     (modules 85)
@@
   )
   (setup
-    (last_trace_width 0.25)
+    (last_trace_width 2)
     (user_trace_width 0.3)
     (user_trace_width 0.4)
@@
     (mod_text_size 1 1)
     (mod_text_width 0.15)
-    (pad_size 6 6)
-    (pad_drill 3)
+    (pad_size 3 3)
+    (pad_drill 1.85)
     (pad_to_mask_clearance 0.2)
     (aux_axis_origin 0 0)
     (visible_elements 7FFFFF7F)
     (pcbplotparams
-      (layerselection 0x00030_80000001)
+      (layerselection 0x010e0_ffffffff)
       (usegerberextensions false)
       (usegerberattributes false)
@@
       (outputformat 1)
       (mirror false)
-      (drillshape 1)
+      (drillshape 0)
       (scaleselection 1)
-      (outputdirectory ""))
+      (outputdirectory ../cam_profi/))
   )
   (net 0 "")
@@
   )
   (module Mlab_SW:5MS1S102AM6QE (layer F.Cu)
-    (at 62.865 -1.27)
+    (at 62.865 -2.286)
     (fp_text reference SW1 (at 0 -2.54) (layer F.SilkS)
       (effects (font (size 1 1) (thickness 0.15)))
@@
     (pad 1 thru_hole circle (at -4.7 -9.53) (size 3 3) (drill 1.85) (layers *.Cu *.Mask)
       (net 8 "Net-(C10-Pad1)"))
-    (pad 4 thru_hole circle (at 6.605 0) (size 3 3) (drill 1.85) (layers *.Cu *.Mask))
-    (pad 4 thru_hole circle (at -6.605 0) (size 3 3) (drill 1.85) (layers *.Cu *.Mask))
+    (pad 4 thru_hole circle (at 6.605 0) (size 3 3) (drill 1.85) (layers *.Cu *.Mask)
+      (net 1 GND))
+    (pad 4 thru_hole circle (at -6.605 0) (size 3 3) (drill 1.85) (layers *.Cu *.Mask)
+      (net 1 GND))
   )
   (module Mlab_D:FIX-LED-313 (layer F.Cu)
@@
     (effects (font (size 1.27 1.27) (thickness 0.3)))
   )
-  (dimension 81.28 (width 0.3) (layer F.SilkS)
-    (gr_text "81,280 mm" (at 40.64 -106.24) (layer F.SilkS)
-      (effects (font (size 1.5 1.5) (thickness 0.3)))
-    )
-    (feature1 (pts (xy 81.28 -101.6) (xy 81.28 -104.726421)))
-    (feature2 (pts (xy 0 -101.6) (xy 0 -104.726421)))
-    (crossbar (pts (xy 0 -104.14) (xy 81.28 -104.14)))
-    (arrow1a (pts (xy 81.28 -104.14) (xy 80.153496 -103.553579)))
-    (arrow1b (pts (xy 81.28 -104.14) (xy 80.153496 -104.726421)))
-    (arrow2a (pts (xy 0 -104.14) (xy 1.126504 -103.553579)))
-    (arrow2b (pts (xy 0 -104.14) (xy 1.126504 -104.726421)))
-  )
-  (dimension 101.631745 (width 0.3) (layer F.SilkS)
-    (gr_text "101,632 mm" (at 105.050255 -53.348993 88.56790382) (layer F.SilkS)
-      (effects (font (size 1.5 1.5) (thickness 0.3)))
-    )
-    (feature1 (pts (xy 78.74 -3.175) (xy 102.267149 -2.586821)))
-    (feature2 (pts (xy 81.28 -104.775) (xy 104.807149 -104.186821)))
-    (crossbar (pts (xy 104.220911 -104.201477) (xy 101.680911 -2.601477)))
-    (arrow1a (pts (xy 101.680911 -2.601477) (xy 101.122827 -3.742285)))
-    (arrow1b (pts (xy 101.680911 -2.601477) (xy 102.295302 -3.712973)))
-    (arrow2a (pts (xy 104.220911 -104.201477) (xy 103.60652 -103.089981)))
-    (arrow2b (pts (xy 104.220911 -104.201477) (xy 104.778995 -103.060669)))
-  )
   (gr_line (start 0.254 -0.254) (end 0.254 -101.346) (layer Edge.Cuts) (width 0.2))
   (gr_line (start 0.254 -0.254) (end 81.026 -0.254) (layer Edge.Cuts) (width 0.2))
@@
   (segment (start 69.5325 -79.0575) (end 67.945 -79.0575) (width 0.4) (layer B.Cu) (net 7))
   (segment (start 74.93 -73.66) (end 69.5325 -79.0575) (width 0.4) (layer B.Cu) (net 7))
-  (segment (start 58.165 -15.849999) (end 58.165 -10.8) (width 2) (layer B.Cu) (net 8))
-  (segment (start 57.15 -16.864999) (end 58.165 -15.849999) (width 2) (layer B.Cu) (net 8))
-  (segment (start 54.244841 -16.864999) (end 57.15 -16.864999) (width 2) (layer B.Cu) (net 8))
-  (segment (start 53.34 -17.76984) (end 54.244841 -16.864999) (width 2) (layer B.Cu) (net 8))
-  (segment (start 53.34 -17.79524) (end 53.34 -17.76984) (width 2) (layer B.Cu) (net 8))
+  (segment (start 54.244841 -16.864999) (end 53.34 -17.76984) (width 2) (layer B.Cu) (net 8))
+  (segment (start 57.350001 -16.864999) (end 54.244841 -16.864999) (width 2) (layer B.Cu) (net 8))
+  (segment (start 58.166 -16.049) (end 57.350001 -16.864999) (width 2) (layer B.Cu) (net 8))
+  (segment (start 58.166 -14.988) (end 58.166 -16.049) (width 2) (layer B.Cu) (net 8))
+  (segment (start 58.165 -11.816) (end 58.165 -14.987) (width 2) (layer B.Cu) (net 8))
+  (segment (start 58.165 -14.987) (end 58.166 -14.988) (width 2) (layer B.Cu) (net 8))
+  (segment (start 53.34 -17.76984) (end 53.34 -17.79524) (width 2) (layer B.Cu) (net 8))
   (segment (start 37.1475 -40.64) (end 37.1475 -43.18) (width 0.4) (layer B.Cu) (net 9))
   (segment (start 37.455 -37.375) (end 37.455 -40.3325) (width 0.4) (layer B.Cu) (net 9))
@@
   (segment (start 63.462084 -83.515) (end 64.719584 -84.7725) (width 0.4) (layer B.Cu) (net 13))
   (segment (start 67.945 -84.7725) (end 70.485 -84.7725) (width 0.4) (layer B.Cu) (net 13))
+  (segment (start 62.865 -11.816) (end 62.865 -13.93732) (width 2) (layer B.Cu) (net 14))
+  (segment (start 62.865 -13.93732) (end 62.865 -16.41602) (width 2) (layer B.Cu) (net 14))
   (segment (start 65.26602 -16.41602) (end 65.36 -16.51) (width 2) (layer B.Cu) (net 14))
-  (segment (start 62.865 -10.8) (end 62.865 -16.41602) (width 2) (layer B.Cu) (net 14))
   (segment (start 61.595 -16.41602) (end 62.865 -16.41602) (width 2) (layer B.Cu) (net 14))
   (segment (start 62.865 -16.41602) (end 65.26602 -16.41602) (width 2) (layer B.Cu) (net 14))
