File: motor_drivers/NEMASTEP01A/hw/sch_pcb/NEMASTEP01A.sch (KiCad schematic (older format))
At the start: 8 parts, among them J1 JUMP_3X2, M1 HOLE, M2 HOLE, M3 HOLE, M4 HOLE

Commit message: update:NEMASTEP01A.sch
Parts:
- removed D1: 0.0V, Mlab_D:Diode-MiniMELF_Standard, symbol MLAB_D:D_ZENER
- removed J1: JUMP_3X2, Mlab_Pin_Headers:Straight_2x03, symbol MLAB_Jumpers:JUMP_3X2
- removed M1, M2, M3, M4: HOLE, Mlab_Mechanical:MountingHole_3mm, symbol MLAB_MECHANICAL:HOLE
- added C10, C21, C4, C6, C7, C9: 100n, Capacitor_SMD:C_0805_2012Metric, symbol Device:C
- added C11, C12, C13, C14: 1n, Capacitor_SMD:C_0805_2012Metric, symbol Device:C
- added C15: 1n/50V, Capacitor_SMD:C_0805_2012Metric, symbol Device:C
- added C16: 100n/50V, Capacitor_SMD:C_0805_2012Metric, symbol Device:C
- added C17: 4u7/50V, Capacitor_SMD:C_1206_3216Metric, symbol Device:C
- added C18: 100u/50V, Capacitor_SMD:CP_Elec_10x10.5, symbol Device:CP
- added C19, C20: 1u/50V, Capacitor_SMD:C_0805_2012Metric, symbol Device:C
- added C22, C23: 10u, Capacitor_SMD:C_0805_2012Metric, symbol Device:C
- added C3: 100p, Capacitor_SMD:C_0805_2012Metric, symbol Device:C
- added C5: 1500p, Capacitor_SMD:C_0805_2012Metric, symbol Device:C
- added C8: 1u, Capacitor_SMD:C_0805_2012Metric, symbol Device:C
- added D1: LED, LED_SMD:LED_0805_2012Metric, symbol Device:LED
- added J1: MOT, symbol Connector_Generic:Conn_01x04
- added J2: IN, symbol Connector_Generic:Conn_01x05
- added L1: LPS4018-103MRB1, Inductor_SMD:L_Coilcraft_LPS4018, symbol pspice:INDUCTOR
- added MH1, MH2: MountingHole_Pad, MountingHole:MountingHole_3.2mm_M3_DIN965_Pad, symbol Mechanical:MountingHole_Pad
- added R1, R8: 12k, Resistor_SMD:R_0805_2012Metric, symbol Device:R
- added R10: 100k, Resistor_SMD:R_0805_2012Metric, symbol Device:R
- added R11, R12: R330, Resistor_SMD:R_0805_2012Metric, symbol Device:R
- added R13, R14, R15, R16: 120R, Resistor_SMD:R_0805_2012Metric, symbol Device:R
- added R17: 43k2_1%, Resistor_SMD:R_0805_2012Metric, symbol Device:R
- added R18: 8k2_1%, Resistor_SMD:R_0805_2012Metric, symbol Device:R
- added R19: 330R, Resistor_SMD:R_0805_2012Metric, symbol Device:R
- added R2, R9: 3k3, Resistor_SMD:R_0805_2012Metric, symbol Device:R
- added R3: 2k, Resistor_SMD:R_0805_2012Metric, symbol Device:R
- added R4, R6, R7: 4k7, Resistor_SMD:R_0805_2012Metric, symbol Device:R
- added R5: 47k, Resistor_SMD:R_0805_2012Metric, symbol Device:R
- added SW1: SW_DIP_x03, symbol Switch:SW_DIP_x03
- added U1: LV8728MR, SOIC3O W:SOIC-30W_Pitch1mm, symbol Driver_Motor:LV8728MR
- added U2: TPS62175DQC, Package_SON:WSON-10-1EP_2x3mm_P0.5mm_EP0.84x2.4mm_ThermalVias, symbol Regulator_Switching:TPS62175DQC
Connections:
- net labels added: DIR, DOWN, ENABLE, FDT, MD1, MD2, MD3, RESET, STEP, VMOT, VREF, VREG1
- wire segments 25 -> 206
- no-connect marks 0 -> 1
