File: sensors/PCRD04B/hw/sch_pcb/PCRD04B.sch (KiCad schematic (older format))
At the start: 8 parts, among them J1 0 ... Umax, M1 HOLE, M2 HOLE, M3 HOLE, M4 HOLE

Commit message: Editace modulu
Parts:
- removed C1: C/U, symbol Device:CP_Small
- removed C2: 100nF, symbol Device:C_Small
- added BT1: CH28-2032, Mlab_Batery:CH28-2032, symbol Device:Battery_Cell
- added C1: 47uF, Mlab_C:TantalC_SizeC_Reflow, symbol Device:CP
- added C10, C11, C12, C13, C14, C16, C20: 100nF, Mlab_R:SMD-0805, symbol Device:C
- added C15: 3n3, Mlab_R:SMD-0805, symbol Device:C
- added C17, C3: 4u7, Mlab_R:SMD-0805, symbol Device:C
- added C18: 2n2, Mlab_R:SMD-0805, symbol Device:C
- added C19: 1nF, Mlab_R:SMD-0805, symbol Device:C
- added C2, C21, C22, C23: EMI_Filter_C, Mlab_L:FIR1, symbol Device:EMI_Filter_C
- added C4, C6, C7, C8, C9: 10uF, Mlab_R:SMD-0805, symbol Device:C
- added C5: 1pF - 251R15S1R0AV4E, Mlab_R:SMD-0805, symbol Device:C
- added D2: D_Photo, Mlab_D:HAMAMATSU_S2744-09_rozs, symbol Device:D_Photo
- added J11, J2, J3, J4, J5, J6, J7: HEADER_2x01_PARALLEL, Mlab_Pin_Headers:Straight_2x01, symbol MLAB_HEADER:HEADER_2x01_PARALLEL
- added M5: HOLE, Mlab_Mechanical:BMIS-209-C, symbol MLAB_MECHANICAL:HOLE
- added M6: HOLE, Mlab_Mechanical:BMI-S-210-F, symbol MLAB_MECHANICAL:HOLE
- added R10, R8: 1k, Mlab_R:SMD-0805, symbol Device:R
- added R11: 4k7, Mlab_R:SMD-0805, symbol Device:R
- added R12, R7: 10k, Mlab_R:SMD-0805, symbol Device:R
- added R13: 2k2, Mlab_R:SMD-0805, symbol Device:R
- added R15: -, Mlab_R:SMD-0805, symbol Device:R
- added R2, R3, R4, R5: 100, Mlab_R:SMD-0805, symbol Device:R
- added R6: 10M, Mlab_R:SMD-0805, symbol Device:R
- added R9: 15k, Mlab_R:SMD-0805, symbol Device:R
- added U1, U2: OPA2314, Mlab_IO:SOIC-8_3.9x4.9mm_Pitch1.27mm, symbol MLAB_IO:AD8692
- added U3: ISL21080DIH312Z-TK 1V25, Package_TO_SOT_SMD:SOT-23, symbol Reference_Voltage:ISL21070CIH320Z-TK
- added U4: TS7211, Package_TO_SOT_SMD:SOT-23-5_HandSoldering, symbol Amplifier_Operational:OP179GRT
- added U5: TS5A4594, Package_TO_SOT_SMD:SOT-23-5_HandSoldering, symbol MLAB_IO:TS5A4594
- added U6: LM4041CIM3-1.2(neosazovat), Package_TO_SOT_SMD:SOT-23, symbol MLAB_D:LM4041CIM3-1.2
- D1: footprint (none) -> Mlab_D:Diode-SMA_Standard
- J1: value 0 ... Umax -> 3.6V; footprint (none) -> Mlab_Pin_Headers:Straight_2x03
- M1, M2, M3, M4: footprint (none) -> Mlab_Mechanical:MountingHole_3mm
Connections:
- net labels added: #PeakDetect/Trace, A, A/D, K, REF, VCC1, VCC2, VCC3, VCC4
- wire segments 27 -> 189
Other:
- note added: "CR2032"
- moved on the sheet: D1

Commit message: Edit
Parts:
- M5: value HOLE -> BMIS-209-C
- M6: value HOLE -> BMI-S-210-F
Changed lines of the file:
@@
 P 9850 1900
 F 0 "M6" V 9750 1900 60  0000 C CNN
-F 1 "HOLE" H 9850 1800 60  0001 C CNN
+F 1 "BMI-S-210-F" H 9850 1800 60  0001 C CNN
 F 2 "Mlab_Mechanical:BMI-S-210-F" H 9850 1900 60  0001 C CNN
 F 3 "" H 9850 1900 60  0000 C CNN
@@
 P 9650 1900
 F 0 "M5" V 9550 1900 60  0000 C CNN
-F 1 "HOLE" H 9650 1800 60  0001 C CNN
+F 1 "BMIS-209-C" H 9650 1800 60  0001 C CNN
 F 2 "Mlab_Mechanical:BMIS-209-C" H 9650 1900 60  0001 C CNN
 F 3 "" H 9650 1900 60  0000 C CNN

Commit message: edit
Parts:
- added C24, C25: EMI_Filter_C, Mlab_L:FIR1, symbol Device:EMI_Filter_C
- added R1: 10R, Mlab_R:SMD-0805, symbol Device:R
Connections:
- net GND: now also C24.2, C25.2
- net K: now also C24.3; no longer BT1.1 (+)
- net REF: now also C25.3; no longer BT1.2 (-)
- net at U2.6 (-), U2.7, U4.4 (-): now also R1.2; no longer C22.1
- new net: BT1.1 (+), C24.1
- new net: BT1.2 (-), C25.1
- new net: C22.1, R1.1
Other:
- moved on the sheet: BT1, C19, D2, R13, U2B
Changed lines of the file:
@@
 L MLAB_IO:AD8692 U2
 U 2 1 5B39C306
-P 9400 3800
-F 0 "U2" H 9500 3650 70  0000 L CNN
-F 1 "OPA2314" H 9400 3550 70  0000 L CNN
-F 2 "Mlab_IO:SOIC-8_3.9x4.9mm_Pitch1.27mm" H 9400 3800 60  0001 C CNN
-F 3 "" H 9941 3679 60  0000 L CNN
-	2    9400 3800
+P 9050 3800
+F 0 "U2" H 9150 3650 70  0000 L CNN
+F 1 "OPA2314" H 9050 3550 70  0000 L CNN
+F 2 "Mlab_IO:SOIC-8_3.9x4.9mm_Pitch1.27mm" H 9050 3800 60  0001 C CNN
+F 3 "" H 9591 3679 60  0000 L CNN
+	2    9050 3800
 	1    0    0    -1
 $EndComp
@@
 L Device:Battery_Cell BT1
 U 1 1 5B3A047F
-P 800 4800
-F 0 "BT1" H 550 4800 50  0000 L CNN
-F 1 "CH28-2032" H 200 4900 50  0000 L CNN
-F 2 "Mlab_Batery:CH28-2032" V 800 4860 50  0001 C CNN
-F 3 "~" V 800 4860 50  0001 C CNN
-	1    800  4800
+P 800 4600
+F 0 "BT1" H 950 4850 50  0000 L CNN
+F 1 "CH28-2032" H 650 4950 50  0000 L CNN
+F 2 "Mlab_Batery:CH28-2032" V 800 4660 50  0001 C CNN
+F 3 "~" V 800 4660 50  0001 C CNN
+	1    800  4600
 	-1   0    0    -1
 $EndComp
@@
 L Device:D_Photo D2
 U 1 1 5B3A05A5
-P 1250 4550
-F 0 "D2" H 1200 4845 50  0000 C CNN
-F 1 "D_Photo" H 1200 4754 50  0000 C CNN
-F 2 "Mlab_D:HAMAMATSU_S2744-09_rozs" H 1200 4550 50  0001 C CNN
-F 3 "~" H 1200 4550 50  0001 C CNN
-	1    1250 4550
-	1    0    0    -1
-$EndComp
-Wire Wire Line
-	800  4950 800  4900
-Wire Wire Line
-	800  4950 1050 4950
-Wire Wire Line
-	800  4600 800  4550
-Wire Wire Line
-	1900 4550 1900 4750
-Wire Wire Line
-	1050 4950 1050 5050
-Wire Wire Line
-	1050 5050 1150 5050
-Connection ~ 1050 4950
-Wire Wire Line
-	1050 4950 1750 4950
-Text Label 1150 5050 0    60   ~ 0
+P 1700 4350
+F 0 "D2" H 1650 4645 50  0000 C CNN
+F 1 "D_Photo" H 1650 4554 50  0000 C CNN
+F 2 "Mlab_D:HAMAMATSU_S2744-09_rozs" H 1650 4350 50  0001 C CNN
+F 3 "~" H 1650 4350 50  0001 C CNN
+	1    1700 4350
+	1    0    0    -1
+$EndComp
+Text Label 1550 5050 0    60   ~ 0
 REF
-Text Notes 700  4950 1    60   ~ 0
+Text Notes 700  4750 1    60   ~ 0
 CR2032
 $Comp
@@
 $EndComp
 Wire Wire Line
-	1900 4550 1900 4150
-Wire Wire Line
 	1900 4150 2250 4150
-Connection ~ 1900 4550
 Wire Wire Line
 	2250 3750 1900 3750
@@
 U 1 1 5B3B85BF
 P 7900 4400
-F 0 "U5" H 8000 4800 60  0000 L CNN
-F 1 "TS5A4594" H 8000 4700 60  0000 L CNN
+F 0 "U5" H 7400 4850 60  0000 L CNN
+F 1 "TS5A4594" H 7400 4750 60  0000 L CNN
 F 2 "Package_TO_SOT_SMD:SOT-23-5_HandSoldering" H 8300 5100 60  0001 C CNN
 F 3 "" H 8300 5100 60  0001 C CNN
@@
 Wire Wire Line
 	7350 4350 7350 3700
-Wire Wire Line
-	7350 3700 8200 3700
 $Comp
 L Device:R R13
 U 1 1 5B3BD0FF
-P 8350 3700
-F 0 "R13" V 8450 3650 50  0000 L CNN
-F 1 "2k2" V 8350 3700 50  0000 C CNN
-F 2 "Mlab_R:SMD-0805" V 8280 3700 50  0001 C CNN
-F 3 "~" H 8350 3700 50  0001 C CNN
-	1    8350 3700
+P 7650 3700
+F 0 "R13" V 7750 3650 50  0000 L CNN
+F 1 "2k2" V 7650 3700 50  0000 C CNN
+F 2 "Mlab_R:SMD-0805" V 7580 3700 50  0001 C CNN
+F 3 "~" H 7650 3700 50  0001 C CNN
+	1    7650 3700
 	0    1    1    0
 $EndComp
@@
 L Device:C C19
 U 1 1 5B3BD161
-P 8600 3900
-F 0 "C19" H 8715 3946 50  0000 L CNN
-F 1 "1nF" H 8715 3855 50  0000 L CNN
-F 2 "Mlab_R:SMD-0805" H 8638 3750 50  0001 C CNN
-F 3 "~" H 8600 3900 50  0001 C CNN
-	1    8600 3900
-	1    0    0    -1
-$EndComp
-Wire Wire Line
-	8500 3700 8600 3700
+P 8250 3900
+F 0 "C19" H 8365 3946 50  0000 L CNN
+F 1 "1nF" H 8365 3855 50  0000 L CNN
+F 2 "Mlab_R:SMD-0805" H 8288 3750 50  0001 C CNN
+F 3 "~" H 8250 3900 50  0001 C CNN
+	1    8250 3900
+	1    0    0    -1
+$EndComp
 Text Label 3350 5300 0    60   ~ 0
 REF
@@
 	1    0    0    -1
 $EndComp
-Wire Wire Line
-	8600 3750 8600 3700
-Connection ~ 8600 3700
-Wire Wire Line
-	8600 3700 8900 3700
 $Comp
 L power:GND #PWR012
 U 1 1 5B41D3E4
-P 8600 4100
-F 0 "#PWR012" H 8600 3850 50  0001 C CNN
-F 1 "GND" H 8605 3927 50  0000 C CNN
-F 2 "" H 8600 4100 50  0001 C CNN
-F 3 "" H 8600 4100 50  0001 C CNN
-	1    8600 4100
-	1    0    0    -1
-$EndComp
-Wire Wire Line
-	8600 4100 8600 4050
-Wire Wire Line
-	9300 3400 9300 3300
-Text Label 9300 3300 0    60   ~ 0
+P 8250 4100
+F 0 "#PWR012" H 8250 3850 50  0001 C CNN
+F 1 "GND" H 8255 3927 50  0000 C CNN
+F 2 "" H 8250 4100 50  0001 C CNN
+F 3 "" H 8250 4100 50  0001 C CNN
+	1    8250 4100
+	1    0    0    -1
+$EndComp
+Wire Wire Line
+	8950 3400 8950 3300
+Text Label 8950 3300 0    60   ~ 0
 VCC2
 $Comp
 L power:GND #PWR013
 U 1 1 5B424852
-P 9300 4250
-F 0 "#PWR013" H 9300 4000 50  0001 C CNN
-F 1 "GND" H 9305 4077 50  0000 C CNN
-F 2 "" H 9300 4250 50  0001 C CNN
-F 3 "" H 9300 4250 50  0001 C CNN
-	1    9300 4250
-	1    0    0    -1
-$EndComp
-Wire Wire Line
-	9300 4250 9300 4200
-Wire Wire Line
-	8900 3900 8900 4500
+P 8950 4250
+F 0 "#PWR013" H 8950 4000 50  0001 C CNN
+F 1 "GND" H 8955 4077 50  0000 C CNN
+F 2 "" H 8950 4250 50  0001 C CNN
+F 3 "" H 8950 4250 50  0001 C CNN
+	1    8950 4250
+	1    0    0    -1
+$EndComp
+Wire Wire Line
+	8950 4250 8950 4200
+Wire Wire Line
+	8550 3900 8550 4500
 Wire Wire Line
 	6850 5900 6850 5250
@@
 Connection ~ 10650 5250
 Wire Wire Line
-	9900 3800 9950 3800
-Text Label 10450 3800 0    60   ~ 0
+	9550 3800 9600 3800
+Text Label 10600 3800 1    60   ~ 0
 A/D
 Wire Wire Line
-	9950 3800 9950 4500
-Wire Wire Line
-	9950 4500 8900 4500
-Connection ~ 8900 4500
-Wire Wire Line
-	8900 4500 8900 5900
+	9600 3800 9600 4500
+Wire Wire Line
+	9600 4500 8550 4500
+Connection ~ 8550 4500
+Wire Wire Line
+	8550 4500 8550 5900
 $Comp
 L power:VCC #PWR015
@@
 	1    0    0    -1
 $EndComp
-Text Label 1500 4550 2    60   ~ 0
+Text Label 1850 4350 2    60   ~ 0
 A
-Text Label 850  4550 0    60   ~ 0
+Text Label 1450 4350 0    60   ~ 0
 K
 $Comp
@@
 $EndComp
 Wire Wire Line
-	8900 5900 6850 5900
-Wire Wire Line
 	6750 4450 7450 4450
 Wire Wire Line
 	7900 4900 7900 4850
 Wire Wire Line
-	9950 3800 10050 3800
-Connection ~ 9950 3800
+	9600 3800 9700 3800
+Connection ~ 9600 3800
 $Comp
 L power:GND #PWR027
@@
 Wire Wire Line
 	10250 4250 10250 4000
-Wire Wire Line
-	10450 3800 10700 3800
 $Comp
 L Device:EMI_Filter_C C2
@@
 Wire Wire Line
 	9600 1050 9750 1050
-Wire Wire Line
-	1350 4550 1900 4550
-Wire Wire Line
-	800  4550 1050 4550
+$Comp
+L Device:R R1
+U 1 1 5B690004
+P 9850 3800
+F 0 "R1" V 9950 3750 50  0000 L CNN
+F 1 "10R" V 9850 3800 50  0000 C CNN
+F 2 "Mlab_R:SMD-0805" V 9780 3800 50  0001 C CNN
+F 3 "~" H 9850 3800 50  0001 C CNN
+	1    9850 3800
+	0    1    1    0
+$EndComp
+Wire Wire Line
+	8250 4100 8250 4050
+Wire Wire Line
+	7350 3700 7500 3700
+Wire Wire Line
+	7800 3700 8250 3700
+Wire Wire Line
+	8250 3700 8250 3750
+Wire Wire Line
+	8550 5900 6850 5900
+Wire Wire Line
+	8250 3700 8550 3700
+Connection ~ 8250 3700
+Wire Wire Line
+	10000 3800 10050 3800
+Wire Wire Line
+	10450 3800 10700 3800
+$Comp
+L Device:EMI_Filter_C C24
+U 1 1 5B6E701C
+P 1200 4450
+F 0 "C24" H 1200 4755 50  0000 C CNN
+F 1 "EMI_Filter_C" H 1200 4664 50  0000 C CNN
+F 2 "Mlab_L:FIR1" V 1200 4450 50  0001 C CNN
+F 3 "http://www.murata.com/~/media/webrenewal/support/library/catalog/products/emc/emifil/c31e.ashx?la=en-gb" V 1200 4450 50  0001 C CNN
+	1    1200 4450
+	1    0    0    -1
+$EndComp
+Wire Wire Line
+	1500 4950 1500 5050
+Wire Wire Line
+	1500 5050 1550 5050
+Wire Wire Line
+	1500 4950 1750 4950
+$Comp
+L Device:EMI_Filter_C C25
+U 1 1 5B6FB081
+P 1200 5050
+F 0 "C25" H 900 5050 50  0000 C CNN
+F 1 "EMI_Filter_C" H 850 4950 50  0000 C CNN
+F 2 "Mlab_L:FIR1" V 1200 5050 50  0001 C CNN
+F 3 "http://www.murata.com/~/media/webrenewal/support/library/catalog/products/emc/emifil/c31e.ashx?la=en-gb" V 1200 5050 50  0001 C CNN
+	1    1200 5050
+	1    0    0    -1
+$EndComp
+Wire Wire Line
+	1400 4950 1500 4950
+Connection ~ 1500 4950
+Wire Wire Line
+	800  4950 1000 4950
+Wire Wire Line
+	800  4400 800  4350
+Wire Wire Line
+	800  4350 1000 4350
+Wire Wire Line
+	1400 4350 1500 4350
+$Comp
+L power:GND #PWR0105
+U 1 1 5B722886
+P 1200 5200
+F 0 "#PWR0105" H 1200 4950 50  0001 C CNN
+F 1 "GND" H 1205 5027 50  0000 C CNN
+F 2 "" H 1200 5200 50  0001 C CNN
+F 3 "" H 1200 5200 50  0001 C CNN
+	1    1200 5200
+	1    0    0    -1
+$EndComp
+Wire Wire Line
+	1900 4150 1900 4350
+Wire Wire Line
+	1800 4350 1900 4350
+Connection ~ 1900 4350
+Wire Wire Line
+	1900 4350 1900 4750
+Wire Wire Line
+	1200 4600 1200 4550
+Wire Wire Line
+	800  4700 800  4950
+Wire Wire Line
+	1200 5200 1200 5150
+$Comp
+L power:GND #PWR0106
+U 1 1 5B75FEF8
+P 1200 4600
+F 0 "#PWR0106" H 1200 4350 50  0001 C CNN
+F 1 "GND" H 1205 4427 50  0000 C CNN
+F 2 "" H 1200 4600 50  0001 C CNN
+F 3 "" H 1200 4600 50  0001 C CNN
+	1    1200 4600
+	1    0    0    -1
+$EndComp
 $EndSCHEMATC

Commit message: edit
Parts:
- C19: value 1nF -> 1nF/NP0
- C2, C22: value EMI_Filter_C -> NFM21CC221R1H3D-220pF
- C21, C23, C24, C25: value EMI_Filter_C -> NFM21PC105-1uF
- C5: value 1pF - 251R15S1R0AV4E -> 1pFNP0 251R15S1R0AV4E
- D2: value D_Photo -> S2744-09
- R9: value 15k -> 4k7
Changed lines of the file:
@@
 U 1 1 5B3A047F
 P 800 4600
-F 0 "BT1" H 950 4850 50  0000 L CNN
-F 1 "CH28-2032" H 650 4950 50  0000 L CNN
+F 0 "BT1" V 950 4300 50  0000 L CNN
+F 1 "CH28-2032" V 1050 4300 50  0000 L CNN
 F 2 "Mlab_Batery:CH28-2032" V 800 4660 50  0001 C CNN
 F 3 "~" V 800 4660 50  0001 C CNN
@@
 P 1700 4350
 F 0 "D2" H 1650 4645 50  0000 C CNN
-F 1 "D_Photo" H 1650 4554 50  0000 C CNN
+F 1 "S2744-09" H 1650 4554 50  0000 C CNN
 F 2 "Mlab_D:HAMAMATSU_S2744-09_rozs" H 1650 4350 50  0001 C CNN
 F 3 "~" H 1650 4350 50  0001 C CNN
@@
 P 2400 4150
 F 0 "C5" V 2148 4150 50  0000 C CNN
-F 1 "1pF - 251R15S1R0AV4E" V 2239 4150 50  0000 C CNN
+F 1 "1pFNP0 251R15S1R0AV4E" V 2250 4150 50  0000 C CNN
 F 2 "Mlab_R:SMD-0805" H 2438 4000 50  0001 C CNN
 F 3 "~" H 2400 4150 50  0001 C CNN
@@
 P 4150 5700
 F 0 "R9" V 4250 5650 50  0000 L CNN
-F 1 "15k" V 4150 5700 50  0000 C CNN
+F 1 "4k7" V 4150 5700 50  0000 C CNN
 F 2 "Mlab_R:SMD-0805" V 4080 5700 50  0001 C CNN
 F 3 "~" H 4150 5700 50  0001 C CNN
@@
 U 1 1 5B3BD161
 P 8250 3900
-F 0 "C19" H 8365 3946 50  0000 L CNN
-F 1 "1nF" H 8365 3855 50  0000 L CNN
+F 0 "C19" V 8350 3700 50  0000 L CNN
+F 1 "1nF/NP0" V 8450 3700 50  0000 L CNN
 F 2 "Mlab_R:SMD-0805" H 8288 3750 50  0001 C CNN
 F 3 "~" H 8250 3900 50  0001 C CNN
@@
 P 9950 1150
 F 0 "C21" H 9950 1455 50  0000 C CNN
-F 1 "EMI_Filter_C" H 9950 1364 50  0000 C CNN
+F 1 "NFM21PC105-1uF" H 9850 1350 50  0000 C CNN
 F 2 "Mlab_L:FIR1" V 9950 1150 50  0001 C CNN
 F 3 "http://www.murata.com/~/media/webrenewal/support/library/catalog/products/emc/emifil/c31e.ashx?la=en-gb" V 9950 1150 50  0001 C CNN
@@
 P 10250 3900
 F 0 "C22" H 10250 4205 50  0000 C CNN
-F 1 "EMI_Filter_C" H 10250 4114 50  0000 C CNN
+F 1 "NFM21CC221R1H3D-220pF" H 9900 4100 50  0000 C CNN
 F 2 "Mlab_L:FIR1" V 10250 3900 50  0001 C CNN
 F 3 "http://www.murata.com/~/media/webrenewal/support/library/catalog/products/emc/emifil/c31e.ashx?la=en-gb" V 10250 3900 50  0001 C CNN
@@
 P 9300 5250
 F 0 "C2" H 9300 5555 50  0000 C CNN
-F 1 "EMI_Filter_C" H 9300 5464 50  0000 C CNN
+F 1 "NFM21CC221R1H3D-220pF" H 9300 5464 50  0000 C CNN
 F 2 "Mlab_L:FIR1" V 9300 5250 50  0001 C CNN
 F 3 "http://www.murata.com/~/media/webrenewal/support/library/catalog/products/emc/emifil/c31e.ashx?la=en-gb" V 9300 5250 50  0001 C CNN
@@
 P 10350 5850
 F 0 "C23" H 10350 6155 50  0000 C CNN
-F 1 "EMI_Filter_C" H 10350 6064 50  0000 C CNN
+F 1 "NFM21PC105-1uF" H 10350 6064 50  0000 C CNN
 F 2 "Mlab_L:FIR1" V 10350 5850 50  0001 C CNN
 F 3 "http://www.murata.com/~/media/webrenewal/support/library/catalog/products/emc/emifil/c31e.ashx?la=en-gb" V 10350 5850 50  0001 C CNN
@@
 P 1200 4450
 F 0 "C24" H 1200 4755 50  0000 C CNN
-F 1 "EMI_Filter_C" H 1200 4664 50  0000 C CNN
+F 1 "NFM21PC105-1uF" H 1000 4650 50  0000 C CNN
 F 2 "Mlab_L:FIR1" V 1200 4450 50  0001 C CNN
 F 3 "http://www.murata.com/~/media/webrenewal/support/library/catalog/products/emc/emifil/c31e.ashx?la=en-gb" V 1200 4450 50  0001 C CNN
@@
 P 1200 5050
 F 0 "C25" H 900 5050 50  0000 C CNN
-F 1 "EMI_Filter_C" H 850 4950 50  0000 C CNN
+F 1 "NFM21PC105-1uF" H 850 4950 50  0000 C CNN
 F 2 "Mlab_L:FIR1" V 1200 5050 50  0001 C CNN
 F 3 "http://www.murata.com/~/media/webrenewal/support/library/catalog/products/emc/emifil/c31e.ashx?la=en-gb" V 1200 5050 50  0001 C CNN
