File: sensors/CCP2019V01A/hw/sch_pcb/CCP2019V01A.sch (KiCad schematic (older format))
At the start: 8 parts, among them J1 JUMP_3X2, M1 HOLE, M2 HOLE, M3 HOLE, M4 HOLE

Commit message: edit
Parts:
- removed C1: 10uF, Mlab_R:SMD-0805, symbol Device:CP_Small
- removed C2: 100nF, Mlab_R:SMD-0805, symbol Device:C_Small
- removed D1: 0.0V, Mlab_D:Diode-MiniMELF_Standard, symbol MLAB_D:D_ZENER
- removed J1: JUMP_3X2, Mlab_Pin_Headers:Straight_2x03, symbol MLAB_Jumpers:JUMP_3X2
- added C1: 47uF, Mlab_C:TantalC_SizeC_Reflow, symbol Device:CP
- added C10, C11, C12, C13, C14, C16, C20: 100nF, Mlab_R:SMD-0805, symbol Device:C
- added C15: 3n3, Mlab_R:SMD-0805, symbol Device:C
- added C17, C3: 4u7, Mlab_R:SMD-0805, symbol Device:C
- added C18: 2n2, Mlab_R:SMD-0805, symbol Device:C
- added C19: 1nF/NP0, Mlab_R:SMD-0805, symbol Device:C
- added C2, C22: NFM21CC221R1H3D-220pF, Mlab_L:FIR1, symbol Device:EMI_Filter_C
- added C21, C23, C4, C6, C7, C8, C9: 10uF, Mlab_R:SMD-0805, symbol Device:C
- added C24: 1uF, Mlab_R:SMD-0805, symbol Device:C
- added C5: 1pFNP0 251R15S1R0AV4E, Mlab_R:SMD-0805, symbol Device:C
- added D2: S2744-09, Mlab_D:HAMAMATSU_S2744-09_rozs, symbol Device:D_Photo
- added M5: BMIS-209-C, Mlab_Mechanical:BMIS-209-C, symbol MLAB_MECHANICAL:HOLE
- added M6: BMI-S-210-F, Mlab_Mechanical:BMI-S-210-F, symbol MLAB_MECHANICAL:HOLE
- added R1: 10R, Mlab_R:SMD-0805, symbol Device:R
- added R10, R8: 1k, Mlab_R:SMD-0805, symbol Device:R
- added R11, R15, R19, R22, R9: 4k7, Mlab_R:SMD-0805, symbol Device:R
- added R12, R7: 10k, Mlab_R:SMD-0805, symbol Device:R
- added R13: 2k2, Mlab_R:SMD-0805, symbol Device:R
- added R2, R3, R4, R5: 470R, Mlab_R:SMD-0805, symbol Device:R
- added R6: 10M, Mlab_R:SMD-0805, symbol Device:R
- added U1, U2: OPA2314, Mlab_IO:SOIC-8_3.9x4.9mm_Pitch1.27mm, symbol MLAB_IO:AD8692
- added U3: ISL21080DIH312Z-TK 1V25, Package_TO_SOT_SMD:SOT-23, symbol Reference_Voltage:ISL21070CIH320Z-TK
- added U4: TS7211, Package_TO_SOT_SMD:SOT-23-5_HandSoldering, symbol Amplifier_Operational:OP179GRT
- added U5: TS5A4594, Package_TO_SOT_SMD:SOT-23-5_HandSoldering, symbol MLAB_IO:TS5A4594
Connections:
- net labels added: #PeakDetect/Trace, +3.3V, +5V, A, A/D, K, PA0, PA1, REF, Ubiasout, VCC1, VCC2, VCC3, VCC4
- net labels removed: VCC
- wire segments 25 -> 169
Other:
- note removed: "POWER INPUT"
- moved on the sheet: M2

Commit message: edit
Connections:
- net A/D renamed PA0
Changed lines of the file:
@@
 F1 "power.sch" 60
 $EndSheet
-Text Label 10700 3800 0    60   ~ 0
-PA0
-Text Label 10550 5600 0    60   ~ 0
-PA1
 Text Label 10300 5600 0    60   ~ 0
 REF
 Wire Wire Line
 	10300 5600 10550 5600
+Text GLabel 10700 3800 2    60   Input ~ 0
+PA0
+Text GLabel 10550 5600 2    60   Input ~ 0
+PA1
 $EndSCHEMATC

Commit message: edit
Parts:
- removed C2, C22: NFM21CC221R1H3D-220pF, Mlab_L:FIR1, symbol Device:EMI_Filter_C
- removed M5: BMIS-209-C, Mlab_Mechanical:BMIS-209-C, symbol MLAB_MECHANICAL:HOLE
- added C2: 100nF, Mlab_R:SMD-0805, symbol Device:C
- added M7: BMI-S-210-F, Mlab_Mechanical:BMI-S-210-F, symbol MLAB_MECHANICAL:HOLE
- D2: footprint Mlab_D:HAMAMATSU_S2744-09_rozs -> Mlab_D:HAMAMATSU_S2744-09
Connections:
- net GND: now also C2.2, M7.1
- net PA0: now also R1.1
- net at C23.1, R19.1, R22.2: now also C2.1
Other:
- moved on the sheet: C24, R22
Changed lines of the file:
@@
 EESchema Schematic File Version 4
 LIBS:CCP2019V01A-cache
-EELAYER 26 0
+EELAYER 29 0
 EELAYER END
 $Descr A4 11693 8268
@@
 F 0 "D2" H 1650 4645 50  0000 C CNN
 F 1 "S2744-09" H 1650 4554 50  0000 C CNN
-F 2 "Mlab_D:HAMAMATSU_S2744-09_rozs" H 1650 4350 50  0001 C CNN
+F 2 "Mlab_D:HAMAMATSU_S2744-09" H 1650 4350 50  0001 C CNN
 F 3 "~" H 1650 4350 50  0001 C CNN
 	1    1700 4350
@@
 Wire Wire Line
 	7100 5650 7100 5450
-Text Label 9750 5150 0    60   ~ 0
-#PeakDetect/Trace
 Wire Wire Line
 	7500 5150 7550 5150
@@
 Wire Notes Line
 	9700 1000 11100 1000
-$Comp
-L MLAB_MECHANICAL:HOLE M5
-U 1 1 5B69B79B
-P 9800 750
-F 0 "M5" V 9700 750 60  0000 C CNN
-F 1 "BMIS-209-C" H 9800 650 60  0001 C CNN
-F 2 "Mlab_Mechanical:BMIS-209-C" H 9800 750 60  0001 C CNN
-F 3 "" H 9800 750 60  0000 C CNN
-	1    9800 750
-	0    -1   -1   0
-$EndComp
-Wire Wire Line
-	10000 650  9800 650
-Wire Wire Line
-	9800 650  9800 700
 Connection ~ 10000 650
-$Comp
-L Device:EMI_Filter_C C22
-U 1 1 5B6C4183
-P 10250 3900
-F 0 "C22" H 10250 4205 50  0000 C CNN
-F 1 "NFM21CC221R1H3D-220pF" H 9900 4100 50  0000 C CNN
-F 2 "Mlab_L:FIR1" V 10250 3900 50  0001 C CNN
-F 3 "http://www.murata.com/~/media/webrenewal/support/library/catalog/products/emc/emifil/c31e.ashx?la=en-gb" V 10250 3900 50  0001 C CNN
-	1    10250 3900
-	1    0    0    -1
-$EndComp
 Wire Wire Line
 	6750 4450 7450 4450
@@
 	9600 3800 9700 3800
 Connection ~ 9600 3800
-$Comp
-L power:GND #PWR027
-U 1 1 5B6ED0AF
-P 10250 4250
-F 0 "#PWR027" H 10250 4000 50  0001 C CNN
-F 1 "GND" H 10255 4077 50  0000 C CNN
-F 2 "" H 10250 4250 50  0001 C CNN
-F 3 "" H 10250 4250 50  0001 C CNN
-	1    10250 4250
-	1    0    0    -1
-$EndComp
-Wire Wire Line
-	10250 4250 10250 4000
-$Comp
-L Device:EMI_Filter_C C2
-U 1 1 5B729EB5
-P 9300 5250
-F 0 "C2" H 9300 5555 50  0000 C CNN
-F 1 "NFM21CC221R1H3D-220pF" H 9300 5464 50  0000 C CNN
-F 2 "Mlab_L:FIR1" V 9300 5250 50  0001 C CNN
-F 3 "http://www.murata.com/~/media/webrenewal/support/library/catalog/products/emc/emifil/c31e.ashx?la=en-gb" V 9300 5250 50  0001 C CNN
-	1    9300 5250
-	1    0    0    -1
-$EndComp
-Wire Wire Line
-	8350 5150 9100 5150
-Connection ~ 8350 5150
-Wire Wire Line
-	9500 5150 10700 5150
-$Comp
-L power:GND #PWR028
-U 1 1 5B73E3FB
-P 9300 5400
-F 0 "#PWR028" H 9300 5150 50  0001 C CNN
-F 1 "GND" H 9305 5227 50  0000 C CNN
-F 2 "" H 9300 5400 50  0001 C CNN
-F 3 "" H 9300 5400 50  0001 C CNN
-	1    9300 5400
-	1    0    0    -1
-$EndComp
-Wire Wire Line
-	9300 5400 9300 5350
 $Comp
 L Device:R R1
@@
 Connection ~ 8250 3700
 Wire Wire Line
-	10000 3800 10050 3800
-Wire Wire Line
-	10450 3800 10700 3800
-Wire Wire Line
 	1500 4950 1750 4950
 Wire Wire Line
@@
 L Device:R R22
 U 1 1 5C61685E
-P 2000 6750
-F 0 "R22" V 2100 6700 50  0000 L CNN
-F 1 "4k7" V 2000 6750 50  0000 C CNN
-F 2 "Mlab_R:SMD-0805" V 1930 6750 50  0001 C CNN
-F 3 "~" H 2000 6750 50  0001 C CNN
-	1    2000 6750
+P 2600 6750
+F 0 "R22" V 2700 6700 50  0000 L CNN
+F 1 "4k7" V 2600 6750 50  0000 C CNN
+F 2 "Mlab_R:SMD-0805" V 2530 6750 50  0001 C CNN
+F 3 "~" H 2600 6750 50  0001 C CNN
+	1    2600 6750
 	0    1    1    0
 $EndComp
@@
 L Device:C C24
 U 1 1 5C616902
-P 2250 7000
-F 0 "C24" H 2365 7046 50  0000 L CNN
-F 1 "1uF" H 2365 6955 50  0000 L CNN
-F 2 "Mlab_R:SMD-0805" H 2288 6850 50  0001 C CNN
-F 3 "~" H 2250 7000 50  0001 C CNN
-	1    2250 7000
-	1    0    0    -1
-$EndComp
-Wire Wire Line
-	2150 6750 2250 6750
-Connection ~ 2250 6750
-Wire Wire Line
-	2250 6750 2450 6750
-Wire Wire Line
-	2250 6750 2250 6850
-Wire Wire Line
-	2250 7150 2450 7150
+P 2850 7000
+F 0 "C24" H 2965 7046 50  0000 L CNN
+F 1 "1uF" H 2965 6955 50  0000 L CNN
+F 2 "Mlab_R:SMD-0805" H 2888 6850 50  0001 C CNN
+F 3 "~" H 2850 7000 50  0001 C CNN
+	1    2850 7000
+	1    0    0    -1
+$EndComp
+Wire Wire Line
+	2750 6750 2850 6750
+Connection ~ 2850 6750
+Wire Wire Line
+	2850 6750 3050 6750
+Wire Wire Line
+	2850 6750 2850 6850
+Wire Wire Line
+	2850 7150 3050 7150
 Wire Wire Line
 	950  6750 1000 6750
@@
 	1750 6850 1750 6750
 Connection ~ 1750 6750
-Wire Wire Line
-	1750 6750 1850 6750
-Text Label 2450 6750 0    60   ~ 0
+Text Label 3050 6750 0    60   ~ 0
 Ubiasout
-Text Label 2450 7150 0    60   ~ 0
+Text Label 3050 7150 0    60   ~ 0
 REF
 Text Label 1000 4350 0    60   ~ 0
@@
 F1 "power.sch" 60
 $EndSheet
-Text Label 10300 5600 0    60   ~ 0
+Text Label 10450 4050 0    60   ~ 0
 REF
 Wire Wire Line
-	10300 5600 10550 5600
+	10450 4050 10700 4050
 Text GLabel 10700 3800 2    60   Input ~ 0
 PA0
-Text GLabel 10550 5600 2    60   Input ~ 0
+Text GLabel 10700 4050 2    60   Input ~ 0
 PA1
+Wire Wire Line
+	10000 3800 10700 3800
+$Comp
+L Device:C C2
+U 1 1 5C52C88C
+P 2200 7000
+F 0 "C2" H 2315 7046 50  0000 L CNN
+F 1 "100nF" H 2315 6955 50  0000 L CNN
+F 2 "Mlab_R:SMD-0805" H 2238 6850 50  0001 C CNN
+F 3 "" H 2200 7000 50  0001 C CNN
+	1    2200 7000
+	1    0    0    -1
+$EndComp
+Wire Wire Line
+	1750 6750 2200 6750
+Wire Wire Line
+	2200 6850 2200 6750
+Connection ~ 2200 6750
+Wire Wire Line
+	2200 6750 2450 6750
+$Comp
+L power:GND #PWR0119
+U 1 1 5C53D6D2
+P 2200 7200
+F 0 "#PWR0119" H 2200 6950 50  0001 C CNN
+F 1 "GND" H 2205 7027 50  0000 C CNN
+F 2 "" H 2200 7200 50  0001 C CNN
+F 3 "" H 2200 7200 50  0001 C CNN
+	1    2200 7200
+	1    0    0    -1
+$EndComp
+Wire Wire Line
+	2200 7200 2200 7150
+$Comp
+L MLAB_MECHANICAL:HOLE M7
+U 1 1 5C564E7A
+P 9600 750
+F 0 "M7" V 9500 750 60  0000 C CNN
+F 1 "BMI-S-210-F" H 9600 650 60  0001 C CNN
+F 2 "Mlab_Mechanical:BMI-S-210-F" H 9600 750 60  0001 C CNN
+F 3 "" H 9600 750 60  0000 C CNN
+	1    9600 750
+	0    -1   -1   0
+$EndComp
+Wire Wire Line
+	9600 650  9600 700
+Wire Wire Line
+	9600 650  10000 650
 $EndSCHEMATC
