File: sensors/CCP2019V01A/hw/sch_pcb/cpu.sch (KiCad schematic (older format))
At the start: 39 parts, among them J17 MCC-SD, J19 HEADER_2x01_PARALLEL, J22 HEADER_2x03, J29 HEADER_2x01_PARALLEL, J30 HEADER_2x01_PARALLEL, J42 HEADER_2x01_PARALLEL, U10 ATMEGA1284P-AU, U11 PCF85263A, U12 AT24CS64-SSHM, U7 ISL21080CIH320Z-TK, Y1 16MHz, Y2 ABS07-120-32.768KHZ-T

Commit message: edit
Parts:
- D4: footprint Mlab_D:FIX-LED-313 -> Mlab_D:LED_1206
Changed lines of the file:
@@
 Wire Wire Line
 	6850 1600 6950 1600
-Text Label 6950 1500 0    60   ~ 0
-PA0
-Text Label 6950 1600 0    60   ~ 0
-PA1
 Text Label 6950 2400 0    60   ~ 0
 PB0
@@
 F 0 "D4" H 9600 1550 50  0000 R CNN
 F 1 "HLMP-K150+FIX-LED-313" H 9800 1450 50  0000 R CNN
-F 2 "Mlab_D:FIX-LED-313" H 9650 1300 50  0001 C CNN
+F 2 "Mlab_D:LED_1206" H 9650 1300 50  0001 C CNN
 F 3 "~" H 9650 1300 50  0001 C CNN
 	1    9650 1300
@@
 Wire Wire Line
 	4050 800  4050 850
-Connection ~ 1650 6500
-Connection ~ 3450 6900
-Connection ~ 1650 6600
-Connection ~ 1650 6700
-Connection ~ 1650 6800
-Connection ~ 1650 6900
-Connection ~ 1650 7000
-Connection ~ 1650 7100
 Text Label 4600 1500 1    60   ~ 0
 RST#_P
@@
 	1    0    0    -1
 $EndComp
+Text GLabel 6950 1500 2    60   Input ~ 0
+PA0
+Text GLabel 6950 1600 2    60   Input ~ 0
+PA1
 $EndSCHEMATC

Commit message: edit
Parts:
- removed C29, C41, C46: 100nF, Mlab_R:SMD-0805, symbol CCP2019V01A-rescue:C-device-DATALOGGER01A-rescue
- removed C36: 10uF, Mlab_R:SMD-0805, symbol CCP2019V01A-rescue:C-device-DATALOGGER01A-rescue
- removed J17: MCC-SD, Connector_Card:SD_TE_2041021, symbol CCP2019V01A-rescue:SD_Card-Connector-DATALOGGER01A-rescue
- removed J29, J30, J42: HEADER_2x01_PARALLEL, Mlab_Pin_Headers:Straight_2x01, symbol MLAB_HEADER:HEADER_2x01_PARALLEL
- removed R14, R16, R17, R18: 100, Mlab_R:SMD-0805, symbol CCP2019V01A-rescue:R-device-DATALOGGER01A-rescue
- removed U12: AT24CS64-SSHM, Package_SO:SOIC-8_3.9x4.9mm_P1.27mm, symbol Memory_EEPROM:AT24CS64-SSHM
- removed U7: ISL21080CIH320Z-TK, Package_TO_SOT_SMD:SOT-23, symbol CCP2019V01A-rescue:ISL21070CIH320Z-TK-references-DATALOGGER01A-rescue
- added J4, J5, J6, J7: HEADER_1x01, Mlab_Pin_Headers:Straight_1x01, symbol MLAB_HEADER:HEADER_1x01
Connections:
- net VDD is gone; now on net +3V3: U11.3 (VBAT)
- net LED: now also U10.21 ((PCINT18/TCK)PC2); no longer U10.26 ((PCINT23/TOSC2)PC7)
- net RX0: now also J6.1
- net TX0: now also J7.1
- net PC3: now reaches U10.22 ((PCINT19/TMS)PC3)
- net PC3: now also J5.1
- net AREF: no longer names the net of C40.1, C44.1, U10.29 (AREF)
- net INTA: no longer names the net of U11.9 (INTA)
- net PB0: no longer names the net of U10.40 ((PCINT8/T0/XCK)PB0)
- net PB4: no longer names the net of U10.44 ((PCINT12/OC0B/~SS~)PB4)
- removed net SD_VDD: U10.41 ((PCINT9/CLKO/T1)PB1), U10.42 ((PCINT10/AIN0/INT2)PB2), U10.43 ((PCINT11/AIN1/OC0)PB3)
- new net PC7: J4.1, U10.26 ((PCINT23/TOSC2)PC7)
- no-connect marks 0 -> 23
