File: sensors/CCP2019V01A/hw/sch_pcb/power.sch (KiCad schematic (older format))
At the start: 21 parts, among them J1 HEADER_2x03_PARALLEL, U6 TPS613221ADBV, U8 TPS613222ADBV

Commit message: edit
Parts:
- removed BT1: BX0037, Mlab_Batery:BX0037, symbol CCP2019V01A-rescue:Battery_Cell-device-DATALOGGER01A-rescue
- removed C37: 47uF, Mlab_C:TantalC_SizeC_Reflow, symbol CCP2019V01A-rescue:CP-device-DATALOGGER01A-rescue
- removed J1: HEADER_2x03_PARALLEL, Mlab_Pin_Headers:Straight_2x03, symbol MLAB_HEADER:HEADER_2x03_PARALLEL
- added C22, C36: 10uF, Mlab_R:SMD-0805, symbol CCP2019V01A-rescue:C-device-DATALOGGER01A-rescue
- added C29: NFM21PC105-1uF, Mlab_L:FIR1, symbol CCP2019V01A-rescue:EMI_Filter_C-device-DATALOGGER01A-rescue
- added C55: 100nF, Mlab_R:SMD-0805, symbol CCP2019V01A-rescue:C-device-DATALOGGER01A-rescue
- added D3: BZV55C-5,6V, Diode_SMD:D_MiniMELF, symbol CCP2019V01A-rescue:D-device-DATALOGGER01A-rescue
- added F2: SR010-15 100mA, Mlab_R:SMD-0805, symbol CCP2019V01A-rescue:Polyfuse-device-DATALOGGER01A-rescue
- added J1, J2, J3: HEADER_2x01_PARALLEL, Mlab_Pin_Headers:Straight_1x02, symbol MLAB_HEADER:HEADER_2x01_PARALLEL
- added R24, R25, R27: -, Mlab_R:SMD-0805, symbol Device:R
- added R28: 0R, Mlab_R:SMD-0805, symbol Device:R
- D1: value M4 -> BZV55C-5,6V; footprint Mlab_D:Diode-SMA_Standard -> Diode_SMD:D_MiniMELF
- F1: value 750mA -> SR010-15 100mA; footprint Mlab_F:1812 -> Mlab_R:SMD-0805
Connections:
- net +3V3: now also R27.1
- net +5V: now also R25.1
- net GND: now also C22.2, C29.2, C36.2, C55.2, D3.2 (A), J2.1, J2.2
- net VDD: now also R28.1; no longer C45.3, C48.1
- net 5: now reaches F1.2
- net 5: now also J1.1, J1.2, R24.1
- net at C45.1, D1.1 (K), F1.1: now also C22.1
- new net: C29.1, C36.1, D3.1 (K), F2.1
- new net: C29.3, C55.1, R27.2
- new net: C45.3, C48.1, R25.2, R28.2
- new net 3: F2.2, J3.1, J3.2, R24.2
Other:
- note removed: "Batery"
- note removed: "IN Power"
- moved on the sheet: C25, C32, C38, C42, C45, C48, C49, C50, C51, C52, C53, C54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
