File: RF/ISM01A/hw/sch_pcb/ISM01A.sch (KiCad schematic (older format))
At the start: 8 parts, among them J1 JUMP_3X2, M1 HOLE, M2 HOLE, M3 HOLE, M4 HOLE

Commit message: Edit
Parts:
- removed C1: 10uF, Mlab_R:SMD-0805, symbol Device:CP_Small
- added C? (x6): 10uF, Mlab_R:SMD-0805, symbol Device:C_Small
- added C? (x3): 8,2pF, Mlab_R:SMD-0805, symbol Device:C_Small
- added C? (x2): 6.8pf, Mlab_R:SMD-0805, symbol Device:C_Small
- added C? (x2): 15pF, Mlab_R:SMD-0805, symbol Device:C_Small
- added C?: NFM21PC105, symbol Device:EMI_Filter_C
- added C?: 5.1pF, Mlab_R:SMD-0805, symbol Device:C_Small
- added C?: 2.7pF, Mlab_R:SMD-0805, symbol Device:C_Small
- added C?: 33pF, Mlab_R:SMD-0805, symbol Device:C_Small
- added C?: 100pF, Mlab_R:SMD-0805, symbol Device:C_Small
- added C? (x2): 100nF, Mlab_R:SMD-0805, symbol Device:C_Small
- added C?: 10nF, Mlab_R:SMD-0805, symbol Device:C_Small
- added J?: JUMP_3X2, Mlab_Pin_Headers:Straight_2x03, symbol MLAB_Jumpers:JUMP_3X2
- added J? (x2): SMA, symbol MLAB_CONNECTORS:SMA
- added J?: BMIS-210, symbol MLAB_Jumpers:CONN1_1
- added J? (x18): HEADER_2x01_PARALLEL, symbol MLAB_HEADER:HEADER_2x01_PARALLEL
- added L? (x2): 0R, symbol Device:L_Small
- added L? (x4): 18nH, symbol Device:L_Small
- added L?: 39nH, symbol Device:L_Small
- added L?: 220nH, symbol Device:L_Small
- added L? (x2): 56nH, symbol Device:L_Small
- added R? (x2): 0R, symbol Device:R
- added U?: Si1060-A-GM, symbol MLAB_IO:Si1060-A-GM
- added U?: LM1117, symbol MLAB_U:LM1117
- added Y?: ABS07-120-32.768KHZ, symbol Device:Crystal
- added Y?: ABM3B-30.000MHZ-10-1-U-T, symbol Device:Crystal_GND24
- D1: value 0.0V -> M4
Connections:
- net labels added: +3.3V, P0.6, P1.4, P1.5, P1.6, P2.7C2D, RX, TX
- wire segments 25 -> 144
Other:
- note added: "RF Shield"
- note added: "SBIT(LED_RED, SFR_P1, 6);\nSBIT(LED_GREEN, SFR_P1, 5);\n"

Commit message: edit
Parts:
- added C22, C23, C25, C26, C27, C28: 10nF, Mlab_R:SMD-0805, symbol Device:C_Small
- added D2, D3: LED, Mlab_D:LED_1206, symbol Device:LED
- added R10, R11, R12, R13, R14, R15, R16, R17, R18, R19, R2, R3, R4, R5, R6, R7, R8, R9: 33R, Mlab_R:SMD-0805, symbol Device:R
- added R20: 1k, Mlab_R:SMD-0805, symbol Device:R
- added R22, R23: 200R, Mlab_R:SMD-0805, symbol Device:R
- C21: renamed from C?; footprint (none) -> Mlab_L:FIR1
- J10, J11, J12, J13, J14, J15, J16, J17, J18, J19, J20, J21, J22, J23, J6, J7, J8, J9: renamed from J?; footprint (none) -> Mlab_Pin_Headers:Straight_2x01
- J2, J3: renamed from J?; footprint (none) -> Mlab_CON:SMA6251A13G50
- J5: renamed from J?; footprint (none) -> Mlab_Mechanical:BMI-S-210-F
- L1, L10, L2, L3, L4, L5, L6, L7, L8, L9: renamed from L?; footprint (none) -> Mlab_R:SMD-0805
- R1, R21: renamed from R?; footprint (none) -> Mlab_R:SMD-0805
- U1: renamed from U?; footprint (none) -> Mlab_IO:SOT-223
- U2: renamed from U?; footprint (none) -> Package_DFN_QFN:QFN-36-1EP_5x6mm_P0.5mm_EP3.6x4.1mm
- Y1: renamed from Y?; footprint (none) -> Mlab_XTAL:ABS07
- Y2: renamed from Y?; footprint (none) -> Crystal:Crystal_SMD_Abracon_ABM3B-4Pin_5.0x3.2mm
- gave numbers to parts that had none: 21
Connections:
- net +3V3: now also R20.1
- net GND: now also C22.2, C23.2, C25.2, C26.2, C27.2, C28.2
- net P0.6: now also R6.1; no longer U2.24 (P0.6/CNVSTR)
- net P1.4: now also R5.1; no longer U2.6 (P1.4)
- net P1.5: now also R4.1; no longer U2.5 (P1.5)
- net P1.6: now also R3.1; no longer U2.4 (P1.6)
- net P2.7C2D: now also R2.1; no longer U2.1 (P2.7/C2D)
- net RX: now also C27.1, R7.1; no longer U2.25 (P0.5/RX)
- net TX: now also C28.1, R8.1; no longer U2.26 (P0.4/TX)
- net GPIO2: now reaches J22.1, J22.2
- net GPIO2: now also C25.1, R18.1; no longer U2.10 (GPIO2)
- net GPIO3: now reaches J23.1, J23.2
- net GPIO3: now also C26.1, R19.1; no longer U2.11 (GPIO3)
- net TXRAMP: now reaches J17.1, J17.2
- net TXRAMP: now also R13.1; no longer U2.19 (TXRAMP)
- net GPIO0: now reaches J20.1, J20.2
- net GPIO0: now also C22.1, R16.1; no longer U2.21 (GPIO0)
- net GPIO1: now reaches J21.1, J21.2
- net GPIO1: now also C23.1, R17.1; no longer U2.22 (GPIO1)
- net #IRQ: now reaches J19.1, J19.2
- net #IRQ: now also R21.1, R15.1; no longer U2.23 (#IRQ)
- net P0.3: now reaches J13.1, J13.2
- net P0.3: now also R9.1; no longer U2.27 (P0.3/XTAL2)
- net P0.2: now reaches J14.1, J14.2
- net P0.2: now also R10.1; no longer U2.28 (P0.2/XTAL1)
- net P0.1: now reaches J15.1, J15.2
- net P0.1: now also R21.2, R11.1; no longer U2.29 (P0.1/AGND)
- net P0.0: now reaches J16.1, J16.2
- net P0.0: now also R12.1; no longer U2.30 (P0.0/VREF)
- net #RST_C2CK: now reaches J18.1, J18.2
- net #RST_C2CK: now also R14.1, R20.2; no longer U2.36 (#RST/C2CK)
- new net: R2.2, U2.1 (P2.7/C2D)
- new net: R18.2, U2.10 (GPIO2)
- new net: R19.2, U2.11 (GPIO3)
- new net: R13.2, U2.19 (TXRAMP)
- new net: R16.2, U2.21 (GPIO0)
- new net: R17.2, U2.22 (GPIO1)
- new net: R15.2, U2.23 (#IRQ)
- new net: R6.2, U2.24 (P0.6/CNVSTR)
- new net: R7.2, U2.25 (P0.5/RX)
- new net: R8.2, U2.26 (P0.4/TX)
- new net: R9.2, U2.27 (P0.3/XTAL2)
- new net: R10.2, U2.28 (P0.2/XTAL1)
- new net: R11.2, U2.29 (P0.1/AGND)
- new net: R12.2, U2.30 (P0.0/VREF)
- new net: R14.2, U2.36 (#RST/C2CK)
- new net: R3.2, U2.4 (P1.6)
- new net: R4.2, U2.5 (P1.5)
- new net: R5.2, U2.6 (P1.4)
Other:
- moved on the sheet: J10, J11, J12, J13, J14, J15, J16, J17, J18, J19, J20, J21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

Commit message: edit
Parts:
- U2: footprint Package_DFN_QFN:QFN-36-1EP_5x6mm_P0.5mm_EP3.6x4.1mm -> Package_DFN_QFN:QFN-36-1EP_5x6mm_P0.5mm_EP3.6x4.1mm_ThermalVias
Changed lines of the file:
@@
 F 0 "U2" H 4600 2850 60  0000 C CNN
 F 1 "Si1060-A-GM" H 4700 2700 60  0000 C CNN
-F 2 "Package_DFN_QFN:QFN-36-1EP_5x6mm_P0.5mm_EP3.6x4.1mm" H 4550 4100 60  0001 C CNN
+F 2 "Package_DFN_QFN:QFN-36-1EP_5x6mm_P0.5mm_EP3.6x4.1mm_ThermalVias" H 4550 4100 60  0001 C CNN
 F 3 "" H 4550 4100 60  0001 C CNN
 	1    4850 3650

Commit message: edit
Parts:
- added J24, J25: HEADER_1x02, Mlab_Pin_Headers:Straight_1x02, symbol MLAB_HEADER:HEADER_1x02
- added Q1, Q2: BC817, Package_TO_SOT_SMD:SOT-23, symbol Device:Q_NPN_BEC
- D2: value LED -> RED
- D3: value LED -> GREEN
- R22, R23: value 200R -> 150R
Connections:
- net +3V3: now also D2.2 (A), D3.2 (A)
- net GND: now also Q1.2 (E), Q2.2 (E)
- net P1.4: now also J24.2
- net P1.5: now also J25.2
- net at D2.1 (K): now also R22.1
- net at D3.1 (K): now also R23.1
- net at R22.2: now also Q1.3 (C)
- net at R23.2: now also Q2.3 (C)
- new net: J24.1, Q1.1 (B)
- new net: J25.1, Q2.1 (B)
Other:
- note removed: "SBIT(LED_RED, SFR_P1, 6);\nSBIT(LED_GREEN, SFR_P1, 5);\n"
- moved on the sheet: D2, D3, R22, R23
Changed lines of the file:
@@
 	3050 2350 3350 2350
 Connection ~ 3350 2350
-Text Notes 8050 3600 0    60   ~ 0
-SBIT(LED_RED,	SFR_P1, 6);\nSBIT(LED_GREEN,	SFR_P1, 5);\n
 $Comp
 L Device:C_Small C15
@@
 L Device:LED D2
 U 1 1 5C1996B5
-P 9900 3550
-F 0 "D2" V 9845 3628 50  0000 L CNN
-F 1 "LED" V 9936 3628 50  0000 L CNN
-F 2 "Mlab_D:LED_1206" H 9900 3550 50  0001 C CNN
-F 3 "~" H 9900 3550 50  0001 C CNN
-	1    9900 3550
-	0    1    1    0
+P 9550 3250
+F 0 "D2" V 9495 3328 50  0000 L CNN
+F 1 "RED" V 9586 3328 50  0000 L CNN
+F 2 "Mlab_D:LED_1206" H 9550 3250 50  0001 C CNN
+F 3 "~" H 9550 3250 50  0001 C CNN
+	1    9550 3250
+	0    -1   -1   0
 $EndComp
 $Comp
 L Device:LED D3
 U 1 1 5C199C16
-P 10300 3550
-F 0 "D3" V 10245 3628 50  0000 L CNN
-F 1 "LED" V 10336 3628 50  0000 L CNN
-F 2 "Mlab_D:LED_1206" H 10300 3550 50  0001 C CNN
-F 3 "~" H 10300 3550 50  0001 C CNN
-	1    10300 3550
-	0    1    1    0
+P 10800 3250
+F 0 "D3" V 10745 3328 50  0000 L CNN
+F 1 "GREEN" V 10836 3328 50  0000 L CNN
+F 2 "Mlab_D:LED_1206" H 10800 3250 50  0001 C CNN
+F 3 "~" H 10800 3250 50  0001 C CNN
+	1    10800 3250
+	0    -1   -1   0
 $EndComp
 $Comp
 L Device:R R22
 U 1 1 5C199F7B
-P 9900 3100
-F 0 "R22" H 9970 3146 50  0000 L CNN
-F 1 "200R" H 9970 3055 50  0000 L CNN
-F 2 "Mlab_R:SMD-0805" V 9830 3100 50  0001 C CNN
-F 3 "~" H 9900 3100 50  0001 C CNN
-	1    9900 3100
+P 9550 3650
+F 0 "R22" H 9620 3696 50  0000 L CNN
+F 1 "150R" H 9620 3605 50  0000 L CNN
+F 2 "Mlab_R:SMD-0805" V 9480 3650 50  0001 C CNN
+F 3 "~" H 9550 3650 50  0001 C CNN
+	1    9550 3650
 	1    0    0    -1
 $EndComp
@@
 L Device:R R23
 U 1 1 5C19A40D
-P 10300 3100
-F 0 "R23" H 10370 3146 50  0000 L CNN
-F 1 "200R" H 10370 3055 50  0000 L CNN
-F 2 "Mlab_R:SMD-0805" V 10230 3100 50  0001 C CNN
-F 3 "~" H 10300 3100 50  0001 C CNN
-	1    10300 3100
-	1    0    0    -1
-$EndComp
+P 10800 3650
+F 0 "R23" H 10870 3696 50  0000 L CNN
+F 1 "150R" H 10870 3605 50  0000 L CNN
+F 2 "Mlab_R:SMD-0805" V 10730 3650 50  0001 C CNN
+F 3 "~" H 10800 3650 50  0001 C CNN
+	1    10800 3650
+	1    0    0    -1
+$EndComp
+$Comp
+L Device:Q_NPN_BEC Q1
+U 1 1 5C06117E
+P 9450 4100
+F 0 "Q1" H 9641 4146 50  0000 L CNN
+F 1 "BC817" H 9641 4055 50  0000 L CNN
+F 2 "Package_TO_SOT_SMD:SOT-23" H 9650 4200 50  0001 C CNN
+F 3 "~" H 9450 4100 50  0001 C CNN
+	1    9450 4100
+	1    0    0    -1
+$EndComp
+$Comp
+L power:GND #PWR0140
+U 1 1 5C062773
+P 9550 4350
+F 0 "#PWR0140" H 9550 4100 50  0001 C CNN
+F 1 "GND" H 9555 4177 50  0000 C CNN
+F 2 "" H 9550 4350 50  0001 C CNN
+F 3 "" H 9550 4350 50  0001 C CNN
+	1    9550 4350
+	1    0    0    -1
+$EndComp
+Wire Wire Line
+	9550 4350 9550 4300
+Wire Wire Line
+	9550 3900 9550 3800
+Wire Wire Line
+	9550 3500 9550 3400
+$Comp
+L power:+3.3V #PWR0141
+U 1 1 5C07BB62
+P 9550 3050
+F 0 "#PWR0141" H 9550 2900 50  0001 C CNN
+F 1 "+3.3V" H 9565 3223 50  0000 C CNN
+F 2 "" H 9550 3050 50  0001 C CNN
+F 3 "" H 9550 3050 50  0001 C CNN
+	1    9550 3050
+	1    0    0    -1
+$EndComp
+Wire Wire Line
+	9550 3100 9550 3050
+$Comp
+L Device:Q_NPN_BEC Q2
+U 1 1 5C09D287
+P 10700 4100
+F 0 "Q2" H 10891 4146 50  0000 L CNN
+F 1 "BC817" H 10891 4055 50  0000 L CNN
+F 2 "Package_TO_SOT_SMD:SOT-23" H 10900 4200 50  0001 C CNN
+F 3 "~" H 10700 4100 50  0001 C CNN
+	1    10700 4100
+	1    0    0    -1
+$EndComp
+Wire Wire Line
+	10800 3400 10800 3500
+$Comp
+L power:GND #PWR0142
+U 1 1 5C0A568E
+P 10800 4350
+F 0 "#PWR0142" H 10800 4100 50  0001 C CNN
+F 1 "GND" H 10805 4177 50  0000 C CNN
+F 2 "" H 10800 4350 50  0001 C CNN
+F 3 "" H 10800 4350 50  0001 C CNN
+	1    10800 4350
+	1    0    0    -1
+$EndComp
+Wire Wire Line
+	10800 3800 10800 3900
+Wire Wire Line
+	10800 4350 10800 4300
+$Comp
+L power:+3.3V #PWR0143
+U 1 1 5C0B66F5
+P 10800 3050
+F 0 "#PWR0143" H 10800 2900 50  0001 C CNN
+F 1 "+3.3V" H 10815 3223 50  0000 C CNN
+F 2 "" H 10800 3050 50  0001 C CNN
+F 3 "" H 10800 3050 50  0001 C CNN
+	1    10800 3050
+	1    0    0    -1
+$EndComp
+Wire Wire Line
+	10800 3050 10800 3100
+$Comp
+L MLAB_HEADER:HEADER_1x02 J25
+U 1 1 5C0BF8EB
+P 10150 4050
+F 0 "J25" H 10069 3763 60  0000 C CNN
+F 1 "HEADER_1x02" H 10069 3869 60  0000 C CNN
+F 2 "Mlab_Pin_Headers:Straight_1x02" H 10150 4100 60  0001 C CNN
+F 3 "" H 10150 4100 60  0000 C CNN
+	1    10150 4050
+	-1   0    0    1
+$EndComp
+$Comp
+L MLAB_HEADER:HEADER_1x02 J24
+U 1 1 5C0BFAB9
+P 8900 4050
+F 0 "J24" H 8819 3763 60  0000 C CNN
+F 1 "HEADER_1x02" H 8819 3869 60  0000 C CNN
+F 2 "Mlab_Pin_Headers:Straight_1x02" H 8900 4100 60  0001 C CNN
+F 3 "" H 8900 4100 60  0000 C CNN
+	1    8900 4050
+	-1   0    0    1
+$EndComp
+Text Label 10400 4000 0    60   ~ 0
+P1.5
+Text Label 9150 4000 0    60   ~ 0
+P1.4
+Wire Wire Line
+	10350 4100 10500 4100
+Wire Wire Line
+	10350 4000 10400 4000
+Wire Wire Line
+	9100 4100 9250 4100
+Wire Wire Line
+	9100 4000 9150 4000
 $EndSCHEMATC

Commit message: edit
Parts:
- added J26: HEADER_2x01_PARALLEL, Mlab_Pin_Headers:Straight_2x01, symbol MLAB_HEADER:HEADER_2x01_PARALLEL
Connections:
- net GND: now also J26.1, J26.2
Changed lines of the file:
@@
 Wire Wire Line
 	9100 4000 9150 4000
+$Comp
+L MLAB_HEADER:HEADER_2x01_PARALLEL J26
+U 1 1 5C061FC2
+P 8900 2500
+F 0 "J26" H 9100 2500 60  0000 C CNN
+F 1 "HEADER_2x01_PARALLEL" H 8818 2641 60  0001 C CNN
+F 2 "Mlab_Pin_Headers:Straight_2x01" H 8900 2500 60  0001 C CNN
+F 3 "" H 8900 2500 60  0000 C CNN
+	1    8900 2500
+	-1   0    0    1
+$EndComp
+$Comp
+L power:GND #PWR04
+U 1 1 5C0621C8
+P 9200 2550
+F 0 "#PWR04" H 9200 2300 50  0001 C CNN
+F 1 "GND" H 9205 2377 50  0000 C CNN
+F 2 "" H 9200 2550 50  0001 C CNN
+F 3 "" H 9200 2550 50  0001 C CNN
+	1    9200 2550
+	1    0    0    -1
+$EndComp
+Wire Wire Line
+	9150 2500 9200 2500
+Wire Wire Line
+	9200 2500 9200 2550
 $EndSCHEMATC

Commit message: Edit
Parts:
- removed C24: 10uF, Mlab_R:SMD-0805, symbol Device:C_Small
- removed J5: BMIS-210, Mlab_Mechanical:BMI-S-210-F, symbol MLAB_Jumpers:CONN1_1
Other:
- note removed: "RF Shield"
Changed lines of the file:
@@
 Text Notes 9950 2150 0    60   ~ 0
 MOUNTING HOLES
-Connection ~ 9550 1350
 Wire Wire Line
 	10250 1800 10050 1800
@@
 Wire Wire Line
 	10150 950  9850 950
-Connection ~ 9550 950
-Wire Wire Line
-	9550 950  9550 1050
-Wire Wire Line
-	9550 1250 9550 1350
 $Comp
 L MLAB_Jumpers:JUMP_3X2 J1
@@
 F 3 "" H 1300 6950 60  0000 C CNN
 	1    1300 6950
-	1    0    0    -1
-$EndComp
-$Comp
-L Device:C_Small C24
-U 1 1 5C000C22
-P 9550 1150
-F 0 "C24" H 9550 1250 50  0000 L CNN
-F 1 "10uF" H 9550 1050 50  0000 L CNN
-F 2 "Mlab_R:SMD-0805" H 9550 1150 60  0001 C CNN
-F 3 "" H 9550 1150 60  0000 C CNN
-F 4 "C0805_100n" H 9550 1150 50  0001 C CNN "UST_id"
-	1    9550 1150
 	1    0    0    -1
 $EndComp
@@
 	7400 4850 7400 4750
 $Comp
-L MLAB_Jumpers:CONN1_1 J5
-U 1 1 5C0A274C
-P 4000 6600
-F 0 "J5" V 3857 6551 50  0000 R CNN
-F 1 "BMIS-210" V 3773 6551 40  0000 R CNN
-F 2 "Mlab_Mechanical:BMI-S-210-F" H 4050 6550 60  0001 C CNN
-F 3 "" H 4050 6550 60  0000 C CNN
-	1    4000 6600
-	0    -1   -1   0
-$EndComp
-$Comp
-L power:GND #PWR0132
-U 1 1 5C0A2C6F
-P 3950 6950
-F 0 "#PWR0132" H 3950 6700 50  0001 C CNN
-F 1 "GND" H 3955 6777 50  0000 C CNN
-F 2 "" H 3950 6950 50  0001 C CNN
-F 3 "" H 3950 6950 50  0001 C CNN
-	1    3950 6950
-	1    0    0    -1
-$EndComp
-Wire Wire Line
-	3950 6950 3950 6900
-Text Notes 4050 6950 0    60   ~ 0
-RF Shield
-$Comp
 L Device:R R21

Commit message: Edit
Connections:
- net #IRQ: no longer R21.1
- net #RST_C2CK: no longer R20.2
- net P0.1: no longer R21.2
- net #IRQ_1: now reaches R15.2, U2.23 (#IRQ)
- net #IRQ_1: now also R21.1
- net P0.1_1: now reaches R11.2, U2.29 (P0.1/AGND)
- net P0.1_1: now also R21.2
- net #RST_1: now reaches R14.2, U2.36 (#RST/C2CK)
- net #RST_1: now also R20.2
Other:
- moved on the sheet: J10, J11, J12, J13, J14, J15, J16, J17, J18, J19, J20, J21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

Commit message: edit
Parts:
- C1, C18, C20, C3, C5: UST_ID (none) -> 5c70984812875079b91f8bbd; UST_id C0805_100n -> (none)
- C10, C11, C9: UST_ID (none) -> 5c70984712875079b91f8b2f; UST_id C0805_100n -> (none)
- C12: UST_ID (none) -> 5c70984712875079b91f8b28; UST_id C0805_100n -> (none)
- C13: UST_ID (none) -> 5c70984812875079b91f8ba2; UST_id C0805_100n -> (none)
- C14, C22, C23, C25, C26, C27, C28: UST_ID (none) -> 5c70984712875079b91f8b49; UST_id C0805_100n -> (none)
- C15: UST_ID (none) -> 5c70984712875079b91f8b37; UST_id C0805_100n -> (none)
- C16, C19, C2: UST_ID (none) -> 5c70984712875079b91f8b4c; UST_id C0805_100n -> (none)
- C17: UST_ID (none) -> 5c70984712875079b91f8b3b; UST_id C0805_100n -> (none)
- C4, C6: UST_ID (none) -> 5c70984712875079b91f8b2e; UST_id C0805_100n -> (none)
- C7, C8: UST_ID (none) -> 5c70984712875079b91f8b32; UST_id C0805_100n -> (none)
- D1: UST_ID (none) -> 5c70984512875079b91f88ac
- D2: UST_ID (none) -> 5c70984412875079b91f8896
- D3: UST_ID (none) -> 5c70984412875079b91f8895
- J2, J3: UST_ID (none) -> 5c70984412875079b91f87ac
- L1, L2, R1, R21: UST_ID (none) -> 5c70984512875079b91f896b
- L10, L9: UST_ID (none) -> 5c70984812875079b91f8ba4
- L3, L4, L5, L6: UST_ID (none) -> 5c70984412875079b91f8806
- L7: UST_ID (none) -> 5c70984412875079b91f8809
- L8: UST_ID (none) -> 5c70984412875079b91f880d
- Q1, Q2: UST_ID (none) -> 5c70984712875079b91f8aec
- R10, R11, R12, R13, R14, R15, R16, R17, R18, R19, R2, R3, R4, R5, R6, R7, R8, R9: UST_ID (none) -> 5c70984512875079b91f8970
- R20: UST_ID (none) -> 5c70984512875079b91f898c
- R22, R23: UST_ID (none) -> 5c70984512875079b91f897a
- U1: UST_ID (none) -> 5c70984712875079b91f8af9
- U2: UST_ID (none) -> 5c70984812875079b91f8ba3
- Y1: UST_ID (none) -> 5c70984712875079b91f8b1b
- Y2: UST_ID (none) -> 5c70984712875079b91f8ba1
