File: mechanical/WINDGAUGE03A/hw/sch_pcb/WINDGAUGE03A_PCB01A/WINDGAUGE03A_PCB01A.sch (KiCad schematic (older format))
At the start: 9 parts, among them M1 HOLE, M2 HOLE, M3 HOLE, M4 HOLE, U1 SDP3x

Commit message: edit
Parts:
- added C? (x3): 100nF, Mlab_R:SMD-0805, symbol Device:C
- added U2: ICM-20948, Sensor_Motion:InvenSense_QFN-24_3x3mm_P0.4mm, symbol Sensor_Motion:ICM-20948
Connections:
- net labels added: VDDIO
- wire segments 16 -> 29
- no-connect marks 0 -> 3
Changed lines of the file:
@@
 EESchema Schematic File Version 4
-EELAYER 26 0
+LIBS:WINDGAUGE03A_PCB01A-cache
+EELAYER 29 0
 EELAYER END
 $Descr A4 11693 8268
@@
 SDA
 $Comp
-L power:VDD #PWR?
+L power:VDD #PWR0103
 U 1 1 5C5D0C06
 P 5300 3000
-F 0 "#PWR?" H 5300 2850 50  0001 C CNN
+F 0 "#PWR0103" H 5300 2850 50  0001 C CNN
 F 1 "VDD" H 5317 3173 50  0000 C CNN
 F 2 "" H 5300 3000 50  0001 C CNN
@@
 Wire Wire Line
 	5300 3100 5300 3000
+NoConn ~ 4750 3650
+$Comp
+L Sensor_Motion:ICM-20948 U2
+U 1 1 5C5C5B62
+P 4050 5150
+F 0 "U2" H 3700 5800 50  0000 C CNN
+F 1 "ICM-20948" H 4150 4800 50  0000 C CNN
+F 2 "Sensor_Motion:InvenSense_QFN-24_3x3mm_P0.4mm" H 4050 4150 50  0001 C CNN
+F 3 "http://www.invensense.com/wp-content/uploads/2016/06/DS-000189-ICM-20948-v1.3.pdf" H 4050 5000 50  0001 C CNN
+	1    4050 5150
+	1    0    0    -1
+$EndComp
+NoConn ~ 4550 5050
+NoConn ~ 4550 5150
+$Comp
+L Device:C C?
+U 1 1 5C5C720C
+P 4700 5550
+F 0 "C?" H 4815 5596 50  0000 L CNN
+F 1 "100nF" H 4815 5505 50  0000 L CNN
+F 2 "Mlab_R:SMD-0805" H 4738 5400 50  0001 C CNN
+F 3 "~" H 4700 5550 50  0001 C CNN
+	1    4700 5550
+	1    0    0    -1
+$EndComp
+$Comp
+L Device:C C?
+U 1 1 5C5C84AA
+P 3550 4100
+F 0 "C?" H 3665 4146 50  0000 L CNN
+F 1 "100nF" H 3665 4055 50  0000 L CNN
+F 2 "Mlab_R:SMD-0805" H 3588 3950 50  0001 C CNN
+F 3 "~" H 3550 4100 50  0001 C CNN
+	1    3550 4100
+	1    0    0    -1
+$EndComp
+$Comp
+L Device:C C?
+U 1 1 5C5C951D
+P 4350 4100
+F 0 "C?" H 4465 4146 50  0000 L CNN
+F 1 "100nF" H 4465 4055 50  0000 L CNN
+F 2 "Mlab_R:SMD-0805" H 4388 3950 50  0001 C CNN
+F 3 "~" H 4350 4100 50  0001 C CNN
+	1    4350 4100
+	1    0    0    -1
+$EndComp
+$Comp
+L power:GND #PWR?
+U 1 1 5C5C9FCC
+P 4350 4300
+F 0 "#PWR?" H 4350 4050 50  0001 C CNN
+F 1 "GND" H 4355 4127 50  0000 C CNN
+F 2 "" H 4350 4300 50  0001 C CNN
+F 3 "" H 4350 4300 50  0001 C CNN
+	1    4350 4300
+	1    0    0    -1
+$EndComp
+Wire Wire Line
+	4150 3850 4150 3950
+Wire Wire Line
+	4350 3950 4150 3950
+Connection ~ 4150 3950
+Wire Wire Line
+	4150 3950 4150 4450
+Wire Wire Line
+	4350 4300 4350 4250
+Wire Wire Line
+	3550 3950 3950 3950
+Wire Wire Line
+	3950 3950 3950 4450
+Wire Wire Line
+	3950 3950 3950 3850
+Connection ~ 3950 3950
+$Comp
+L power:GND #PWR?
+U 1 1 5C5CBFC0
+P 3550 4300
+F 0 "#PWR?" H 3550 4050 50  0001 C CNN
+F 1 "GND" H 3555 4127 50  0000 C CNN
+F 2 "" H 3550 4300 50  0001 C CNN
+F 3 "" H 3550 4300 50  0001 C CNN
+	1    3550 4300
+	1    0    0    -1
+$EndComp
+Wire Wire Line
+	3550 4300 3550 4250
+Wire Wire Line
+	4550 5350 4700 5350
+Wire Wire Line
+	4700 5350 4700 5400
+$Comp
+L power:GND #PWR?
+U 1 1 5C5CCD2E
+P 4700 5950
+F 0 "#PWR?" H 4700 5700 50  0001 C CNN
+F 1 "GND" H 4705 5777 50  0000 C CNN
+F 2 "" H 4700 5950 50  0001 C CNN
+F 3 "" H 4700 5950 50  0001 C CNN
+	1    4700 5950
+	1    0    0    -1
+$EndComp
+$Comp
+L power:GND #PWR?
+U 1 1 5C5CDB1F
+P 4050 5950
+F 0 "#PWR?" H 4050 5700 50  0001 C CNN
+F 1 "GND" H 4055 5777 50  0000 C CNN
+F 2 "" H 4050 5950 50  0001 C CNN
+F 3 "" H 4050 5950 50  0001 C CNN
+	1    4050 5950
+	1    0    0    -1
+$EndComp
+Wire Wire Line
+	4700 5700 4700 5950
+Wire Wire Line
+	4050 5950 4050 5850
+Wire Wire Line
+	3550 5150 3200 5150
+Text Label 3200 5150 0    60   ~ 0
+VDDIO
+Text Label 3950 3850 1    60   ~ 0
+VDDIO
+$Comp
+L power:VDD #PWR?
+U 1 1 5C5CF95D
+P 4150 3850
+F 0 "#PWR?" H 4150 3700 50  0001 C CNN
+F 1 "VDD" H 4167 4023 50  0000 C CNN
+F 2 "" H 4150 3850 50  0001 C CNN
+F 3 "" H 4150 3850 50  0001 C CNN
+	1    4150 3850
+	1    0    0    -1
+$EndComp
 $EndSCHEMATC

Commit message: edit
Parts:
- removed M1, M2, M3, M4: HOLE, Mlab_Mechanical:MountingHole_3mm, symbol MLAB_MECHANICAL:HOLE
- removed R1, R2: 0R, Mlab_R:SMD-0805, symbol Device:R
- added C5, C6, C7, C8: 1uF, Mlab_R:SMD-0805, symbol Device:C
- added C? (x2): 100nF, Mlab_R:SMD-0805, symbol Device:C
- added J1: SM07B-GHS-TB, Connector_JST:JST_GH_SM07B-GHS-TB_1x07-1MP_P1.25mm_Horizontal, symbol MLAB_CONNECTORS_JST:SM07B-GHS-TB
- added R? (x4): -, Mlab_R:SMD-0805, symbol Device:R
- added R? (x4): 10k, Mlab_R:SMD-0805, symbol Device:R
- added U4: MIC5504-3.3YM5-TR, Package_TO_SOT_SMD:SOT-23-5, symbol Regulator_Linear:MIC5504-3.3YM5
- added U5: MIC5504-1.8YM5-TR, Package_TO_SOT_SMD:SOT-23-5, symbol Regulator_Linear:MIC5504-1.8YM5
- added U6: TXS0108EPW, Package_SO:TSSOP-20_4.4x6.5mm_P0.65mm, symbol Logic_LevelTranslator:TXS0108EPW
- gave numbers to parts that had none: 3
Connections:
- net labels added: !SPI_SS1_1V8, !SPI_SS1_3V3, !SPI_SS2_3V3, +1V8, +3.3V, +5V, P_SCL_1V8, P_SCL_3V3, P_SDA_1V8, P_SDA_3V3, SPI_EXT_MISO_1V8, SPI_EXT_MISO_3V3, SPI_EXT_MOSI_1V8, SPI_EXT_MOSI_3V3, SPI_EXT_SCK_1V8, SPI_EXT_SCK_3V3
- net labels removed: SCL, SDA, VDD, VDDIO
- wire segments 29 -> 103
Other:
- note added: "SPI - Dronecode Autopilot\nConnector Standard"
- note removed: "MOUNTING HOLES"
- moved on the sheet: C1, C2, C3, C4, R3, U1, U2

Commit message: edit
Parts:
- removed R3: 0R, Mlab_R:SMD-0805, symbol Device:R
- added C11: 10uF, Mlab_R:SMD-0805, symbol Device:C
- added D1: BZV55C-5,6V, Diode_SMD:D_MiniMELF, symbol Device:D
- C1, C2, C3, C4, C5, C6, C7, C8: footprint Mlab_R:SMD-0805 -> Mlab_R:SMD-0603
- C10, C9: renamed from C?; footprint Mlab_R:SMD-0805 -> Mlab_R:SMD-0603
- R1, R6, R7, R8, R9: renamed from R?; footprint Mlab_R:SMD-0805 -> Mlab_R:SMD-0603
- R2: renamed from R?; value - -> 0R; footprint Mlab_R:SMD-0805 -> Mlab_R:SMD-0603
- R4, R5: renamed from R?; value - -> 10k; footprint Mlab_R:SMD-0805 -> Mlab_R:SMD-0603
Connections:
- net !SPI_SS1_1V8: now also U6.6 (A5); no longer U6.8 (A7)
- net !SPI_SS1_3V3: now also U6.15 (B5); no longer U6.13 (B7)
- net +1V8: no longer C3.1, U2.13 (VDD)
- net +3V3: now also C3.1, U2.13 (VDD)
- net +5V: now also C11.1, D1.1 (K)
- net GND: now also U1.9 (ADDR), C11.2, D1.2 (A)
- net P_SCL_1V8: now also U6.4 (A3); no longer U6.3 (A2)
- net P_SCL_3V3: now also U6.17 (B3); no longer U6.18 (B2)
- net P_SDA_1V8: now also U6.5 (A4); no longer U6.1 (A1)
- net P_SDA_3V3: now also U6.16 (B4); no longer U6.20 (B1)
- net SPI_EXT_MISO_1V8: now also U6.3 (A2); no longer U6.6 (A5)
- net SPI_EXT_MISO_3V3: now also U6.18 (B2); no longer U6.15 (B5)
- net SPI_EXT_MOSI_1V8: now also U6.8 (A7); no longer U6.5 (A4)
- net SPI_EXT_MOSI_3V3: now also U6.13 (B7); no longer U6.16 (B4)
- net INT1_1V8: now reaches U2.12 (INT1)
- net INT1_1V8: now also U6.1 (A1)
- net !SPI_SS2_3V3 renamed INT1_3V3
- net INT1_3V3: now also U6.20 (B1)
Other:
- note added: "ADDR\n0x21\n"
- note removed: "ADDR\n0R - 0x21\n1,2k - 0x22\n2,7k - 0x23"
- note removed: "VDD 2,7-5,5V"

Commit message: edit
Parts:
- J1: symbol MLAB_CONNECTORS_JST:SM07B-GHS-TB -> WINDGAUGE03A_PCB01A-rescue:SM07B-GHS-TB-MLAB_CONNECTORS_JST
Changed lines of the file:
@@
 !SPI_SS1_3V3
 $Comp
-L MLAB_CONNECTORS_JST:SM07B-GHS-TB J1
+L WINDGAUGE03A_PCB01A-rescue:SM07B-GHS-TB-MLAB_CONNECTORS_JST J1
 U 1 1 5C5FCA2D
 P 1300 1600

Commit message: edit
Connections:
- net !SPI_SS1_1V8: now also U6.5 (A4); no longer U6.6 (A5)
- net !SPI_SS1_3V3: now also U6.16 (B4); no longer U6.15 (B5)
- net P_SDA_1V8: now also U6.6 (A5); no longer U6.5 (A4)
- net P_SDA_3V3: now also U6.15 (B5); no longer U6.16 (B4)
- net SPI_EXT_MOSI_1V8: now also U6.7 (A6); no longer U6.8 (A7)
- net SPI_EXT_MOSI_3V3: now also U6.14 (B6); no longer U6.13 (B7)
- net SPI_EXT_SCK_1V8: now also U6.8 (A7); no longer U6.7 (A6)
- net SPI_EXT_SCK_3V3: now also U6.13 (B7); no longer U6.14 (B6)
Changed lines of the file:
@@
 	1    0    0    -1
 $EndComp
-Text Label 6750 3500 0    60   ~ 0
+Text Label 6750 3600 0    60   ~ 0
 P_SDA_3V3
 Text Label 6750 3400 0    60   ~ 0
@@
 Wire Wire Line
 	6650 3300 6750 3300
-Text Label 5000 3500 0    60   ~ 0
+Text Label 5000 3600 0    60   ~ 0
 P_SDA_1V8
 Text Label 5350 3400 0    60   ~ 0
@@
 Text Label 4300 5450 0    60   ~ 0
 P_SCL_1V8
-Text Label 6750 3800 0    60   ~ 0
+Text Label 6750 3700 0    60   ~ 0
 SPI_EXT_MOSI_3V3
 Text Label 6750 3300 0    60   ~ 0
 SPI_EXT_MISO_3V3
-Text Label 6750 3600 0    60   ~ 0
+Text Label 6750 3500 0    60   ~ 0
 !SPI_SS1_3V3
-Text Label 6750 3700 0    60   ~ 0
+Text Label 6750 3800 0    60   ~ 0
 SPI_EXT_SCK_3V3
 Text Label 5000 3300 0    60   ~ 0
 SPI_EXT_MISO_1V8
-Text Label 5000 3700 0    60   ~ 0
+Text Label 5000 3800 0    60   ~ 0
 SPI_EXT_SCK_1V8
-Text Label 5000 3600 0    60   ~ 0
+Text Label 5000 3500 0    60   ~ 0
 !SPI_SS1_1V8
 Wire Wire Line
@@
 Wire Wire Line
 	5850 3400 5350 3400
-Text Label 5000 3800 0    60   ~ 0
+Text Label 5000 3700 0    60   ~ 0
 SPI_EXT_MOSI_1V8
 Wire Wire Line

Commit message: edit
Parts:
- C1, C10, C2, C3, C4, C9: UST_ID (none) -> 5c70984712875079b91f8b4c
- C11: UST_ID (none) -> 5c70984812875079b91f8bbd
- C5, C6, C7, C8: UST_ID (none) -> 5c70984712875079b91f8b50
- D1: UST_ID (none) -> 5c70984512875079b91f88b1
- J1: UST_ID (none) -> 5c7250081287500b4e112e78
- R2: UST_ID (none) -> 5c70984512875079b91f896b
- R4, R5, R6, R7, R8, R9: UST_ID (none) -> 5c70984612875079b91f899f
- U1: UST_ID (none) -> 5c70984812875079b91f8bd0
- U2: UST_ID (none) -> 5c725a431287500b4e112ef5
- U4: UST_ID (none) -> 5c7255e81287500b4e112ea2
- U5: UST_ID (none) -> 5c7256781287500b4e112eba
- U6: UST_ID (none) -> 5c7258471287500b4e112edd
Changed lines of the file:
@@
 EESchema Schematic File Version 4
 LIBS:WINDGAUGE03A_PCB01A-cache
-EELAYER 26 0
+EELAYER 29 0
 EELAYER END
 $Descr A4 11693 8268
@@
 F 2 "Mlab_IO:SDP3x" H 4200 1750 60  0001 C CNN
 F 3 "" H 4200 1750 60  0001 C CNN
+F 4 "5c70984812875079b91f8bd0" H 4200 1750 50  0001 C CNN "UST_ID"
 	1    4200 1750
 	1    0    0    -1
@@
 F 2 "Mlab_R:SMD-0603" H 4888 800 50  0001 C CNN
 F 3 "~" H 4850 950 50  0001 C CNN
+F 4 "5c70984712875079b91f8b4c" H 4850 950 50  0001 C CNN "UST_ID"
 	1    4850 950
 	1    0    0    -1
@@
 F 2 "Connector_JST:JST_GH_SM07B-GHS-TB_1x07-1MP_P1.25mm_Horizontal" H 1217 2091 60  0001 C CNN
 F 3 "" H 1300 1950 60  0000 C CNN
+F 4 "5c7250081287500b4e112e78" H 1300 1600 50  0001 C CNN "UST_ID"
 	1    1300 1600
 	-1   0    0    -1
@@
 F 2 "Mlab_R:SMD-0603" H 3438 4250 50  0001 C CNN
 F 3 "~" H 3400 4400 50  0001 C CNN
+F 4 "5c70984712875079b91f8b4c" H 3400 4400 50  0001 C CNN "UST_ID"
 	1    3400 4400
 	1    0    0    -1
@@
 F 2 "Mlab_R:SMD-0603" H 2638 4250 50  0001 C CNN
 F 3 "~" H 2600 4400 50  0001 C CNN
+F 4 "5c70984712875079b91f8b4c" H 2600 4400 50  0001 C CNN "UST_ID"
 	1    2600 4400
 	1    0    0    -1
@@
 F 2 "Mlab_R:SMD-0603" H 3788 5700 50  0001 C CNN
 F 3 "~" H 3750 5850 50  0001 C CNN
+F 4 "5c70984712875079b91f8b4c" H 3750 5850 50  0001 C CNN "UST_ID"
 	1    3750 5850
 	1    0    0    -1
@@
 F 2 "Sensor_Motion:InvenSense_QFN-24_3x3mm_P0.4mm" H 3100 4450 50  0001 C CNN
 F 3 "http://www.invensense.com/wp-content/uploads/2016/06/DS-000189-ICM-20948-v1.3.pdf" H 3100 5300 50  0001 C CNN
+F 4 "5c725a431287500b4e112ef5" H 3100 5450 50  0001 C CNN "UST_ID"
 	1    3100 5450
 	1    0    0    -1
@@
 F 2 "Package_TO_SOT_SMD:SOT-23-5" H 10300 1900 50  0001 C CNN
 F 3 "http://ww1.microchip.com/downloads/en/DeviceDoc/MIC550X.pdf" H 10050 2550 50  0001 C CNN
+F 4 "5c7256781287500b4e112eba" H 10300 2300 50  0001 C CNN "UST_ID"
 	1    10300 2300
 	1    0    0    -1
@@
 F 2 "Mlab_R:SMD-0603" H 9438 1050 50  0001 C CNN
 F 3 "~" H 9400 1200 50  0001 C CNN
+F 4 "5c70984712875079b91f8b50" H 9400 1200 50  0001 C CNN "UST_ID"
 	1    9400 1200
 	1    0    0    -1
@@
 F 2 "Mlab_R:SMD-0603" H 10888 1050 50  0001 C CNN
 F 3 "~" H 10850 1200 50  0001 C CNN
+F 4 "5c70984712875079b91f8b50" H 10850 1200 50  0001 C CNN "UST_ID"
 	1    10850 1200
 	1    0    0    -1
@@
 F 2 "Mlab_R:SMD-0603" H 9438 2250 50  0001 C CNN
 F 3 "~" H 9400 2400 50  0001 C CNN
+F 4 "5c70984712875079b91f8b50" H 9400 2400 50  0001 C CNN "UST_ID"
 	1    9400 2400
 	1    0    0    -1
@@
 F 2 "Mlab_R:SMD-0603" H 10888 2250 50  0001 C CNN
 F 3 "~" H 10850 2400 50  0001 C CNN
+F 4 "5c70984712875079b91f8b50" H 10850 2400 50  0001 C CNN "UST_ID"
 	1    10850 2400
 	1    0    0    -1
@@
 F 2 "Package_TO_SOT_SMD:SOT-23-5" H 10300 700 50  0001 C CNN
 F 3 "http://ww1.microchip.com/downloads/en/DeviceDoc/MIC550X.pdf" H 10050 1350 50  0001 C CNN
+F 4 "5c7255e81287500b4e112ea2" H 10300 1100 50  0001 C CNN "UST_ID"
 	1    10300 1100
 	1    0    0    -1
@@
 F 2 "Package_SO:TSSOP-20_4.4x6.5mm_P0.65mm" H 6250 2750 50  0001 C CNN
 F 3 "www.ti.com/lit/ds/symlink/txs0108e.pdf" H 6250 3400 50  0001 C CNN
+F 4 "5c7258471287500b4e112edd" H 6250 3500 50  0001 C CNN "UST_ID"
 	1    6250 3500
 	1    0    0    -1
@@
 F 2 "Mlab_R:SMD-0603" H 5688 2500 50  0001 C CNN
 F 3 "~" H 5650 2650 50  0001 C CNN
+F 4 "5c70984712875079b91f8b4c" H 5650 2650 50  0001 C CNN "UST_ID"
 	1    5650 2650
 	-1   0    0    1
@@
 F 2 "Mlab_R:SMD-0603" H 6738 2500 50  0001 C CNN
 F 3 "~" H 6700 2650 50  0001 C CNN
+F 4 "5c70984712875079b91f8b4c" H 6700 2650 50  0001 C CNN "UST_ID"
 	1    6700 2650
 	1    0    0    -1
@@
 F 2 "Mlab_R:SMD-0603" V 730 5350 50  0001 C CNN
 F 3 "~" H 800 5350 50  0001 C CNN
+F 4 "5c70984512875079b91f896b" H 800 5350 50  0001 C CNN "UST_ID"
 	1    800  5350
 	1    0    0    -1
@@
 F 2 "Mlab_R:SMD-0603" V 3280 1050 50  0001 C CNN
 F 3 "~" H 3350 1050 50  0001 C CNN
+F 4 "5c70984612875079b91f899f" H 3350 1050 50  0001 C CNN "UST_ID"
 	1    3350 1050
 	1    0    0    -1
@@
 F 2 "Mlab_R:SMD-0603" V 3530 1050 50  0001 C CNN
 F 3 "~" H 3600 1050 50  0001 C CNN
+F 4 "5c70984612875079b91f899f" H 3600 1050 50  0001 C CNN "UST_ID"
 	1    3600 1050
 	1    0    0    -1
@@
 F 2 "Mlab_R:SMD-0603" V 3780 4950 50  0001 C CNN
 F 3 "~" H 3850 4950 50  0001 C CNN
+F 4 "5c70984612875079b91f899f" H 3850 4950 50  0001 C CNN "UST_ID"
 	1    3850 4950
 	1    0    0    -1
@@
 F 2 "Mlab_R:SMD-0603" V 4030 4950 50  0001 C CNN
 F 3 "~" H 4100 4950 50  0001 C CNN
+F 4 "5c70984612875079b91f899f" H 4100 4950 50  0001 C CNN "UST_ID"
 	1    4100 4950
 	1    0    0    -1
@@
 F 2 "Mlab_R:SMD-0603" V 980 4950 50  0001 C CNN
 F 3 "~" H 1050 4950 50  0001 C CNN
+F 4 "5c70984612875079b91f899f" H 1050 4950 50  0001 C CNN "UST_ID"
 	1    1050 4950
 	1    0    0    -1
@@
 F 2 "Mlab_R:SMD-0603" V 1230 4950 50  0001 C CNN
 F 3 "~" H 1300 4950 50  0001 C CNN
+F 4 "5c70984612875079b91f899f" H 1300 4950 50  0001 C CNN "UST_ID"
 	1    1300 4950
 	1    0    0    -1
@@
 F 2 "Diode_SMD:D_MiniMELF" H 950 2950 50  0001 C CNN
 F 3 "~" H 950 2950 50  0001 C CNN
+F 4 "5c70984512875079b91f88b1" H 950 2950 50  0001 C CNN "UST_ID"
 	1    950  2950
 	0    1    1    0
@@
 F 2 "Mlab_R:SMD-0805" H 1388 2800 50  0001 C CNN
 F 3 "~" H 1350 2950 50  0001 C CNN
+F 4 "5c70984812875079b91f8bbd" H 1350 2950 50  0001 C CNN "UST_ID"
 	1    1350 2950
 	1    0    0    -1

Commit message: edit description
Other:
- note added: "SCL"
- note added: "SDA"
Changed lines of the file:
@@
-EESchema Schematic File Version 4
-LIBS:WINDGAUGE03A_PCB01A-cache
-EELAYER 29 0
+EESchema Schematic File Version 5
+EELAYER 30 0
 EELAYER END
 $Descr A4 11693 8268
@@
 Comment3 "nickname <email@example.com>"
 Comment4 "BSD"
+Comment5 ""
+Comment6 ""
+Comment7 ""
+Comment8 ""
+Comment9 ""
 $EndDescr
 $Comp
@@
 NoConn ~ 6650 3900
 NoConn ~ 5850 3900
+Text Notes 2450 1550 0    60   ~ 0
+SDA
+Text Notes 2450 1350 0    60   ~ 0
+SCL
 $EndSCHEMATC
