File: sensors/GPS01C/hw/sch_pcb/GPS01C.sch (KiCad schematic (older format))
At the start: 53 parts, among them M1 HOLE, M2 HOLE, M3 HOLE, M4 HOLE

Commit message: Schema
Parts:
- added J? (x5): HEADER_2x01_PARALLEL, symbol MLAB_HEADER:HEADER_2x01_PARALLEL
- added JP? (x2): Jumper_2_Bridged, symbol Jumper:Jumper_2_Bridged
- added R? (x2): 10k, symbol Device:R
Connections:
- net +3V3: now also J?.1, J?.2, R?.1, R?.1
- net GND: now also J?.1, J?.1, J?.2, J?.2
- net SDA/#CS: now also JP?.2 (B)
- net TIMEPULSE: now also J?.1, J?.2
- net LNEN: now reaches U?.14 (LNA_EN)
- net LNEN: now also J?.1, J?.2
- net CLK renamed SCL/CLK
- net SCL/CLK: now also JP?.2 (B)
- new net: JP?.1 (A), R?.2 (x2)
- no-connect marks 1 -> 0
Other:
- moved on the sheet: C?, D?, J?, JP?, L?, R?, U?

Commit message: Edit
Parts:
- removed JP? (x3): Jumper_2_Bridged, symbol Jumper:Jumper_2_Bridged
- added J17: u.FL, Connector_Coaxial:U.FL_Molex_MCRF_73412-0110_Vertical, symbol MLAB_CONNECTORS:SMA
- added JP2: Jumper_2_Bridged, Mlab_Pin_Headers:Straight_1x02, symbol Jumper:Jumper_2_Bridged
- added JP9: Jumper_2_Open, Mlab_Pin_Headers:Straight_1x02, symbol Jumper:Jumper_2_Open
- added R15: 10k, Mlab_R:SMD-0805, symbol Device:R
- C1: renamed from C?; footprint (none) -> Capacitor_THT:CP_Radial_D8.0mm_P3.50mm
- C2, C3, C4, C5, C6, C7: renamed from C?; footprint (none) -> Mlab_R:SMD-0805
- D1: renamed from D?; footprint (none) -> Diode_SMD:D_MiniMELF
- D2: renamed from D?; footprint (none) -> Diode_SMD:D_SMA
- D3, D4, D5, D6: renamed from D?; footprint (none) -> Mlab_D:LED_1206
- F1: renamed from F?; footprint (none) -> Mlab_F:1812
- J1, J15, J3: renamed from J?; footprint (none) -> Mlab_Pin_Headers:Straight_2x03
- J10, J11, J12, J13, J14, J16, J4, J5, J6, J7, J8, J9: renamed from J?; footprint (none) -> Mlab_Pin_Headers:Straight_2x01
- J18: renamed from J?; footprint (none) -> Connector_Coaxial:SMB_Jack_Vertical
- J2: renamed from J?; footprint (none) -> Connector_USB:USB_B_OST_USB-B1HSxx_Horizontal
- JP1: renamed from JP?; footprint (none) -> Mlab_Pin_Headers:Straight_1x03
- JP4: renamed from JP?; footprint (none) -> Jumper:SolderJumper-2_P1.3mm_Open_RoundedPad1.0x1.5mm
- JP6, JP7, JP8: renamed from JP?; footprint (none) -> Mlab_Pin_Headers:Straight_1x02
- L1: renamed from L?; footprint (none) -> Inductor_SMD:L_1210_3225Metric
- L2: renamed from L?; footprint (none) -> Mlab_R:SMD-0805
- R1, R10, R11, R12, R13, R14, R2, R3, R4, R5, R6, R7, R8, R9: renamed from R?; footprint (none) -> Mlab_R:SMD-0805
- gave numbers to parts that had none: 3
Connections:
- net +3V3: now also JP2.2 (B), JP9.1 (A); no longer D3.2 (A)
- net GEO_STAT: now also D4.2 (A); no longer R12.1
- net GND: now also R12.2, R13.2, R14.2, J17.2, R15.2; no longer D4.1 (K), D5.1 (K), D6.1 (K)
- net RTK_STAT: now also D5.2 (A); no longer R13.1
- net SCL/CLK: now also R3.2
- net SDA/#CS: now also R2.2
- net TIMEPULSE: now also D6.2 (A); no longer J16.1, J16.2, R14.1
- net at J18.1, L2.2, U3.11 (RF_IN): now also J17.1
- net at JP6.1 (A), U3.3 (TIMEPULSE): now also J16.1, J16.2
- net at U3.7 (VDD_USB): now also JP2.1 (A), R15.1
- new net: D3.2 (A), JP9.2 (B)
- new net: D4.1 (K), R12.1
- new net: D5.1 (K), R13.1
- new net: D6.1 (K), R14.1
Other:
- moved on the sheet: D3, D4, D5, D6, J16, R10, R12, R13, R14

Commit message: Edit
Connections:
- net #SAFEB: now reaches J12.1, J12.2, U3.1 (~SAFEBOOT)
- net D_SEL: now reaches JP4.2 (B), U3.2 (D_SEL)
- net EXTINT: now reaches J11.1, J11.2, U3.4 (EXTINT)
- net VDD_USB: now reaches JP2.1 (A), R15.1, U3.7 (VDD_USB)
- net #RESET: now reaches J13.1, J13.2, U3.8 (~RESET)
Changed lines of the file:
@@
 Wire Wire Line
 	5000 1800 5000 1900
+Text Label 4450 4050 0    60   ~ 0
+EXTINT
+Text Label 4450 4350 0    60   ~ 0
+#RESET
+Text Label 4450 4250 0    60   ~ 0
+#SAFEB
+Text Label 4350 4450 0    60   ~ 0
+D_SEL
+Connection ~ 4650 4450
+Wire Wire Line
+	4350 4450 4650 4450
+Text Label 5450 2450 3    60   ~ 0
+VDD_USB
 $EndSCHEMATC
