File: power_supply/STEPUPDC01A/hw/sch_pcb/STEPUPDC01A.kicad_pcb (KiCad board)
At the start: 2 copper layers, 0 parts

Commit message: edit
Parts:
- added C1: 10uF, Mlab_R:SMD-0805, B.Cu at (106.7, 62.2)
- added C3: 1uF/50V, Mlab_R:SMD-0805, B.Cu at (113.7, 66.7)
- added C4: 100nF, Mlab_R:SMD-0805, B.Cu at (113.7, 69.2)
- added C5: 100nF, Mlab_R:SMD-0805, B.Cu at (110.5, 74.3)
- added C6: 1uF/50V, Mlab_R:SMD-0805, B.Cu at (108.0, 74.3)
- added D1: M4, Mlab_D:Diode-SMA_Standard, B.Cu at (111.8, 54.0)
- added D2: NSR05T40XV2T5G, Diode_SMD:D_SOD-523, B.Cu at (113.0, 64.8)
- added J1: HEADER_2x03_PARALLEL, Mlab_Pin_Headers:Straight_2x03, F.Cu at (103.5, 57.1)
- added J2: HEADER_1x02, Mlab_Pin_Headers:Straight_1x02, F.Cu at (116.8, 72.4)
- added J4: HEADER_2x04_PARALLEL, Mlab_Pin_Headers:Straight_2x04, F.Cu at (103.5, 68.6)
- added L1: 47uH -DE0703-47, Mlab_L:DE0703, B.Cu at (112.4, 59.7)
- added M1: HOLE, Mlab_Mechanical:MountingHole_3mm, F.Cu at (113.7, 78.7)
- added M2: HOLE, Mlab_Mechanical:MountingHole_3mm, F.Cu at (103.5, 48.3)
- added M3: HOLE, Mlab_Mechanical:MountingHole_3mm, F.Cu at (113.7, 48.3)
- added M4: HOLE, Mlab_Mechanical:MountingHole_3mm, F.Cu at (103.5, 78.7)
- added R1: 10k, Mlab_R:SMD-0805, B.Cu at (116.8, 67.9)
- added R2: 140k, Mlab_R:SMD-0805, B.Cu at (110.5, 70.5)
- added R3: 6k49, Mlab_R:SMD-0805, B.Cu at (108.0, 70.5)
- added R4: 100R, Mlab_R:SMD-0805, B.Cu at (113.0, 72.4)
- added U1: MAX5026, Package_TO_SOT_SMD:SOT-23-6_Handsoldering, B.Cu at (109.2, 66.0)

Commit message: Edit
Parts:
- moved R3 0.06 mm to (108.0, 70.5), turned to 270 degrees
Routing:
- net GND: track 0.00 -> 95.1 mm, vias 0 -> 49
- net /#SHDN: track 0.00 -> 19.6 mm, vias 0 -> 1
- net /Vout: track 0.00 -> 18.2 mm
- net /Vin: track 0.00 -> 15.6 mm, vias 0 -> 2
- net Net-(C3-Pad1): track 0.00 -> 11.0 mm
- net Net-(D2-Pad2): track 0.00 -> 7.05 mm
- net /FB: track 0.00 -> 4.90 mm
- added copper zone on B.Cu, net /Vin
- added copper zone on B.Cu, net GND
- added copper zone on F.Cu, net GND
- added copper zone on B.Cu, net Net-(D2-Pad2)
Other:
- board outline added: 19.8 x 40.1 mm
- net class Default: via_dia 0.6 -> 0.8
- net class MLAB_default: via_dia 0.6 -> 0.8
- net class MLAB_power: via_drill 0.6 -> 0.4
- rule via_min_drill: 0.3 -> 0.4
- rule via_min_size: 0.4 -> 0.8
- board text added: "#SHDN"
- board text added: "2018"
- board text added: "3-11V"
- board text added: "GND"
- board text added: "JACHO"
- board text added: "MAX 36V"
- board text added: "MLAB.CZ"
- board text added: "POWER IN"
- board text added: "POWER OUT"
- board text added: "STEPUPDC01A"

Commit message: Edit
Connections:
- M1 pad 1: GND -> Net-(M1-Pad1)
- M2 pad 1: GND -> Net-(M2-Pad1)
- M3 pad 1: GND -> Net-(M3-Pad1)
- M4 pad 1: GND -> Net-(M4-Pad1)
Changed lines of the file:
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@@
     (zones 0)
     (modules 20)
-    (nets 8)
+    (nets 12)
   )
   (page A4)
@@
   )
   (setup
-    (last_trace_width 0.3)
+    (last_trace_width 0.25)
     (user_trace_width 0.3)
     (user_trace_width 0.4)
@@
   (net 6 /#SHDN)
   (net 7 /FB)
+  (net 8 "Net-(M1-Pad1)")
+  (net 9 "Net-(M2-Pad1)")
+  (net 10 "Net-(M3-Pad1)")
+  (net 11 "Net-(M4-Pad1)")
   (net_class Default "This is the default net class."
     (clearance 0.2)
@@
     (add_net "Net-(C3-Pad1)")
     (add_net "Net-(D2-Pad2)")
+    (add_net "Net-(M1-Pad1)")
+    (add_net "Net-(M2-Pad1)")
+    (add_net "Net-(M3-Pad1)")
+    (add_net "Net-(M4-Pad1)")
   )
   (net_class MLAB_default ""
@@
     (fp_circle (center 0 0) (end 2.99974 0) (layer Cmts.User) (width 0.381))
     (pad 1 thru_hole circle (at 0 0) (size 6 6) (drill 3) (layers *.Cu *.Adhes *.Mask)
-      (net 2 GND) (clearance 1) (zone_connect 2))
+      (net 8 "Net-(M1-Pad1)") (clearance 1) (zone_connect 2))
     (model ${MLAB}/src/3d/mechanical/m3_komplet.step
       (at (xyz 0 0 0))
@@
     (fp_circle (center 0 0) (end 2.99974 0) (layer Cmts.User) (width 0.381))
     (pad 1 thru_hole circle (at 0 0) (size 6 6) (drill 3) (layers *.Cu *.Adhes *.Mask)
-      (net 2 GND) (clearance 1) (zone_connect 2))
+      (net 9 "Net-(M2-Pad1)") (clearance 1) (zone_connect 2))
     (model ${MLAB}/src/3d/mechanical/m3_komplet.step
       (at (xyz 0 0 0))
@@
     (fp_circle (center 0 0) (end 2.99974 0) (layer Cmts.User) (width 0.381))
     (pad 1 thru_hole circle (at 0 0) (size 6 6) (drill 3) (layers *.Cu *.Adhes *.Mask)
-      (net 2 GND) (clearance 1) (zone_connect 2))
+      (net 10 "Net-(M3-Pad1)") (clearance 1) (zone_connect 2))
     (model ${MLAB}/src/3d/mechanical/m3_komplet.step
       (at (xyz 0 0 0))
@@
     (fp_circle (center 0 0) (end 2.99974 0) (layer Cmts.User) (width 0.381))
     (pad 1 thru_hole circle (at 0 0) (size 6 6) (drill 3) (layers *.Cu *.Adhes *.Mask)
-      (net 2 GND) (clearance 1) (zone_connect 2))
+      (net 11 "Net-(M4-Pad1)") (clearance 1) (zone_connect 2))
     (model ${MLAB}/src/3d/mechanical/m3_komplet.step
       (at (xyz 0 0 0))
@@
   (segment (start 117.645001 62.694999) (end 117.475 62.865) (width 0.3) (layer B.Cu) (net 2))
   (via (at 117.475 62.865) (size 0.8) (drill 0.4) (layers F.Cu B.Cu) (net 2))
-  (segment (start 111.1 51.435) (end 117.475 51.435) (width 0.3) (layer B.Cu) (net 2))
+  (segment (start 110.744 52.197) (end 117.119 52.197) (width 0.3) (layer B.Cu) (net 2))
   (segment (start 109.76 53.975) (end 109.76 52.775) (width 0.3) (layer B.Cu) (net 2))
   (segment (start 109.76 52.775) (end 111.1 51.435) (width 0.3) (layer B.Cu) (net 2))

Commit message: Module documentation update.
Other:
- net class Default removed
- net class MLAB_default removed
- net class MLAB_power removed
